File: hardware/ubuntu-v2.1/circuits/TriggerAndCVs_connectors.brd (EAGLE design)
At the start: 64.8 x 41.6 mm, 11 parts, among them J1 6p-2.54

Commit message: Add files via upload
Parts:
- removed J1: 6p-2.54, pinhead:2X08/90
- added JP4: MOLEX_54548-1671MOLEX_54548-1671_0_0, Molex - 54548-1671:MOLEX_54548-1671_0
Connections:
- removed net N$1: CV_IN2.P$1, J1.1
- removed net N$2: CV_IN1.P$1, J1.3
- removed net N$3: CV_OUT2.P$1, J1.5
- removed net N$4: CV_OUT1.P$1, J1.7
- removed net N$5: J1.4, TRIG_OUT2.P$1
- removed net N$6: J1.6, TRIG_OUT1.P$1
- removed net N$7: J1.8, TRIG_IN2.P$1
- removed net N$8: J1.10, TRIG_IN1.P$1
- new net CV_IN_1: CV_IN1.P$1, JP4.8
- new net CV_IN_2: CV_IN2.P$1, JP4.7
- new net CV_OUT_1: CV_OUT1.P$1, JP4.10
- new net CV_OUT_2: CV_OUT2.P$1, JP4.6
- new net TRIG_IN_1: JP4.5, TRIG_IN1.P$1
- new net TRIG_IN_2: JP4.3, TRIG_IN2.P$1
- new net TRIG_OUT_1: JP4.4, TRIG_OUT1.P$1
- new net TRIG_OUT_2: JP4.1, TRIG_OUT2.P$1
- net GND: now also JP4.2, JP4.MP1, JP4.MP2; no longer J1.2
- net MIDI_RX_PIN4: now also JP4.12; no longer J1.14
- net MIDI_RX_PIN5: now also JP4.14; no longer J1.12
- net MIDI_TX_PIN4: now also JP4.15; no longer J1.11
- net MIDI_TX_PIN5: now also JP4.16; no longer J1.9
Routing:
- net N$5: track 64.1 -> 0.00 mm, vias 1 -> 0
- net N$7: track 42.7 -> 0.00 mm, vias 1 -> 0
- net N$6: track 41.7 -> 0.00 mm
- net N$1: track 39.7 -> 0.00 mm, vias 1 -> 0
- net N$8: track 39.5 -> 0.00 mm
- net TRIG_IN_2: track 0.00 -> 36.8 mm
- net TRIG_IN_1: track 0.00 -> 30.6 mm
- net TRIG_OUT_2: track 0.00 -> 29.8 mm
- net CV_IN_2: track 0.00 -> 26.8 mm
- net CV_IN_1: track 0.00 -> 25.7 mm
- net N$2: track 25.2 -> 0.00 mm
- net N$3: track 22.9 -> 0.00 mm
- net TRIG_OUT_1: track 0.00 -> 22.1 mm
- net MIDI_TX_PIN4: track 40.7 -> 19.3 mm
- net MIDI_RX_PIN4: track 52.9 -> 32.9 mm, vias 1 -> 0
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Other:
- board size 64.8 x 41.6 mm -> 64.8 x 42.9 mm

Commit message: Add files via upload
Parts:
- JP4: value MOLEX_54548-1671MOLEX_54548-1671_0_0 -> MOLEX_51281-2494MOLEX_51281-2494_0_0; device Molex - 54548-1671:MOLEX_54548-1671_0 -> Molex - 51281-2494:MOLEX_51281-2494_0
Connections:
- net CV_IN_1: now also JP4.9
- net CV_OUT_1: now also JP4.11
- net GND: now also JP4.19, JP4.20, JP4.21, JP4.22, JP4.23, JP4.24; no longer JP4.2
- net MIDI_RX_PIN4: now also JP4.13
- net MIDI_TX_PIN5: now also JP4.17
- net TRIG_OUT_2: now also JP4.2
Routing:
- net TRIG_IN_2: track 36.8 -> 33.9 mm
- net MIDI_TX_PIN5: track 26.4 -> 29.2 mm
- net MIDI_RX_PIN5: track 35.6 -> 38.2 mm
- net MIDI_TX_PIN4: track 19.3 -> 21.6 mm
- net CV_IN_1: track 25.7 -> 26.9 mm
- net CV_OUT_1: track 16.2 -> 17.4 mm
- net CV_OUT_2: track 17.5 -> 16.5 mm
- net MIDI_RX_PIN4: track 32.9 -> 34.0 mm
- net CV_IN_2: track 26.8 -> 25.8 mm
- net TRIG_IN_1: track 30.6 -> 29.6 mm
- net TRIG_OUT_2: track 29.8 -> 29.0 mm
- net TRIG_OUT_1: track 22.1 -> 21.4 mm
