File: hardware/ubuntu-v2.1/circuits/TriggerAndCVs_connectors.sch (EAGLE design)
At the start: 11 parts, among them J1 6p-2.54

Commit message: Add files via upload
Parts:
- removed J1: 6p-2.54, pinhead:PINHD-2X8/90
- added JP4: MOLEX_54548-1671MOLEX_54548-1671_0_0, Molex - 54548-1671:MOLEX_54548-1671MOLEX_54548-1671_0_0
Connections:
- removed net N$1: CV_IN2.2, J1.1
- removed net N$2: CV_IN1.2, J1.3
- removed net N$3: CV_OUT2.2, J1.5
- removed net N$4: CV_OUT1.2, J1.7
- removed net N$5: J1.4, TRIG_OUT2.2
- removed net N$6: J1.6, TRIG_OUT1.2
- removed net N$7: J1.8, TRIG_IN2.2
- removed net N$8: J1.10, TRIG_IN1.2
- new net CV_IN_1: CV_IN1.2, JP4.8
- new net CV_IN_2: CV_IN2.2, JP4.7
- new net CV_OUT_1: CV_OUT1.2, JP4.10
- new net CV_OUT_2: CV_OUT2.2, JP4.6
- new net TRIG_IN_1: JP4.5, TRIG_IN1.2
- new net TRIG_IN_2: JP4.3, TRIG_IN2.2
- new net TRIG_OUT_1: JP4.4, TRIG_OUT1.2
- new net TRIG_OUT_2: JP4.1, TRIG_OUT2.2
- net GND: now also JP4.2, JP4.MP1, JP4.MP2; no longer J1.2
- net MIDI_RX_PIN4: now also JP4.12; no longer J1.14
- net MIDI_RX_PIN5: now also JP4.14; no longer J1.12
- net MIDI_TX_PIN4: now also JP4.15; no longer J1.11
- net MIDI_TX_PIN5: now also JP4.16; no longer J1.9

Commit message: Add files via upload
Parts:
- JP4: value MOLEX_54548-1671MOLEX_54548-1671_0_0 -> MOLEX_51281-2494MOLEX_51281-2494_0_0; device Molex - 54548-1671:MOLEX_54548-1671MOLEX_54548-1671_0_0 -> Molex - 51281-2494:MOLEX_51281-2494MOLEX_51281-2494_0_0
Connections:
- net CV_IN_1: now also JP4.9
- net CV_OUT_1: now also JP4.11
- net GND: now also JP4.19, JP4.20, JP4.21, JP4.22, JP4.23, JP4.24; no longer JP4.2
- net MIDI_RX_PIN4: now also JP4.13
- net MIDI_TX_PIN5: now also JP4.17
- net TRIG_OUT_2: now also JP4.2
Other:
- moved on the sheet: CV_IN1, CV_IN2, CV_OUT1, CV_OUT2, MIDI_RX, MIDI_TX
