File: hardware/ubuntu-v2.1/circuits/TriggersCV_Circuitry.brd (EAGLE design)
At the start: 78.1 x 43.8 mm, 39 parts, among them IC1 TL072D, IC10 74AHCT1G125DBV, IC11 74AHCT1G125DBV, J1 MOLEX_78127-1408MOLEX_78127-1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, Q1 MMBT3904, Q6 MMBT3904

Commit message: Add files via upload
Parts:
- removed D5: 250mA/100V, SparkFun-DiscreteSemi:SOD-323
- removed J_PANEL: 6p-2.54, Molex - 54548-1671:MOLEX_54548-1671_0
- removed OK1: OG-OPTOCOUPLERS_6N137SMT, TriggersCV_Circuitry:OG-OPTOCOUPLERS_DIL8-SMD
- removed R35: 220, resistor:R0603
- removed R37: 10k, resistor:R0603
- removed R39, R40: 51, resistor:R0603
- added JP1_MIDI: (no value), pinhead:1X04
- added JP3: MOLEX_51281-2494MOLEX_51281-2494_0_0, Molex - 51281-2494:MOLEX_51281-2494_0
- added JP5_POTS: PINHD-1X6, audio amplifier example:1X06
- added JPWR: POWER, eurorack:POWER_16
- D1, D2, D3, D4, D6, D7: device SparkFun-DiscreteSemi:SOD-323 -> My_Diodes2:SPARKFUN-DISCRETESEMI_SOD-323
- JP4: value MOLEX_54548-1671MOLEX_54548-1671_0_0 -> MOLEX_51281-2494MOLEX_51281-2494_0_0; device Molex - 54548-1671:MOLEX_54548-1671_0 -> Molex - 51281-2494:MOLEX_51281-2494_0
- moved Q1 37.3 mm to (46.4, 26.7), turned to 90 degrees
- moved R9 37.1 mm to (47.0, 12.7), turned to 0 degrees
- moved JP4 34.3 mm to (18.4, 32.4)
- moved R6 32.5 mm to (17.1, 8.89), turned to 0 degrees
- moved R1 30.0 mm to (10.2, 9.36), turned to 270 degrees
- moved R7 28.9 mm to (13.3, 8.89)
- moved D2 28.8 mm to (10.2, 14.4), turned to 90 degrees
- moved C2 28.0 mm to (14.6, 20.3)
- moved R8 26.3 mm to (40.6, 26.0)
- moved IC1 26.2 mm to (22.9, 19.7)
- moved IC10 25.6 mm to (22.9, 26.7)
- moved C1 25.0 mm to (30.5, 18.4)
- moved D4 24.3 mm to (10.2, 20.1), turned to 90 degrees
- moved D1 18.5 mm to (21.0, 9.32), turned to 90 degrees
- moved R27 17.1 mm to (38.7, 13.3)
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Connections:
- net TA15 renamed TA15_POT_2
- net VIN/2 renamed VCC/2
- removed net CV_IN: D3.A, D4.C, J_PANEL.3, R19.1
- removed net CV_IN2: D1.A, D2.C, J_PANEL.1, R1.1
- removed net CV_OUT: J_PANEL.7, R3.1, R4.1
- removed net CV_OUT2: J_PANEL.5, R6.1, R7.1
- removed net N$8: D5.C, OK1.2, R35.1
- removed net TA14: J1.16, R19.2
- removed net TRIG_IN1: J_PANEL.10, R29.1
- removed net TRIG_IN2: J_PANEL.8, R8.1
- removed net TRIG_OUT1: J_PANEL.6, R38.1
- removed net TRIG_OUT2: J_PANEL.4, R43.1
- removed net VIN: R23.2
- new net CV_IN_1: JP3.8, JP3.9
- new net CV_IN_2: D1.A, D2.C, D3.A, D4.C, JP3.7, R1.1, R19.1
- new net CV_OUT_1: JP3.10, JP3.11, R3.1, R4.1
- new net CV_OUT_2: JP3.6, R6.1, R7.1
- new net TA14_POT_1: J1.16, JP5_POTS.2, R19.2
- new net TA_15_POT_2: JP5_POTS.5
- new net TRIG_IN_1: JP3.5, R29.1
- new net TRIG_IN_2: JP3.3, R8.1
- new net TRIG_OUT_1: JP3.4, R38.1
- new net TRIG_OUT_2: JP3.1, JP3.2, R43.1
- net +3V3: no longer OK1.8, R37.2, R39.2
- net GND: now also JP3.19, JP3.20, JP3.21, JP3.22, JP3.23, JP3.24, JP3.MP1, JP3.MP2, JP5_POTS.3, JP5_POTS.6, JPWR.3, JPWR.4, JPWR.5, JPWR.6, JPWR.7, JPWR.8; no longer J_PANEL.2, OK1.5
- net MIDI_RX: no longer OK1.6, R37.1
- net MIDI_RX_PIN4: now also JP1_MIDI.1, JP3.12, JP3.13; no longer J_PANEL.14, R35.2
- net MIDI_RX_PIN5: now also JP1_MIDI.2, JP3.14; no longer D5.A, J_PANEL.12, OK1.3
- net MIDI_TX: no longer R40.2
- net MIDI_TX_PIN4: now also JP1_MIDI.3, JP3.15; no longer J_PANEL.11, R39.1
- net MIDI_TX_PIN5: now also JP1_MIDI.4, JP3.16, JP3.17; no longer J_PANEL.9, R40.1
- net VCC: now also JP5_POTS.1, JP5_POTS.4, JPWR.11, JPWR.12, R23.2
