File: hardware/ubuntu-v2.1/circuits/TriggersCV_Circuitry.sch (EAGLE design)
At the start: 39 parts, among them IC1 TL072D, IC10 74AHCT1G125DBV, IC11 74AHCT1G125DBV, J1 MOLEX_78127-1408MOLEX_78127-1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, Q1 MMBT3904, Q6 MMBT3904

Commit message: Add files via upload
Parts:
- removed D5: 250mA/100V, SparkFun-DiscreteSemi:DIODE-BAS16J
- removed J_PANEL: 6p-2.54, Molex - 54548-1671:MOLEX_54548-1671MOLEX_54548-1671_0_0
- removed OK1: OG-OPTOCOUPLERS_6N137SMT, TriggersCV_Circuitry:OG-OPTOCOUPLERS_6N137SMT
- removed R35: 220, resistor:R-EU_R0603
- removed R37: 10k, resistor:R-EU_R0603
- removed R39, R40: 51, resistor:R-EU_R0603
- added JP1_MIDI: (no value), pinhead:PINHD-1X4
- added JP3: MOLEX_51281-2494MOLEX_51281-2494_0_0, Molex - 51281-2494:MOLEX_51281-2494MOLEX_51281-2494_0_0
- added JP5_POTS: PINHD-1X6, audio amplifier example:PINHD-1X6
- added JPWR: POWER, eurorack:POWER
- D1, D2, D3, D4, D6, D7: device SparkFun-DiscreteSemi:DIODE-BAS16J -> My_Diodes2:SPARKFUN-DISCRETESEMI_DIODE-BAS16J
- JP4: value MOLEX_54548-1671MOLEX_54548-1671_0_0 -> MOLEX_51281-2494MOLEX_51281-2494_0_0; device Molex - 54548-1671:MOLEX_54548-1671MOLEX_54548-1671_0_0 -> Molex - 51281-2494:MOLEX_51281-2494MOLEX_51281-2494_0_0
Connections:
- net TA15 renamed TA15_POT_2
- net VIN/2 renamed VCC/2
- removed net CV_IN: D3.A, D4.C, J_PANEL.3, R19.1
- removed net CV_IN2: D1.A, D2.C, J_PANEL.1, R1.1
- removed net CV_OUT: J_PANEL.7, R3.1, R4.1
- removed net CV_OUT2: J_PANEL.5, R6.1, R7.1
- removed net N$8: D5.C, OK1.A, R35.1
- removed net TA14: J1.16, R19.2
- removed net TRIG_IN1: J_PANEL.10, R29.1
- removed net TRIG_IN2: J_PANEL.8, R8.1
- removed net TRIG_OUT1: J_PANEL.6, R38.1
- removed net TRIG_OUT2: J_PANEL.4, R43.1
- removed net VIN: R23.2
- new net CV_IN_1: JP3.8, JP3.9
- new net CV_IN_2: D1.A, D2.C, D3.A, D4.C, JP3.7, R1.1, R19.1
- new net CV_OUT_1: JP3.10, JP3.11, R3.1, R4.1
- new net CV_OUT_2: JP3.6, R6.1, R7.1
- new net TA14_POT_1: J1.16, JP5_POTS.2, R19.2
- new net TA_15_POT_2: JP5_POTS.5
- new net TRIG_IN_1: JP3.5, R29.1
- new net TRIG_IN_2: JP3.3, R8.1
- new net TRIG_OUT_1: JP3.4, R38.1
- new net TRIG_OUT_2: JP3.1, JP3.2, R43.1
- net +3V3: no longer OK1.VCC, R37.2, R39.2
- net GND: now also JP3.19, JP3.20, JP3.21, JP3.22, JP3.23, JP3.24, JP3.MP1, JP3.MP2, JP5_POTS.3, JP5_POTS.6, JPWR.GND; no longer J_PANEL.2, OK1.GND
- net MIDI_RX: no longer OK1.VO, R37.1
- net MIDI_RX_PIN4: now also JP1_MIDI.1, JP3.12, JP3.13; no longer J_PANEL.14, R35.2
- net MIDI_RX_PIN5: now also JP1_MIDI.2, JP3.14; no longer D5.A, J_PANEL.12, OK1.C
- net MIDI_TX: no longer R40.2
- net MIDI_TX_PIN4: now also JP1_MIDI.3, JP3.15; no longer J_PANEL.11, R39.1
- net MIDI_TX_PIN5: now also JP1_MIDI.4, JP3.16, JP3.17; no longer J_PANEL.9, R40.1
- net VCC: now also JP5_POTS.1, JP5_POTS.4, JPWR.+5V, R23.2
Other:
- note added: "POWER BUS"
