File: hardware/ubuntu-v2.1/circuits/rotary_breakout.brd (EAGLE design)
At the start: 86.4 x 26.7 mm, 29 parts, among them SW2 SWITCH-ALPS_EC12E_SW, SW3 SWITCH-ALPS_EC12E_SW, SW4 SWITCH-ALPS_EC12E_SW, SW5 SWITCH-ALPS_EC12E_SW

Commit message: Add files via upload
Parts:
- removed JP4: MOLEX_54548-1671MOLEX_54548-1671_0_0, Molex - 54548-1671:MOLEX_54548-1671_0
- added JP1: MOLEX_51281-2494MOLEX_51281-2494_0_0, Molex - 51281-2494:MOLEX_51281-2494_0
- moved C3 1.27 mm to (-4.57, 38.9)
Connections:
- net ENC1_A: now also JP1.2; no longer JP4.2
- net ENC1_B: now also JP1.3; no longer JP4.3
- net ENC1_SW: now also JP1.4; no longer JP4.4
- net ENC2_A: now also JP1.5; no longer JP4.5
- net ENC2_B: now also JP1.6; no longer JP4.6
- net ENC2_SW: now also JP1.7; no longer JP4.7
- net ENC3_A: now also JP1.8; no longer JP4.8
- net ENC3_B: now also JP1.9; no longer JP4.9
- net ENC3_SW: now also JP1.10; no longer JP4.10
- net ENC4_A: now also JP1.11; no longer JP4.11
- net ENC4_B: now also JP1.12; no longer JP4.12
- net ENC4_SW: now also JP1.13; no longer JP4.13
- net GND: now also JP1.1, JP1.14, JP1.MP1, JP1.MP2; no longer JP4.1, JP4.14
Routing:
- net ENC3_B: track 22.0 -> 16.8 mm
- net ENC1_B: track 64.0 -> 59.0 mm
- net ENC2_SW: track 41.5 -> 37.8 mm
- net ENC3_A: track 12.5 -> 14.7 mm
- net ENC2_A: track 29.7 -> 27.6 mm
- net ENC1_SW: track 62.8 -> 64.8 mm, vias 1 -> 0
- net ENC1_A: track 49.8 -> 47.9 mm
- net ENC2_B: track 39.3 -> 37.5 mm, vias 2 -> 0
- net ENC3_SW: track 21.6 -> 19.8 mm
- net ENC4_SW: track 16.6 -> 15.3 mm, vias 0 -> 1
- net ENC4_A: track 27.7 -> 28.8 mm
- net N$8: track 14.2 -> 14.9 mm
- net VCC: track 77.9 -> 77.2 mm
- net ENC4_B: track 20.1 -> 20.2 mm, vias 0 -> 2
