File: hardware/boards/mainboard/Mainboard/Mainboard.sch (KiCad schematic (older format))
At the start: 0 parts

Commit message: minor updates
Changed lines of the file:
@@
 S 1000 1000 500  150
 U 5D772FD9
-F0 "kryon-ver2.1-final_1" 50
+F0 "Teensy" 50
 F1 "kryon-ver2.1-final_1.sch" 50
 $EndSheet
@@
 S 3000 1000 500  150
 U 5D772FF8
-F0 "kryon-ver2.1-final_2" 50
+F0 "Power and bypass caps" 50
 F1 "kryon-ver2.1-final_2.sch" 50
 $EndSheet
@@
 S 5000 1000 500  150
 U 5D7730F8
-F0 "kryon-ver2.1-final_3" 50
+F0 "daughter board connectors" 50
 F1 "kryon-ver2.1-final_3.sch" 50
 $EndSheet
