File: hardware/boards/mainboard/Mainboard/codec.sch (KiCad schematic (older format))
At the start: 22 parts, among them U1 CS42448

Commit message: minor updates
Connections:
- wire segments 172 -> 168
Changed lines of the file:
@@
 	6000 2100 6000 1900
 Connection ~ 5900 1900
-Text GLabel 5200 1900 2    70   BiDi ~ 0
+Text GLabel 5200 1900 0    70   BiDi ~ 0
 3V3
 Connection ~ 6200 1900
@@
 	4150 150  4750 150
 Connection ~ 4150 150
-Text GLabel 3550 150  2    70   BiDi ~ 0
+Text GLabel 3550 150  0    70   BiDi ~ 0
 3V3
 Wire Wire Line
@@
 Wire Wire Line
 	12200 3200 12650 3200
-Text Label 12425 3200 0    70   ~ 0
-AGND
-Wire Wire Line
-	10800 3800 11350 3800
-Text Label 11350 3800 0    70   ~ 0
-AGND
-Wire Wire Line
-	10800 4800 11350 4800
-Text Label 11075 4800 0    70   ~ 0
+Text Label 11600 2400 0    70   ~ 0
+AGND
+Text Label 11450 3750 0    70   ~ 0
+AGND
+Text Label 11350 4750 0    70   ~ 0
 AGND
 Wire Wire Line
@@
 AGND
 Connection ~ 7350 7500
-Wire Wire Line
-	2050 2350 1450 2350
 Text Label 1450 2350 0    70   ~ 0
 AGND
-Wire Wire Line
-	2500 4050 1950 4050
 Text Label 1950 4050 0    70   ~ 0
 AGND
@@
 Text Label 700  2100 0    70   ~ 0
 AGND
-Wire Wire Line
-	300  1250 700  2100
 $Sheet
 S 1750 1750 1100 700
@@
 	12200 4750 12200 3750
 Connection ~ 12200 3750
+Wire Wire Line
+	1950 4050 2550 4050
 $EndSCHEMATC
