File: hardware/boards/mainboard/Mainboard/codec.sch (KiCad schematic (older format))
At the start: 22 parts, among them U1 CS42448

Commit message: footprints
Parts:
- C15, C21, C23, C25: footprint Mainboard:C0805K -> Capacitors_SMD:C_0805_HandSoldering
- C16, C17, C18, C19, C20, C24, C26: footprint Mainboard:C0805 -> Capacitors_SMD:C_0805_HandSoldering
- C22: footprint Mainboard:C1206 -> Capacitors_SMD:C_0805_HandSoldering
- FB1: footprint Mainboard:MURATA_BLM21PG221SN1D_1 -> Mainboard:C0805
Changed lines of the file:
@@
 F 0 "C21" H 8100 7445 59  0000 L BNN
 F 1 "0.1u" H 8070 6985 59  0000 L BNN
-F 2 "Mainboard:C0805K" H 8200 7300 50  0001 C CNN
+F 2 "Capacitors_SMD:C_0805_HandSoldering" H 8200 7300 50  0001 C CNN
 F 3 "" H 8200 7300 50  0001 C CNN
 	1    8200 7300
@@
 F 0 "C23" H 9000 7445 59  0000 L BNN
 F 1 "0.1u" H 8970 6985 59  0000 L BNN
-F 2 "Mainboard:C0805K" H 9100 7300 50  0001 C CNN
+F 2 "Capacitors_SMD:C_0805_HandSoldering" H 9100 7300 50  0001 C CNN
 F 3 "" H 9100 7300 50  0001 C CNN
 	1    9100 7300
@@
 F 0 "C25" H 9900 7445 59  0000 L BNN
 F 1 "0.1u" H 9870 6985 59  0000 L BNN
-F 2 "Mainboard:C0805K" H 10000 7300 50  0001 C CNN
+F 2 "Capacitors_SMD:C_0805_HandSoldering" H 10000 7300 50  0001 C CNN
 F 3 "" H 10000 7300 50  0001 C CNN
 	1    10000 7300
@@
 F 0 "C22" H 8550 7250 42  0000 L BNN
 F 1 "100uf" H 8550 7100 42  0000 L BNN
-F 2 "Mainboard:C1206" H 8700 7200 50  0001 C CNN
+F 2 "Capacitors_SMD:C_0805_HandSoldering" H 8700 7200 50  0001 C CNN
 F 3 "" H 8700 7200 50  0001 C CNN
 	1    8700 7200
@@
 F 0 "C26" H 10550 7250 42  0000 L BNN
 F 1 "4.7uf" H 10550 7100 42  0000 L BNN
-F 2 "Mainboard:C0805" H 10700 7200 50  0001 C CNN
+F 2 "Capacitors_SMD:C_0805_HandSoldering" H 10700 7200 50  0001 C CNN
 F 3 "" H 10700 7200 50  0001 C CNN
 	1    10700 7200
@@
 F 0 "C24" H 9450 7250 42  0000 L BNN
 F 1 "22uf" H 9450 7100 42  0000 L BNN
-F 2 "Mainboard:C0805" H 9600 7200 50  0001 C CNN
+F 2 "Capacitors_SMD:C_0805_HandSoldering" H 9600 7200 50  0001 C CNN
 F 3 "" H 9600 7200 50  0001 C CNN
 	1    9600 7200
@@
 F 0 "FB1" H 7600 1680 85  0000 L TNN
 F 1 "MURATA_BLM21PG221SN1DMURATA_BLM21PG221SN1D_0_1" H 7550 1550 50  0001 C CNN
-F 2 "Mainboard:MURATA_BLM21PG221SN1D_1" H 7550 1550 50  0001 C CNN
+F 2 "Mainboard:C0805" H 7550 1550 50  0001 C CNN
 F 3 "" H 7550 1550 50  0001 C CNN
 	1    7550 1550
@@
 F 0 "C15" H 4210 365 59  0000 L BNN
 F 1 "0.1uF" H 4210 165 59  0000 L BNN
-F 2 "Mainboard:C0805K" H 4150 350 50  0001 C CNN
+F 2 "Capacitors_SMD:C_0805_HandSoldering" H 4150 350 50  0001 C CNN
 F 3 "" H 4150 350 50  0001 C CNN
 	1    4150 350
@@
 F 0 "C16" H 6950 2000 42  0000 L BNN
 F 1 "10uf" H 6950 1850 42  0000 L BNN
-F 2 "Mainboard:C0805" H 7100 1950 50  0001 C CNN
+F 2 "Capacitors_SMD:C_0805_HandSoldering" H 7100 1950 50  0001 C CNN
 F 3 "" H 7100 1950 50  0001 C CNN
 	1    7100 1950
@@
 F 0 "C17" H 7250 2000 42  0000 L BNN
 F 1 "100nf" H 7250 1850 42  0000 L BNN
-F 2 "Mainboard:C0805" H 7400 1950 50  0001 C CNN
+F 2 "Capacitors_SMD:C_0805_HandSoldering" H 7400 1950 50  0001 C CNN
 F 3 "" H 7400 1950 50  0001 C CNN
 	1    7400 1950
@@
 F 0 "C18" H 7500 2000 42  0000 L BNN
 F 1 "100nf" H 7500 1850 42  0000 L BNN
-F 2 "Mainboard:C0805" H 7650 1950 50  0001 C CNN
+F 2 "Capacitors_SMD:C_0805_HandSoldering" H 7650 1950 50  0001 C CNN
 F 3 "" H 7650 1950 50  0001 C CNN
 	1    7650 1950
@@
 F 0 "C19" H 7750 2000 42  0000 L BNN
 F 1 "10nf" H 7750 1850 42  0000 L BNN
-F 2 "Mainboard:C0805" H 7900 1950 50  0001 C CNN
+F 2 "Capacitors_SMD:C_0805_HandSoldering" H 7900 1950 50  0001 C CNN
 F 3 "" H 7900 1950 50  0001 C CNN
 	1    7900 1950
@@
 F 0 "C20" H 8000 2000 42  0000 L BNN
 F 1 "10nf" H 8000 1850 42  0000 L BNN
-F 2 "Mainboard:C0805" H 8150 1950 50  0001 C CNN
+F 2 "Capacitors_SMD:C_0805_HandSoldering" H 8150 1950 50  0001 C CNN
 F 3 "" H 8150 1950 50  0001 C CNN
 	1    8150 1950
