File: hardware/boards/mainboard/Mainboard/Audio-out.sch (KiCad schematic (older format))
At the start: 9 parts

Commit message: footprints
Parts:
- C39, C40, C41, C42: footprint Audio-out:C0805 -> Capacitors_SMD:C_0805_HandSoldering
- J_OUT1: footprint Audio-out:ACJS-MV5 -> Mainboard:ACJS-MV5
- R17, R18, R19, R20: footprint Audio-out:R0805 -> Resistors_SMD:R_0805_HandSoldering
Changed lines of the file:
@@
 $Descr A4 11693 8268
 encoding utf-8
-Sheet 9 13
+Sheet 10 13
 Title ""
 Date ""
@@
 AR Path="/5D773153/5D8B335A/E0EA0F9E" Ref="R25"  Part="1"
 AR Path="/5D773153/5D8BB03A/E0EA0F9E" Ref="R29"  Part="1"
-F 0 "R29" H 4150 3959 59  0000 L BNN
+F 0 "R21" H 4150 3959 59  0000 L BNN
 F 1 "10K" H 4150 3770 59  0000 L BNN
-F 2 "Audio-out:R0805" H 4300 3900 50  0001 C CNN
+F 2 "Resistors_SMD:R_0805_HandSoldering" H 4300 3900 50  0001 C CNN
 F 3 "" H 4300 3900 50  0001 C CNN
 	1    4300 3900
@@
 AR Path="/5D773153/5D8B335A/4B69501E" Ref="R27"  Part="1"
 AR Path="/5D773153/5D8BB03A/4B69501E" Ref="R31"  Part="1"
-F 0 "R31" H 4500 3759 59  0000 L BNN
+F 0 "R23" H 4500 3759 59  0000 L BNN
 F 1 "560" H 4500 3570 59  0000 L BNN
-F 2 "Audio-out:R0805" H 4650 3700 50  0001 C CNN
+F 2 "Resistors_SMD:R_0805_HandSoldering" H 4650 3700 50  0001 C CNN
 F 3 "" H 4650 3700 50  0001 C CNN
 	1    4650 3700
@@
 AR Path="/5D773153/5D8B335A/D85E66C8" Ref="R26"  Part="1"
 AR Path="/5D773153/5D8BB03A/D85E66C8" Ref="R30"  Part="1"
-F 0 "R30" H 4150 4609 59  0000 L BNN
+F 0 "R22" H 4150 4609 59  0000 L BNN
 F 1 "10K" H 4150 4420 59  0000 L BNN
-F 2 "Audio-out:R0805" H 4300 4550 50  0001 C CNN
+F 2 "Resistors_SMD:R_0805_HandSoldering" H 4300 4550 50  0001 C CNN
 F 3 "" H 4300 4550 50  0001 C CNN
 	1    4300 4550
@@
 AR Path="/5D773153/5D8B335A/EDD241BD" Ref="R28"  Part="1"
 AR Path="/5D773153/5D8BB03A/EDD241BD" Ref="R32"  Part="1"
-F 0 "R32" H 4500 4409 59  0000 L BNN
+F 0 "R24" H 4500 4409 59  0000 L BNN
 F 1 "560" H 4500 4220 59  0000 L BNN
-F 2 "Audio-out:R0805" H 4650 4350 50  0001 C CNN
+F 2 "Resistors_SMD:R_0805_HandSoldering" H 4650 4350 50  0001 C CNN
 F 3 "" H 4650 4350 50  0001 C CNN
 	1    4650 4350
@@
 AR Path="/5D773153/5D8B335A/6F308249" Ref="J_OUT3"  Part="1"
 AR Path="/5D773153/5D8BB03A/6F308249" Ref="J_OUT4"  Part="1"
-F 0 "J_OUT4" H 7300 3500 50  0001 C CNN
+F 0 "J_OUT2" H 7300 3500 50  0001 C CNN
 F 1 "ACJS-MV-5" H 7300 3500 50  0001 C CNN
-F 2 "Audio-out:ACJS-MV5" H 7300 3500 50  0001 C CNN
+F 2 "Mainboard:ACJS-MV5" H 7300 3500 50  0001 C CNN
 F 3 "" H 7300 3500 50  0001 C CNN
 	1    7300 3500
@@
 AR Path="/5D773153/5D8B335A/D3DD9420" Ref="C48"  Part="1"
 AR Path="/5D773153/5D8BB03A/D3DD9420" Ref="C52"  Part="1"
-F 0 "C52" H 4010 3715 59  0000 L BNN
+F 0 "C44" H 4010 3715 59  0000 L BNN
 F 1 "4.7uF" H 4010 3515 59  0000 L BNN
-F 2 "Audio-out:C0805" H 3950 3700 50  0001 C CNN
+F 2 "Capacitors_SMD:C_0805_HandSoldering" H 3950 3700 50  0001 C CNN
 F 3 "" H 3950 3700 50  0001 C CNN
 	1    3950 3700
@@
 AR Path="/5D773153/5D8B335A/BAA6A02E" Ref="C47"  Part="1"
 AR Path="/5D773153/5D8BB03A/BAA6A02E" Ref="C51"  Part="1"
-F 0 "C51" H 3910 4365 59  0000 L BNN
+F 0 "C43" H 3910 4365 59  0000 L BNN
 F 1 "4.7uF" H 3910 4165 59  0000 L BNN
-F 2 "Audio-out:C0805" H 3850 4350 50  0001 C CNN
+F 2 "Capacitors_SMD:C_0805_HandSoldering" H 3850 4350 50  0001 C CNN
 F 3 "" H 3850 4350 50  0001 C CNN
 	1    3850 4350
@@
 AR Path="/5D773153/5D8B335A/57CFC50E" Ref="C50"  Part="1"
 AR Path="/5D773153/5D8BB03A/57CFC50E" Ref="C54"  Part="1"
-F 0 "C54" H 5760 4565 59  0000 L BNN
+F 0 "C46" H 5760 4565 59  0000 L BNN
 F 1 "2700pF" H 5760 4365 59  0000 L BNN
-F 2 "Audio-out:C0805" H 5700 4550 50  0001 C CNN
+F 2 "Capacitors_SMD:C_0805_HandSoldering" H 5700 4550 50  0001 C CNN
 F 3 "" H 5700 4550 50  0001 C CNN
 	1    5700 4550
@@
 AR Path="/5D773153/5D8B335A/D3171833" Ref="C49"  Part="1"
 AR Path="/5D773153/5D8BB03A/D3171833" Ref="C53"  Part="1"
-F 0 "C53" H 5660 3815 59  0000 L BNN
+F 0 "C45" H 5660 3815 59  0000 L BNN
 F 1 "2700pF" H 5660 3615 59  0000 L BNN
-F 2 "Audio-out:C0805" H 5600 3800 50  0001 C CNN
+F 2 "Capacitors_SMD:C_0805_HandSoldering" H 5600 3800 50  0001 C CNN
 F 3 "" H 5600 3800 50  0001 C CNN
 	1    5600 3800
