File: hardware/boards/mainboard/Mainboard/Midi.sch (KiCad schematic (older format))
At the start: 6 parts

Commit message: footprints
Parts:
- D3: footprint Mainboard:SMA-DIODE -> Diodes_SMD:D_SMA_Handsoldering
- R33, R34, R35, R36: footprint Mainboard:R0805 -> Resistors_SMD:R_0805_HandSoldering
Changed lines of the file:
@@
 $Descr A4 11693 8268
 encoding utf-8
-Sheet 1 13
+Sheet 13 13
 Title ""
 Date ""
@@
 F 0 "D3" H 6100 3519 59  0000 L BNN
 F 1 "DIODESMA" H 6100 3409 59  0000 L BNN
-F 2 "Mainboard:SMA-DIODE" H 6000 3500 50  0001 C CNN
+F 2 "Diodes_SMD:D_SMA_Handsoldering" H 6000 3500 50  0001 C CNN
 F 3 "" H 6000 3500 50  0001 C CNN
 	1    6000 3500
@@
 F 0 "R34" H 5550 3359 59  0000 L BNN
 F 1 "220" H 5550 3170 59  0000 L BNN
-F 2 "Mainboard:R0805" H 5700 3300 50  0001 C CNN
+F 2 "Resistors_SMD:R_0805_HandSoldering" H 5700 3300 50  0001 C CNN
 F 3 "" H 5700 3300 50  0001 C CNN
 	1    5700 3300
@@
 F 0 "R36" H 7150 3259 59  0000 L BNN
 F 1 "220" H 7150 3070 59  0000 L BNN
-F 2 "Mainboard:R0805" H 7300 3200 50  0001 C CNN
+F 2 "Resistors_SMD:R_0805_HandSoldering" H 7300 3200 50  0001 C CNN
 F 3 "" H 7300 3200 50  0001 C CNN
 	1    7300 3200
@@
 F 0 "R33" H 5350 4959 59  0000 L BNN
 F 1 "220" H 5350 4770 59  0000 L BNN
-F 2 "Mainboard:R0805" H 5500 4900 50  0001 C CNN
+F 2 "Resistors_SMD:R_0805_HandSoldering" H 5500 4900 50  0001 C CNN
 F 3 "" H 5500 4900 50  0001 C CNN
 	1    5500 4900
@@
 F 0 "R35" H 5650 5559 59  0000 L BNN
 F 1 "220" H 5650 5370 59  0000 L BNN
-F 2 "Mainboard:R0805" H 5800 5500 50  0001 C CNN
+F 2 "Resistors_SMD:R_0805_HandSoldering" H 5800 5500 50  0001 C CNN
 F 3 "" H 5800 5500 50  0001 C CNN
 	1    5800 5500
