File: hardware/boards/mainboard/Mainboard/kryon-ver2.1-final_3.sch (KiCad schematic (older format))
At the start: 6 parts, among them J1 MOLEX_52892-3033MOLEX_52892-3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, J2 MOLEX_52892-3033MOLEX_52892-3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

Commit message: footprints
Parts:
- D1: footprint Mainboard:SMA-DIODE -> Diodes_SMD:D_SMA_Handsoldering; symbol Mainboard-eagle-import:DIODESMA -> Device:D
- D2: footprint Mainboard:SMA-DIODE -> Diodes_SMD:D_SMA_Handsoldering
Other:
- moved on the sheet: D2
Changed lines of the file:
@@
 $EndComp
 $Comp
-L Mainboard-eagle-import:DIODESMA D1
+L Device:D D1
 U 1 1 74A9BC2C
-P 3100 5800
-F 0 "D1" H 3200 5819 59  0000 L BNN
-F 1 "DIODESMA" H 3200 5709 59  0000 L BNN
-F 2 "Mainboard:SMA-DIODE" H 3100 5800 50  0001 C CNN
-F 3 "" H 3100 5800 50  0001 C CNN
-	1    3100 5800
+P 3650 5850
+F 0 "D1" H 3750 5869 59  0000 L BNN
+F 1 "DIODESMA" H 3750 5759 59  0000 L BNN
+F 2 "Diodes_SMD:D_SMA_Handsoldering" H 3650 5850 50  0001 C CNN
+F 3 "" H 3650 5850 50  0001 C CNN
+	1    3650 5850
 	0    -1   -1   0
 $EndComp
@@
 L Mainboard-eagle-import:DIODESMA D2
 U 1 1 9E0BEA3A
-P 3100 6600
-F 0 "D2" H 3200 6619 59  0000 L BNN
-F 1 "DIODESMA" H 3200 6509 59  0000 L BNN
-F 2 "Mainboard:SMA-DIODE" H 3100 6600 50  0001 C CNN
-F 3 "" H 3100 6600 50  0001 C CNN
-	1    3100 6600
+P 3750 6600
+F 0 "D2" H 3850 6619 59  0000 L BNN
+F 1 "DIODESMA" H 3850 6509 59  0000 L BNN
+F 2 "Diodes_SMD:D_SMA_Handsoldering" H 3750 6600 50  0001 C CNN
+F 3 "" H 3750 6600 50  0001 C CNN
+	1    3750 6600
 	0    -1   -1   0
 $EndComp
