File: hardware/boards/topbreakout/io_breakout-ver2.1_6.sch (KiCad schematic (older format))
At the start: 7 parts, among them U3 ANALOG_DEVICES_AD5754BREZANAL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, U5 MICROCHIP_MCP1700T-2502E-TTMI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

Commit message: cleanup
Changed lines of the file:
@@
 Wire Wire Line
 	4500 4900 3800 4900
-Text Label 3800 4900 2    70   ~ 0
-AVDD
 Wire Wire Line
 	5900 4900 6600 4900
-Text Label 6600 4900 0    70   ~ 0
-AVSS
 Wire Wire Line
 	5900 5500 6300 5500
@@
 Wire Wire Line
 	2200 4300 2200 4000
-Text GLabel 1600 4000 2    70   BiDi ~ 0
+Text GLabel 1600 4000 0    70   BiDi ~ 0
 3V3
 Connection ~ 2200 4000
@@
 	1    0    0    -1
 $EndComp
+Text GLabel 3800 4900 0    70   Input ~ 0
+AVDD
+Text GLabel 6600 4900 2    70   Input ~ 0
+AVSS
 $EndSCHEMATC

Commit message: routed, ERC checks success
Parts:
- C10, C11: footprint topbreakout:C1206 -> Capacitors_SMD:C_0805
Changed lines of the file:
@@
 F 0 "C10" V 2509 2349 59  0000 C CNN
 F 1 "0.1uF" V 2690 2349 59  0000 C CNN
-F 2 "topbreakout:C1206" H 2600 2300 50  0001 C CNN
+F 2 "Capacitors_SMD:C_0805" H 2600 2300 50  0001 C CNN
 F 3 "" H 2600 2300 50  0001 C CNN
 	1    2600 2300
@@
 F 0 "C11" V 3009 2349 59  0000 C CNN
 F 1 "0.1uF" V 3190 2349 59  0000 C CNN
-F 2 "topbreakout:C1206" H 3100 2300 50  0001 C CNN
+F 2 "Capacitors_SMD:C_0805" H 3100 2300 50  0001 C CNN
 F 3 "" H 3100 2300 50  0001 C CNN
 	1    3100 2300

Commit message: revision 1.4 changes
Parts:
- C6, C9: footprint topbreakout:C1206 -> Capacitor_SMD:C_0805_2012Metric
Connections:
- net 3V3 renamed +3V3
Changed lines of the file:
@@
-EESchema Schematic File Version 4
-LIBS:TopBreakout-cache
+EESchema Schematic File Version 5
 EELAYER 30 0
 EELAYER END
@@
 Comment3 ""
 Comment4 ""
+Comment5 ""
+Comment6 ""
+Comment7 ""
+Comment8 ""
+Comment9 ""
 $EndDescr
 Wire Wire Line
@@
 	4500 5500 3700 5500
 Text GLabel 3700 5500 0    70   BiDi ~ 0
-3V3
++3V3
 Wire Wire Line
 	1600 4000 2200 4000
@@
 	2200 4300 2200 4000
 Text GLabel 1600 4000 0    70   BiDi ~ 0
-3V3
++3V3
 Connection ~ 2200 4000
 Wire Wire Line
@@
 F 0 "C6" V 7709 2349 59  0000 C CNN
 F 1 "0.1uF" V 7890 2349 59  0000 C CNN
-F 2 "topbreakout:C1206" H 7800 2300 50  0001 C CNN
+F 2 "Capacitor_SMD:C_0805_2012Metric" H 7800 2300 50  0001 C CNN
 F 3 "" H 7800 2300 50  0001 C CNN
 	1    7800 2300
@@
 F 0 "C9" V 8209 2349 59  0000 C CNN
 F 1 "0.1uF" V 8390 2349 59  0000 C CNN
-F 2 "topbreakout:C1206" H 8300 2300 50  0001 C CNN
+F 2 "Capacitor_SMD:C_0805_2012Metric" H 8300 2300 50  0001 C CNN
 F 3 "" H 8300 2300 50  0001 C CNN
 	1    8300 2300

Commit message: TopBreakout: v1.6
Parts:
- added TP10: TEST-POINT3X5, topbreakout:PAD.03X.05, symbol TopBreakout-eagle-import:TEST-POINT3X5
Connections:
- net DA_SYNC: now also TP10.P$1 (1)
- net GND: no longer C10.2, C11.2, C6.2, C9.2, U5.1 (GND)
- new net: C6.2, C9.2, U5.1 (GND)
- new net: C10.2, C11.2
- no-connect marks 0 -> 5
Changed lines of the file:
@@
 Connection ~ 7800 2500
 Connection ~ 5800 2400
-Text GLabel 8300 2500 0    10   BiDi ~ 0
-GND
 Wire Wire Line
 	2600 2500 3000 2500
@@
 	3000 2700 3000 2500
 Connection ~ 3000 2500
-Text GLabel 2600 2500 0    10   BiDi ~ 0
-GND
 Wire Wire Line
 	4500 5500 3700 5500
@@
 +3V3
 Wire Wire Line
-	1600 4000 2200 4000
-Wire Wire Line
-	2200 4000 2300 4000
-Wire Wire Line
 	2300 4400 4500 4400
 Wire Wire Line
-	2300 4000 2300 4400
-Wire Wire Line
-	4500 4300 2200 4300
-Wire Wire Line
-	2200 4300 2200 4000
+	2300 4000 2300 4300
+Wire Wire Line
+	4500 4300 2300 4300
 Text GLabel 1600 4000 0    70   BiDi ~ 0
 +3V3
-Connection ~ 2200 4000
-Wire Wire Line
-	5900 3700 9500 3700
-Text GLabel 9500 3700 2    70   BiDi ~ 0
+Wire Wire Line
+	5900 3700 6650 3700
+Text GLabel 6650 3700 2    70   BiDi ~ 0
 DA_V1
-Wire Wire Line
-	7200 3900 9000 3900
-Wire Wire Line
-	5900 3800 7200 3800
-Wire Wire Line
-	7200 3800 7200 3900
-Text GLabel 9000 3900 2    70   BiDi ~ 0
-DA_V2
-Wire Wire Line
-	7100 4100 7200 4100
-Wire Wire Line
-	5900 3900 7100 3900
-Wire Wire Line
-	7100 3900 7100 4100
-Text GLabel 7150 4100 2    70   BiDi ~ 0
+Text GLabel 6650 3900 2    70   BiDi ~ 0
 DA_V3
-Wire Wire Line
-	7000 4300 7600 4300
-Wire Wire Line
-	5900 4000 7000 4000
-Wire Wire Line
-	7000 4000 7000 4300
-Text GLabel 7600 4300 2    70   BiDi ~ 0
+Text GLabel 7050 4000 2    70   BiDi ~ 0
 DA_V4
 Wire Wire Line
@@
 Wire Wire Line
 	3100 2200 2600 2200
-Text GLabel 2600 2200 0    70   BiDi ~ 0
+Text GLabel 2150 2200 0    70   BiDi ~ 0
 VIN
 Connection ~ 3100 2200
@@
 AR Path="/5D7F4465/BC758AA8" Ref="TP3"  Part="1"
 F 0 "TP3" H 6000 4300 70  0001 L BNN
-F 1 "TEST-POINT3X5" V 6000 4200 70  0000 R TNN
+F 1 "TEST-POINT3X5" V 6000 4200 70  0001 R TNN
 F 2 "topbreakout:PAD.03X.05" H 6100 4200 50  0001 C CNN
 F 3 "" H 6100 4200 50  0001 C CNN
@@
 AR Path="/FDFA29AC" Ref="C6"  Part="1"
 AR Path="/5D7F4465/FDFA29AC" Ref="C6"  Part="1"
-F 0 "C6" V 7709 2349 59  0000 C CNN
-F 1 "0.1uF" V 7890 2349 59  0000 C CNN
+F 0 "C6" V 7650 2250 59  0000 C CNN
+F 1 "0.1uF" V 7950 2250 59  0000 C CNN
 F 2 "Capacitor_SMD:C_0805_2012Metric" H 7800 2300 50  0001 C CNN
 F 3 "" H 7800 2300 50  0001 C CNN
@@
 AR Path="/5BE03534" Ref="C9"  Part="1"
 AR Path="/5D7F4465/5BE03534" Ref="C9"  Part="1"
-F 0 "C9" V 8209 2349 59  0000 C CNN
-F 1 "0.1uF" V 8390 2349 59  0000 C CNN
+F 0 "C9" V 8150 2250 59  0000 C CNN
+F 1 "0.1uF" V 8450 2250 59  0000 C CNN
 F 2 "Capacitor_SMD:C_0805_2012Metric" H 8300 2300 50  0001 C CNN
 F 3 "" H 8300 2300 50  0001 C CNN
@@
 AR Path="/E5C7F153" Ref="C10"  Part="1"
 AR Path="/5D7F4465/E5C7F153" Ref="C10"  Part="1"
-F 0 "C10" V 2509 2349 59  0000 C CNN
-F 1 "0.1uF" V 2690 2349 59  0000 C CNN
+F 0 "C10" V 2400 2250 59  0000 C CNN
+F 1 "0.1uF" V 2750 2250 59  0000 C CNN
 F 2 "Capacitors_SMD:C_0805" H 2600 2300 50  0001 C CNN
 F 3 "" H 2600 2300 50  0001 C CNN
@@
 AR Path="/608006B0" Ref="C11"  Part="1"
 AR Path="/5D7F4465/608006B0" Ref="C11"  Part="1"
-F 0 "C11" V 3009 2349 59  0000 C CNN
-F 1 "0.1uF" V 3190 2349 59  0000 C CNN
+F 0 "C11" V 2950 2250 59  0000 C CNN
+F 1 "0.1uF" V 3250 2250 59  0000 C CNN
 F 2 "Capacitors_SMD:C_0805" H 3100 2300 50  0001 C CNN
 F 3 "" H 3100 2300 50  0001 C CNN
@@
 Text GLabel 6600 4900 2    70   Input ~ 0
 AVSS
+NoConn ~ 4500 4700
+NoConn ~ 4500 4600
+NoConn ~ 5900 4600
+NoConn ~ 5900 4700
+NoConn ~ 5900 5000
+Connection ~ 2600 2200
+Wire Wire Line
+	2600 2200 2150 2200
+$Comp
+L TopBreakout-eagle-import:TEST-POINT3X5 TP?
+U 1 1 5E0D7D26
+P 3800 4000
+AR Path="/5E0D7D26" Ref="TP?"  Part="1"
+AR Path="/5D7F4465/5E0D7D26" Ref="TP10"  Part="1"
+F 0 "TP10" H 3700 4100 70  0001 L BNN
+F 1 "TEST-POINT3X5" V 3700 4000 70  0001 R TNN
+F 2 "topbreakout:PAD.03X.05" H 3800 4000 50  0001 C CNN
+F 3 "" H 3800 4000 50  0001 C CNN
+	1    3800 4000
+	0    1    1    0
+$EndComp
+Text GLabel 7050 3800 2    70   BiDi ~ 0
+DA_V2
+Wire Wire Line
+	5900 3800 7050 3800
+Wire Wire Line
+	5900 3900 6650 3900
+Wire Wire Line
+	5900 4000 7050 4000
+Connection ~ 2300 4300
+Wire Wire Line
+	2300 4300 2300 4400
+Wire Wire Line
+	1600 4000 2300 4000
 $EndSCHEMATC

Commit message: topbreakout board: v1.6
Parts:
- added TP?: TEST-POINT3X5, topbreakout:PAD.03X.05, symbol TopBreakout-eagle-import:TEST-POINT3X5
Connections:
- net SPI0_MOSI: now also TP?.P$1 (1)
- net SPI0_MISO: no longer names the net of U3.16 (SDO)
- no-connect marks 5 -> 6
Changed lines of the file:
@@
 DA_SYNC
 Wire Wire Line
-	4500 3800 3800 3800
-Text GLabel 3800 3800 0    70   BiDi ~ 0
+	4500 3800 3000 3800
+Text GLabel 3000 3800 0    70   BiDi ~ 0
 SPI0_MOSI
 Wire Wire Line
@@
 Connection ~ 6200 2200
 Connection ~ 6100 4200
-Wire Wire Line
-	4500 3900 3000 3900
-Text GLabel 3000 3900 0    70   BiDi ~ 0
-SPI0_MISO
 $Comp
 L TopBreakout-eagle-import:ANALOG_DEVICES_AD5754BREZANALOG_DEVICES_AD5754BREZ_0_2 U3
@@
 Wire Wire Line
 	1600 4000 2300 4000
+NoConn ~ 4500 3900
+$Comp
+L TopBreakout-eagle-import:TEST-POINT3X5 TP?
+U 1 1 5E139C99
+P 3000 3800
+AR Path="/5E139C99" Ref="TP?"  Part="1"
+AR Path="/5D7F4465/5E139C99" Ref="TP?"  Part="1"
+F 0 "TP?" H 2900 3900 70  0001 L BNN
+F 1 "TEST-POINT3X5" V 2900 3800 70  0001 R TNN
+F 2 "topbreakout:PAD.03X.05" H 3000 3800 50  0001 C CNN
+F 3 "" H 3000 3800 50  0001 C CNN
+	1    3000 3800
+	0    -1   -1   0
+$EndComp
 $EndSCHEMATC
