File: hardware/boards/topbreakout/io_breakout-ver2.1_6.sch (KiCad schematic (older format))
At the start: 9 parts, among them U3 ANALOG_DEVICES_AD5754BREZANAL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, U5 MICROCHIP_MCP1700T-2502E-TTMI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

Commit message: mainboard v1.7
Parts:
- removed TP10: TEST-POINT3X5, topbreakout:PAD.03X.05, symbol TopBreakout-eagle-import:TEST-POINT3X5
- removed U3: ANALOG_DEVICES_AD5754BREZANALOG_DEVICES_AD5754BRE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, topbreakout:ANALOG_DEVICES_AD5754BREZ_2, symbol TopBreakout-eagle-import:ANALOG_DEVICES_AD5754BREZANALOG_DEVICES_AD5754BREZ_0_2
- added U4: ANALOG_DEVICES_AD5754BREZANALOG_DEVICES_AD5754BRE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, topbreakout:ANALOG_DEVICES_AD5754BREZ_2, symbol TopBreakout-eagle-import:ANALOG_DEVICES_AD5754BREZANALOG_DEVICES_AD5754BREZ_0_2
- renumbered C10 to C28, C11 to C29, C6 to C30, C9 to C31, TP11 to TP2
Connections:
- net +3V3: now also U4.11 (~CLR~), U4.14 (DVCC), U4.5 (~2SCOMP~)
- net AVDD: now also U4.24 (AVDD)
- net AVSS: now also U4.1 (AVSS)
- net DA_SYNC: now also U4.7 (~SYNC~)
- net DA_V1: now also U4.3 (VOUTA)
- net DA_V2: now also U4.4 (VOUTB)
- net DA_V3: now also U4.23 (VOUTC)
- net DA_V4: now also U4.22 (VOUTD)
- net GND: now also U4.15 (GND), U4.18 (1_DAC_GND), U4.19 (2_DAC_GND), U4.20 (1_SIG_GND), U4.21 (2_SIG_GND)
- net SPI0_MOSI: now also U4.9 (SDIN)
- net SPI0_SCK: now also U4.8 (SCLK)
- net VREF: now also U4.17 (REFIN)
Changed lines of the file:
@@
-EESchema Schematic File Version 5
+EESchema Schematic File Version 4
 EELAYER 30 0
 EELAYER END
 $Descr A4 11693 8268
 encoding utf-8
-Sheet 7 8
+Sheet 12 13
 Title ""
 Date ""
@@
 Comment3 ""
 Comment4 ""
-Comment5 ""
-Comment6 ""
-Comment7 ""
-Comment8 ""
-Comment9 ""
 $EndDescr
 Wire Wire Line
@@
 Connection ~ 6100 4200
 $Comp
-L TopBreakout-eagle-import:ANALOG_DEVICES_AD5754BREZANALOG_DEVICES_AD5754BREZ_0_2 U3
-U 1 1 5C95457F
+L TopBreakout-eagle-import:ANALOG_DEVICES_AD5754BREZANALOG_DEVICES_AD5754BREZ_0_2 U?
+U 1 1 5E09D778
 P 4700 3400
-AR Path="/5C95457F" Ref="U3"  Part="1"
-AR Path="/5D7F4465/5C95457F" Ref="U3"  Part="1"
-F 0 "U3" H 4700 3300 85  0000 L TNN
+AR Path="/5E09D778" Ref="U?"  Part="1"
+AR Path="/5D7F4465/5E09D778" Ref="U4"  Part="1"
+F 0 "U4" H 4700 3300 85  0000 L TNN
 F 1 "ANALOG_DEVICES_AD5754BREZANALOG_DEVICES_AD5754BREZ_0_2" H 4700 3400 50  0001 C CNN
 F 2 "topbreakout:ANALOG_DEVICES_AD5754BREZ_2" H 4700 3400 50  0001 C CNN
@@
 $EndComp
 $Comp
-L TopBreakout-eagle-import:TEST-POINT3X5 TP3
+L TopBreakout-eagle-import:TEST-POINT3X5 TP?
 U 1 1 BC758AA8
 P 6100 4200
-AR Path="/BC758AA8" Ref="TP3"  Part="1"
+AR Path="/BC758AA8" Ref="TP?"  Part="1"
 AR Path="/5D7F4465/BC758AA8" Ref="TP3"  Part="1"
 F 0 "TP3" H 6000 4300 70  0001 L BNN
@@
 $EndComp
 $Comp
-L TopBreakout-eagle-import:GND #GND2
+L TopBreakout-eagle-import:GND #GND?
 U 1 1 C92C8F3B
 P 6300 6100
-AR Path="/C92C8F3B" Ref="#GND2"  Part="1"
-AR Path="/5D7F4465/C92C8F3B" Ref="#GND02"  Part="1"
-F 0 "#GND02" H 6300 6100 50  0001 C CNN
+AR Path="/C92C8F3B" Ref="#GND?"  Part="1"
+AR Path="/5D7F4465/C92C8F3B" Ref="#GND032"  Part="1"
+F 0 "#GND032" H 6300 6100 50  0001 C CNN
 F 1 "GND" H 6200 6000 59  0000 L BNN
 F 2 "" H 6300 6100 50  0001 C CNN
@@
 $EndComp
 $Comp
-L TopBreakout-eagle-import:GND #GND4
+L TopBreakout-eagle-import:GND #GND?
 U 1 1 6AE2E73F
 P 2600 5100
-AR Path="/6AE2E73F" Ref="#GND4"  Part="1"
-AR Path="/5D7F4465/6AE2E73F" Ref="#GND04"  Part="1"
-F 0 "#GND04" H 2600 5100 50  0001 C CNN
+AR Path="/6AE2E73F" Ref="#GND?"  Part="1"
+AR Path="/5D7F4465/6AE2E73F" Ref="#GND029"  Part="1"
+F 0 "#GND029" H 2600 5100 50  0001 C CNN
 F 1 "GND" H 2500 5000 59  0000 L BNN
 F 2 "" H 2600 5100 50  0001 C CNN
@@
 $EndComp
 $Comp
-L TopBreakout-eagle-import:MICROCHIP_MCP1700T-2502E-TTMICROCHIP_MCP1700T-2502E-TT_0_0 U5
+L TopBreakout-eagle-import:MICROCHIP_MCP1700T-2502E-TTMICROCHIP_MCP1700T-2502E-TT_0_0 U?
 U 1 1 E98390DC
 P 5000 1900
-AR Path="/E98390DC" Ref="U5"  Part="1"
+AR Path="/E98390DC" Ref="U?"  Part="1"
 AR Path="/5D7F4465/E98390DC" Ref="U5"  Part="1"
 F 0 "U5" H 5000 1800 85  0000 L TNN
@@
 $EndComp
 $Comp
-L TopBreakout-eagle-import:GND #GND5
+L TopBreakout-eagle-import:GND #GND?
 U 1 1 6CC61BFB
 P 5800 2500
-AR Path="/6CC61BFB" Ref="#GND5"  Part="1"
-AR Path="/5D7F4465/6CC61BFB" Ref="#GND05"  Part="1"
-F 0 "#GND05" H 5800 2500 50  0001 C CNN
+AR Path="/6CC61BFB" Ref="#GND?"  Part="1"
+AR Path="/5D7F4465/6CC61BFB" Ref="#GND031"  Part="1"
+F 0 "#GND031" H 5800 2500 50  0001 C CNN
 F 1 "GND" H 5700 2400 59  0000 L BNN
 F 2 "" H 5800 2500 50  0001 C CNN
@@
 $EndComp
 $Comp
-L TopBreakout-eagle-import:C-EUC1206 C6
+L TopBreakout-eagle-import:C-EUC1206 C?
 U 1 1 FDFA29AC
 P 7800 2300
-AR Path="/FDFA29AC" Ref="C6"  Part="1"
-AR Path="/5D7F4465/FDFA29AC" Ref="C6"  Part="1"
-F 0 "C6" V 7650 2250 59  0000 C CNN
+AR Path="/FDFA29AC" Ref="C?"  Part="1"
+AR Path="/5D7F4465/FDFA29AC" Ref="C30"  Part="1"
+F 0 "C30" V 7650 2250 59  0000 C CNN
 F 1 "0.1uF" V 7950 2250 59  0000 C CNN
 F 2 "Capacitor_SMD:C_0805_2012Metric" H 7800 2300 50  0001 C CNN
@@
 $EndComp
 $Comp
-L TopBreakout-eagle-import:C-EUC1206 C9
+L TopBreakout-eagle-import:C-EUC1206 C?
 U 1 1 5BE03534
 P 8300 2300
-AR Path="/5BE03534" Ref="C9"  Part="1"
-AR Path="/5D7F4465/5BE03534" Ref="C9"  Part="1"
-F 0 "C9" V 8150 2250 59  0000 C CNN
+AR Path="/5BE03534" Ref="C?"  Part="1"
+AR Path="/5D7F4465/5BE03534" Ref="C31"  Part="1"
+F 0 "C31" V 8150 2250 59  0000 C CNN
 F 1 "0.1uF" V 8450 2250 59  0000 C CNN
 F 2 "Capacitor_SMD:C_0805_2012Metric" H 8300 2300 50  0001 C CNN
@@
 $EndComp
 $Comp
-L TopBreakout-eagle-import:C-EUC1206 C10
+L TopBreakout-eagle-import:C-EUC1206 C?
 U 1 1 E5C7F153
 P 2600 2300
-AR Path="/E5C7F153" Ref="C10"  Part="1"
-AR Path="/5D7F4465/E5C7F153" Ref="C10"  Part="1"
-F 0 "C10" V 2400 2250 59  0000 C CNN
+AR Path="/E5C7F153" Ref="C?"  Part="1"
+AR Path="/5D7F4465/E5C7F153" Ref="C28"  Part="1"
+F 0 "C28" V 2400 2250 59  0000 C CNN
 F 1 "0.1uF" V 2750 2250 59  0000 C CNN
 F 2 "Capacitors_SMD:C_0805" H 2600 2300 50  0001 C CNN
@@
 $EndComp
 $Comp
-L TopBreakout-eagle-import:C-EUC1206 C11
+L TopBreakout-eagle-import:C-EUC1206 C?
 U 1 1 608006B0
 P 3100 2300
-AR Path="/608006B0" Ref="C11"  Part="1"
-AR Path="/5D7F4465/608006B0" Ref="C11"  Part="1"
-F 0 "C11" V 2950 2250 59  0000 C CNN
+AR Path="/608006B0" Ref="C?"  Part="1"
+AR Path="/5D7F4465/608006B0" Ref="C29"  Part="1"
+F 0 "C29" V 2950 2250 59  0000 C CNN
 F 1 "0.1uF" V 3250 2250 59  0000 C CNN
 F 2 "Capacitors_SMD:C_0805" H 3100 2300 50  0001 C CNN
@@
 $EndComp
 $Comp
-L TopBreakout-eagle-import:GND #GND6
+L TopBreakout-eagle-import:GND #GND?
 U 1 1 6DBAC010
 P 3000 2800
-AR Path="/6DBAC010" Ref="#GND6"  Part="1"
-AR Path="/5D7F4465/6DBAC010" Ref="#GND06"  Part="1"
-F 0 "#GND06" H 3000 2800 50  0001 C CNN
+AR Path="/6DBAC010" Ref="#GND?"  Part="1"
+AR Path="/5D7F4465/6DBAC010" Ref="#GND030"  Part="1"
+F 0 "#GND030" H 3000 2800 50  0001 C CNN
 F 1 "GND" H 2900 2700 59  0000 L BNN
 F 2 "" H 3000 2800 50  0001 C CNN
@@
 Wire Wire Line
 	2600 2200 2150 2200
-$Comp
-L TopBreakout-eagle-import:TEST-POINT3X5 TP?
-U 1 1 5E0D7D26
-P 3800 4000
-AR Path="/5E0D7D26" Ref="TP?"  Part="1"
-AR Path="/5D7F4465/5E0D7D26" Ref="TP10"  Part="1"
-F 0 "TP10" H 3700 4100 70  0001 L BNN
-F 1 "TEST-POINT3X5" V 3700 4000 70  0001 R TNN
-F 2 "topbreakout:PAD.03X.05" H 3800 4000 50  0001 C CNN
-F 3 "" H 3800 4000 50  0001 C CNN
-	1    3800 4000
-	0    1    1    0
-$EndComp
 Text GLabel 7050 3800 2    70   BiDi ~ 0
 DA_V2
@@
 P 3000 3800
 AR Path="/5E139C99" Ref="TP?"  Part="1"
-AR Path="/5D7F4465/5E139C99" Ref="TP11"  Part="1"
-F 0 "TP11" H 2900 3900 70  0001 L BNN
+AR Path="/5D7F4465/5E139C99" Ref="TP2"  Part="1"
+F 0 "TP2" H 2900 3900 70  0001 L BNN
 F 1 "TEST-POINT3X5" V 2900 3800 70  0001 R TNN
 F 2 "topbreakout:PAD.03X.05" H 3000 3800 50  0001 C CNN
