File: hardware/boards/topbreakout/io_breakout-ver2.1_1.sch (KiCad schematic (older format))
At the start: 8 parts

Commit message: minor
Connections:
- net labels added: GATE_1, GATE_2, GATE_3, GATE_4
- net labels removed: DA_V5, DA_V6, TAGND
- wire segments 22 -> 16
Other:
- moved on the sheet: JDA6, JDA7, JDA8
Changed lines of the file:
@@
 Wire Wire Line
 	2700 4800 6500 4800
-Text GLabel 6500 4800 2    70   BiDi ~ 0
+Text GLabel 2700 4800 0    70   BiDi ~ 0
 GND
 Wire Wire Line
@@
 Wire Wire Line
 	2700 4000 8300 4000
-Text GLabel 8300 4000 2    70   BiDi ~ 0
+Text GLabel 2700 4000 0    70   BiDi ~ 0
 DA_V1
-Wire Wire Line
-	6000 4200 7700 4200
-Wire Wire Line
-	6000 4100 6000 4200
-Wire Wire Line
-	6000 4100 2700 4100
-Text GLabel 6300 4200 2    70   BiDi ~ 0
+Text GLabel 2700 4200 0    70   BiDi ~ 0
 DA_V2
-Wire Wire Line
-	5900 4400 7100 4400
-Wire Wire Line
-	5900 4200 5900 4400
-Wire Wire Line
-	5900 4200 2700 4200
-Text GLabel 5950 4400 2    70   BiDi ~ 0
+Text GLabel 2700 4400 0    70   BiDi ~ 0
 DA_V3
-Wire Wire Line
-	5800 4600 6500 4600
-Wire Wire Line
-	5800 4300 5800 4600
-Wire Wire Line
-	5800 4300 2700 4300
-Text GLabel 5950 4600 2    70   BiDi ~ 0
+Text GLabel 2700 4600 0    70   BiDi ~ 0
 DA_V4
-Wire Wire Line
-	5700 5100 8300 5100
-Wire Wire Line
-	2700 4400 5700 4400
-Wire Wire Line
-	5700 4400 5700 5100
-Text Label 6400 5100 0    70   ~ 0
-DA_V5
-Wire Wire Line
-	5600 5300 5600 4500
-Wire Wire Line
-	5600 4500 2700 4500
-Wire Wire Line
-	7700 5300 5600 5300
-Text Label 6400 5300 0    70   ~ 0
-DA_V6
-Wire Wire Line
-	7700 5500 7700 5600
-Text GLabel 7700 5600 2    70   BiDi ~ 0
-TAGND
-Wire Wire Line
-	8300 5300 8300 5400
-Text GLabel 8300 5400 2    70   BiDi ~ 0
-TAGND
 $Comp
 L TopBreakout-eagle-import:THONKICONNNEW JDA1
@@
 L TopBreakout-eagle-import:THONKICONNNEW JDA6
 U 1 1 BACB4F63
-P 7900 5400
+P 8500 5800
 AR Path="/BACB4F63" Ref="JDA6"  Part="1"
 AR Path="/5D7F4208/BACB4F63" Ref="JDA6"  Part="1"
-F 0 "JDA6" H 7800 5560 59  0000 L BNN
-F 1 "THONKICONNNEW" H 7900 5400 50  0001 C CNN
-F 2 "topbreakout:WQP-PJ301M-12_JACK" H 7900 5400 50  0001 C CNN
-F 3 "" H 7900 5400 50  0001 C CNN
-	1    7900 5400
+F 0 "JDA6" H 8400 5960 59  0000 L BNN
+F 1 "THONKICONNNEW" H 8500 5800 50  0001 C CNN
+F 2 "topbreakout:WQP-PJ301M-12_JACK" H 8500 5800 50  0001 C CNN
+F 3 "" H 8500 5800 50  0001 C CNN
+	1    8500 5800
 	1    0    0    -1
 $EndComp
@@
 L TopBreakout-eagle-import:THONKICONNNEW JDA7
 U 1 1 651AD31B
-P 8300 3200
+P 8500 6350
 AR Path="/651AD31B" Ref="JDA7"  Part="1"
 AR Path="/5D7F4208/651AD31B" Ref="JDA7"  Part="1"
-F 0 "JDA7" H 8200 3360 59  0000 L BNN
-F 1 "THONKICONNNEW" H 8300 3200 50  0001 C CNN
-F 2 "topbreakout:WQP-PJ301M-12_JACK" H 8300 3200 50  0001 C CNN
-F 3 "" H 8300 3200 50  0001 C CNN
-	1    8300 3200
+F 0 "JDA7" H 8400 6510 59  0000 L BNN
+F 1 "THONKICONNNEW" H 8500 6350 50  0001 C CNN
+F 2 "topbreakout:WQP-PJ301M-12_JACK" H 8500 6350 50  0001 C CNN
+F 3 "" H 8500 6350 50  0001 C CNN
+	1    8500 6350
 	1    0    0    -1
 $EndComp
@@
 L TopBreakout-eagle-import:THONKICONNNEW JDA8
 U 1 1 860915D8
-P 8300 2800
+P 8600 6900
 AR Path="/860915D8" Ref="JDA8"  Part="1"
 AR Path="/5D7F4208/860915D8" Ref="JDA8"  Part="1"
-F 0 "JDA8" H 8200 2960 59  0000 L BNN
-F 1 "THONKICONNNEW" H 8300 2800 50  0001 C CNN
-F 2 "topbreakout:WQP-PJ301M-12_JACK" H 8300 2800 50  0001 C CNN
-F 3 "" H 8300 2800 50  0001 C CNN
-	1    8300 2800
-	1    0    0    -1
-$EndComp
+F 0 "JDA8" H 8500 7060 59  0000 L BNN
+F 1 "THONKICONNNEW" H 8600 6900 50  0001 C CNN
+F 2 "topbreakout:WQP-PJ301M-12_JACK" H 8600 6900 50  0001 C CNN
+F 3 "" H 8600 6900 50  0001 C CNN
+	1    8600 6900
+	1    0    0    -1
+$EndComp
+Wire Wire Line
+	2700 4600 6500 4600
+Wire Wire Line
+	2700 4400 7100 4400
+Wire Wire Line
+	2700 4200 7700 4200
+Wire Wire Line
+	8300 5100 7150 5100
+Wire Wire Line
+	8300 5700 7150 5700
+Wire Wire Line
+	8300 6250 7100 6250
+Wire Wire Line
+	8400 6800 7150 6800
+Text GLabel 7150 5100 0    59   Input ~ 0
+GATE_1
+Text GLabel 7150 5700 0    59   Input ~ 0
+GATE_2
+Text GLabel 7100 6250 0    59   Input ~ 0
+GATE_3
+Text GLabel 7150 6800 0    59   Input ~ 0
+GATE_4
+Wire Wire Line
+	8300 5300 8300 5400
+Wire Wire Line
+	8300 5900 8300 6000
+Wire Wire Line
+	8300 6450 8300 6550
+Wire Wire Line
+	8400 7000 8400 7100
+$Comp
+L power:GND #PWR0101
+U 1 1 5D8C8CCC
+P 8300 5400
+F 0 "#PWR0101" H 8300 5150 50  0001 C CNN
+F 1 "GND" H 8305 5227 50  0000 C CNN
+F 2 "" H 8300 5400 50  0001 C CNN
+F 3 "" H 8300 5400 50  0001 C CNN
+	1    8300 5400
+	1    0    0    -1
+$EndComp
+$Comp
+L power:GND #PWR0102
+U 1 1 5D8C9140
+P 8300 6000
+F 0 "#PWR0102" H 8300 5750 50  0001 C CNN
+F 1 "GND" H 8305 5827 50  0000 C CNN
+F 2 "" H 8300 6000 50  0001 C CNN
+F 3 "" H 8300 6000 50  0001 C CNN
+	1    8300 6000
+	1    0    0    -1
+$EndComp
+$Comp
+L power:GND #PWR0103
+U 1 1 5D8C9D18
+P 8300 6550
+F 0 "#PWR0103" H 8300 6300 50  0001 C CNN
+F 1 "GND" H 8305 6377 50  0000 C CNN
+F 2 "" H 8300 6550 50  0001 C CNN
+F 3 "" H 8300 6550 50  0001 C CNN
+	1    8300 6550
+	1    0    0    -1
+$EndComp
+$Comp
+L power:GND #PWR0104
+U 1 1 5D8CA15E
+P 8400 7100
+F 0 "#PWR0104" H 8400 6850 50  0001 C CNN
+F 1 "GND" H 8405 6927 50  0000 C CNN
+F 2 "" H 8400 7100 50  0001 C CNN
+F 3 "" H 8400 7100 50  0001 C CNN
+	1    8400 7100
+	1    0    0    -1
+$EndComp

Commit message: TopBreakout: v1.6
Connections:
- no-connect marks 0 -> 8
Other:
- note added: "Control Voltage Output"
- note added: "GPIO"
- moved on the sheet: JDA1, JDA2, JDA3, JDA5, JDA6, JDA7, JDA8
Changed lines of the file:
@@
 $EndDescr
 Wire Wire Line
-	2700 4800 6500 4800
-Text GLabel 2700 4800 0    70   BiDi ~ 0
-GND
-Wire Wire Line
-	7100 4600 7100 4700
-Text GLabel 7100 4700 2    70   BiDi ~ 0
-GND
-Wire Wire Line
-	7700 4400 7700 4500
-Text GLabel 7700 4500 2    70   BiDi ~ 0
-GND
-Wire Wire Line
-	8300 4200 8300 4300
-Text GLabel 8300 4300 2    70   BiDi ~ 0
-GND
-Wire Wire Line
-	2700 4000 8300 4000
-Text GLabel 2700 4000 0    70   BiDi ~ 0
-DA_V1
-Text GLabel 2700 4200 0    70   BiDi ~ 0
-DA_V2
-Text GLabel 2700 4400 0    70   BiDi ~ 0
-DA_V3
-Text GLabel 2700 4600 0    70   BiDi ~ 0
+	6100 4800 6500 4800
+Text GLabel 6100 4800 0    70   BiDi ~ 0
+GND
+Text GLabel 6100 4600 0    70   BiDi ~ 0
 DA_V4
-$Comp
-L TopBreakout-eagle-import:THONKICONNNEW JDA1
-U 1 1 59910AC6
-P 8500 4100
-AR Path="/59910AC6" Ref="JDA1"  Part="1"
-AR Path="/5D7F4208/59910AC6" Ref="JDA1"  Part="1"
-F 0 "JDA1" H 8400 4260 59  0000 L BNN
-F 1 "THONKICONNNEW" H 8500 4100 50  0001 C CNN
-F 2 "topbreakout:WQP-PJ301M-12_JACK" H 8500 4100 50  0001 C CNN
-F 3 "" H 8500 4100 50  0001 C CNN
-	1    8500 4100
-	1    0    0    -1
-$EndComp
-$Comp
-L TopBreakout-eagle-import:THONKICONNNEW JDA2
-U 1 1 57C2BC44
-P 7900 4300
-AR Path="/57C2BC44" Ref="JDA2"  Part="1"
-AR Path="/5D7F4208/57C2BC44" Ref="JDA2"  Part="1"
-F 0 "JDA2" H 7800 4460 59  0000 L BNN
-F 1 "THONKICONNNEW" H 7900 4300 50  0001 C CNN
-F 2 "topbreakout:WQP-PJ301M-12_JACK" H 7900 4300 50  0001 C CNN
-F 3 "" H 7900 4300 50  0001 C CNN
-	1    7900 4300
-	1    0    0    -1
-$EndComp
-$Comp
-L TopBreakout-eagle-import:THONKICONNNEW JDA3
-U 1 1 8B6C1486
-P 7300 4500
-AR Path="/8B6C1486" Ref="JDA3"  Part="1"
-AR Path="/5D7F4208/8B6C1486" Ref="JDA3"  Part="1"
-F 0 "JDA3" H 7200 4660 59  0000 L BNN
-F 1 "THONKICONNNEW" H 7300 4500 50  0001 C CNN
-F 2 "topbreakout:WQP-PJ301M-12_JACK" H 7300 4500 50  0001 C CNN
-F 3 "" H 7300 4500 50  0001 C CNN
-	1    7300 4500
-	1    0    0    -1
-$EndComp
 $Comp
 L TopBreakout-eagle-import:THONKICONNNEW JDA4
@@
 L TopBreakout-eagle-import:THONKICONNNEW JDA5
 U 1 1 6DB94A97
-P 8500 5200
+P 2900 2750
 AR Path="/6DB94A97" Ref="JDA5"  Part="1"
 AR Path="/5D7F4208/6DB94A97" Ref="JDA5"  Part="1"
-F 0 "JDA5" H 8400 5360 59  0000 L BNN
-F 1 "THONKICONNNEW" H 8500 5200 50  0001 C CNN
-F 2 "topbreakout:WQP-PJ301M-12_JACK" H 8500 5200 50  0001 C CNN
-F 3 "" H 8500 5200 50  0001 C CNN
-	1    8500 5200
+F 0 "JDA5" H 2800 2910 59  0000 L BNN
+F 1 "THONKICONNNEW" H 2900 2750 50  0001 C CNN
+F 2 "topbreakout:WQP-PJ301M-12_JACK" H 2900 2750 50  0001 C CNN
+F 3 "" H 2900 2750 50  0001 C CNN
+	1    2900 2750
 	1    0    0    -1
 $EndComp
@@
 L TopBreakout-eagle-import:THONKICONNNEW JDA6
 U 1 1 BACB4F63
-P 8500 5800
+P 2900 3350
 AR Path="/BACB4F63" Ref="JDA6"  Part="1"
 AR Path="/5D7F4208/BACB4F63" Ref="JDA6"  Part="1"
-F 0 "JDA6" H 8400 5960 59  0000 L BNN
-F 1 "THONKICONNNEW" H 8500 5800 50  0001 C CNN
-F 2 "topbreakout:WQP-PJ301M-12_JACK" H 8500 5800 50  0001 C CNN
-F 3 "" H 8500 5800 50  0001 C CNN
-	1    8500 5800
+F 0 "JDA6" H 2800 3510 59  0000 L BNN
+F 1 "THONKICONNNEW" H 2900 3350 50  0001 C CNN
+F 2 "topbreakout:WQP-PJ301M-12_JACK" H 2900 3350 50  0001 C CNN
+F 3 "" H 2900 3350 50  0001 C CNN
+	1    2900 3350
 	1    0    0    -1
 $EndComp
@@
 L TopBreakout-eagle-import:THONKICONNNEW JDA7
 U 1 1 651AD31B
-P 8500 6350
+P 2900 3900
 AR Path="/651AD31B" Ref="JDA7"  Part="1"
 AR Path="/5D7F4208/651AD31B" Ref="JDA7"  Part="1"
-F 0 "JDA7" H 8400 6510 59  0000 L BNN
-F 1 "THONKICONNNEW" H 8500 6350 50  0001 C CNN
-F 2 "topbreakout:WQP-PJ301M-12_JACK" H 8500 6350 50  0001 C CNN
-F 3 "" H 8500 6350 50  0001 C CNN
-	1    8500 6350
+F 0 "JDA7" H 2800 4060 59  0000 L BNN
+F 1 "THONKICONNNEW" H 2900 3900 50  0001 C CNN
+F 2 "topbreakout:WQP-PJ301M-12_JACK" H 2900 3900 50  0001 C CNN
+F 3 "" H 2900 3900 50  0001 C CNN
+	1    2900 3900
 	1    0    0    -1
 $EndComp
@@
 L TopBreakout-eagle-import:THONKICONNNEW JDA8
 U 1 1 860915D8
-P 8600 6900
+P 3000 4450
 AR Path="/860915D8" Ref="JDA8"  Part="1"
 AR Path="/5D7F4208/860915D8" Ref="JDA8"  Part="1"
-F 0 "JDA8" H 8500 7060 59  0000 L BNN
-F 1 "THONKICONNNEW" H 8600 6900 50  0001 C CNN
-F 2 "topbreakout:WQP-PJ301M-12_JACK" H 8600 6900 50  0001 C CNN
-F 3 "" H 8600 6900 50  0001 C CNN
-	1    8600 6900
-	1    0    0    -1
-$EndComp
-Wire Wire Line
-	2700 4600 6500 4600
-Wire Wire Line
-	2700 4400 7100 4400
-Wire Wire Line
-	2700 4200 7700 4200
-Wire Wire Line
-	8300 5100 7150 5100
-Wire Wire Line
-	8300 5700 7150 5700
-Wire Wire Line
-	8300 6250 7100 6250
-Wire Wire Line
-	8400 6800 7150 6800
-Text GLabel 7150 5100 0    59   Input ~ 0
+F 0 "JDA8" H 2900 4610 59  0000 L BNN
+F 1 "THONKICONNNEW" H 3000 4450 50  0001 C CNN
+F 2 "topbreakout:WQP-PJ301M-12_JACK" H 3000 4450 50  0001 C CNN
+F 3 "" H 3000 4450 50  0001 C CNN
+	1    3000 4450
+	1    0    0    -1
+$EndComp
+Wire Wire Line
+	6100 4600 6500 4600
+Wire Wire Line
+	2700 2650 1550 2650
+Wire Wire Line
+	2700 3250 1550 3250
+Wire Wire Line
+	2700 3800 1500 3800
+Wire Wire Line
+	2800 4350 1550 4350
+Text GLabel 1550 2650 0    59   Input ~ 0
 GATE_1
-Text GLabel 7150 5700 0    59   Input ~ 0
+Text GLabel 1550 3250 0    59   Input ~ 0
 GATE_2
-Text GLabel 7100 6250 0    59   Input ~ 0
+Text GLabel 1500 3800 0    59   Input ~ 0
 GATE_3
-Text GLabel 7150 6800 0    59   Input ~ 0
+Text GLabel 1550 4350 0    59   Input ~ 0
 GATE_4
 Wire Wire Line
-	8300 5300 8300 5400
-Wire Wire Line
-	8300 5900 8300 6000
-Wire Wire Line
-	8300 6450 8300 6550
-Wire Wire Line
-	8400 7000 8400 7100
+	2700 2850 2700 2950
+Wire Wire Line
+	2700 3450 2700 3550
+Wire Wire Line
+	2700 4000 2700 4100
+Wire Wire Line
+	2800 4550 2800 4650
 $Comp
 L power:GND #PWR0101
 U 1 1 5D8C8CCC
-P 8300 5400
-F 0 "#PWR0101" H 8300 5150 50  0001 C CNN
-F 1 "GND" H 8305 5227 50  0000 C CNN
-F 2 "" H 8300 5400 50  0001 C CNN
-F 3 "" H 8300 5400 50  0001 C CNN
-	1    8300 5400
+P 2700 2950
+F 0 "#PWR0101" H 2700 2700 50  0001 C CNN
+F 1 "GND" H 2705 2777 50  0000 C CNN
+F 2 "" H 2700 2950 50  0001 C CNN
+F 3 "" H 2700 2950 50  0001 C CNN
+	1    2700 2950
 	1    0    0    -1
 $EndComp
@@
 L power:GND #PWR0102
 U 1 1 5D8C9140
-P 8300 6000
-F 0 "#PWR0102" H 8300 5750 50  0001 C CNN
-F 1 "GND" H 8305 5827 50  0000 C CNN
-F 2 "" H 8300 6000 50  0001 C CNN
-F 3 "" H 8300 6000 50  0001 C CNN
-	1    8300 6000
+P 2700 3550
+F 0 "#PWR0102" H 2700 3300 50  0001 C CNN
+F 1 "GND" H 2705 3377 50  0000 C CNN
+F 2 "" H 2700 3550 50  0001 C CNN
+F 3 "" H 2700 3550 50  0001 C CNN
+	1    2700 3550
 	1    0    0    -1
 $EndComp
@@
 L power:GND #PWR0103
 U 1 1 5D8C9D18
-P 8300 6550
-F 0 "#PWR0103" H 8300 6300 50  0001 C CNN
-F 1 "GND" H 8305 6377 50  0000 C CNN
-F 2 "" H 8300 6550 50  0001 C CNN
-F 3 "" H 8300 6550 50  0001 C CNN
-	1    8300 6550
+P 2700 4100
+F 0 "#PWR0103" H 2700 3850 50  0001 C CNN
+F 1 "GND" H 2705 3927 50  0000 C CNN
+F 2 "" H 2700 4100 50  0001 C CNN
+F 3 "" H 2700 4100 50  0001 C CNN
+	1    2700 4100
 	1    0    0    -1
 $EndComp
@@
 L power:GND #PWR0104
 U 1 1 5D8CA15E
-P 8400 7100
-F 0 "#PWR0104" H 8400 6850 50  0001 C CNN
-F 1 "GND" H 8405 6927 50  0000 C CNN
-F 2 "" H 8400 7100 50  0001 C CNN
-F 3 "" H 8400 7100 50  0001 C CNN
-	1    8400 7100
-	1    0    0    -1
-$EndComp
+P 2800 4650
+F 0 "#PWR0104" H 2800 4400 50  0001 C CNN
+F 1 "GND" H 2805 4477 50  0000 C CNN
+F 2 "" H 2800 4650 50  0001 C CNN
+F 3 "" H 2800 4650 50  0001 C CNN
+	1    2800 4650
+	1    0    0    -1
+$EndComp
+Wire Wire Line
+	7100 4150 6000 4150
+Text GLabel 6100 3950 0    70   BiDi ~ 0
+DA_V3
+Text GLabel 6100 3400 0    70   BiDi ~ 0
+DA_V2
+Text GLabel 6100 2700 0    70   BiDi ~ 0
+DA_V1
+Wire Wire Line
+	7700 3600 6000 3600
+Wire Wire Line
+	6100 3400 7700 3400
+Wire Wire Line
+	6100 3950 7100 3950
+Wire Wire Line
+	8300 2900 6050 2900
+Text GLabel 6000 3600 0    70   BiDi ~ 0
+GND
+Text GLabel 6000 4150 0    70   BiDi ~ 0
+GND
+Wire Wire Line
+	6100 2700 8300 2700
+Text GLabel 6050 2900 0    70   BiDi ~ 0
+GND
+$Comp
+L TopBreakout-eagle-import:THONKICONNNEW JDA3
+U 1 1 8B6C1486
+P 7300 4050
+AR Path="/8B6C1486" Ref="JDA3"  Part="1"
+AR Path="/5D7F4208/8B6C1486" Ref="JDA3"  Part="1"
+F 0 "JDA3" H 7200 4210 59  0000 L BNN
+F 1 "THONKICONNNEW" H 7300 4050 50  0001 C CNN
+F 2 "topbreakout:WQP-PJ301M-12_JACK" H 7300 4050 50  0001 C CNN
+F 3 "" H 7300 4050 50  0001 C CNN
+	1    7300 4050
+	1    0    0    -1
+$EndComp
+$Comp
+L TopBreakout-eagle-import:THONKICONNNEW JDA1
+U 1 1 59910AC6
+P 8500 2800
+AR Path="/59910AC6" Ref="JDA1"  Part="1"
+AR Path="/5D7F4208/59910AC6" Ref="JDA1"  Part="1"
+F 0 "JDA1" H 8400 2960 59  0000 L BNN
+F 1 "THONKICONNNEW" H 8500 2800 50  0001 C CNN
+F 2 "topbreakout:WQP-PJ301M-12_JACK" H 8500 2800 50  0001 C CNN
+F 3 "" H 8500 2800 50  0001 C CNN
+	1    8500 2800
+	1    0    0    -1
+$EndComp
+$Comp
+L TopBreakout-eagle-import:THONKICONNNEW JDA2
+U 1 1 57C2BC44
+P 7900 3500
+AR Path="/57C2BC44" Ref="JDA2"  Part="1"
+AR Path="/5D7F4208/57C2BC44" Ref="JDA2"  Part="1"
+F 0 "JDA2" H 7800 3660 59  0000 L BNN
+F 1 "THONKICONNNEW" H 7900 3500 50  0001 C CNN
+F 2 "topbreakout:WQP-PJ301M-12_JACK" H 7900 3500 50  0001 C CNN
+F 3 "" H 7900 3500 50  0001 C CNN
+	1    7900 3500
+	1    0    0    -1
+$EndComp
+Wire Notes Line
+	3650 2050 3650 5000
+Wire Notes Line
+	3650 5000 650  5000
+Wire Notes Line
+	650  5000 650  2050
+Wire Notes Line
+	650  2050 3650 2050
+Wire Notes Line
+	5550 2050 5550 4950
+Wire Notes Line
+	5550 4950 9250 4950
+Wire Notes Line
+	9250 4950 9250 2050
+Wire Notes Line
+	9250 2050 5550 2050
+Text Notes 1200 2000 0    59   ~ 0
+GPIO
+Text Notes 5600 2000 0    59   ~ 0
+Control Voltage Output
+NoConn ~ 8300 2800
+NoConn ~ 7700 3500
+NoConn ~ 7100 4050
+NoConn ~ 6500 4700
+NoConn ~ 2700 2750
+NoConn ~ 2700 3350
+NoConn ~ 2700 3900
+NoConn ~ 2800 4450
 $EndSCHEMATC

Commit message: mainboard v1.7
Parts:
- renumbered JDA5 to JDA1, JDA6 to JDA2, JDA7 to JDA3, JDA8 to JDA4, JDA4 to JDA5, JDA3 to JDA6, JDA2 to JDA7, JDA1 to JDA8
Changed lines of the file:
@@
-EESchema Schematic File Version 5
+EESchema Schematic File Version 4
 EELAYER 30 0
 EELAYER END
 $Descr A4 11693 8268
 encoding utf-8
-Sheet 2 8
+Sheet 7 13
 Title ""
 Date ""
@@
 Comment3 ""
 Comment4 ""
-Comment5 ""
-Comment6 ""
-Comment7 ""
-Comment8 ""
-Comment9 ""
 $EndDescr
 Wire Wire Line
@@
 DA_V4
 $Comp
-L TopBreakout-eagle-import:THONKICONNNEW JDA4
+L TopBreakout-eagle-import:THONKICONNNEW JDA?
 U 1 1 C7D40660
 P 6700 4700
-AR Path="/C7D40660" Ref="JDA4"  Part="1"
-AR Path="/5D7F4208/C7D40660" Ref="JDA4"  Part="1"
-F 0 "JDA4" H 6600 4860 59  0000 L BNN
+AR Path="/C7D40660" Ref="JDA?"  Part="1"
+AR Path="/5D7F4208/C7D40660" Ref="JDA5"  Part="1"
+F 0 "JDA5" H 6600 4860 59  0000 L BNN
 F 1 "THONKICONNNEW" H 6700 4700 50  0001 C CNN
 F 2 "topbreakout:WQP-PJ301M-12_JACK" H 6700 4700 50  0001 C CNN
@@
 $EndComp
 $Comp
-L TopBreakout-eagle-import:THONKICONNNEW JDA5
+L TopBreakout-eagle-import:THONKICONNNEW JDA?
 U 1 1 6DB94A97
 P 2900 2750
-AR Path="/6DB94A97" Ref="JDA5"  Part="1"
-AR Path="/5D7F4208/6DB94A97" Ref="JDA5"  Part="1"
-F 0 "JDA5" H 2800 2910 59  0000 L BNN
+AR Path="/6DB94A97" Ref="JDA?"  Part="1"
+AR Path="/5D7F4208/6DB94A97" Ref="JDA1"  Part="1"
+F 0 "JDA1" H 2800 2910 59  0000 L BNN
 F 1 "THONKICONNNEW" H 2900 2750 50  0001 C CNN
 F 2 "topbreakout:WQP-PJ301M-12_JACK" H 2900 2750 50  0001 C CNN
@@
 $EndComp
 $Comp
-L TopBreakout-eagle-import:THONKICONNNEW JDA6
+L TopBreakout-eagle-import:THONKICONNNEW JDA?
 U 1 1 BACB4F63
 P 2900 3350
-AR Path="/BACB4F63" Ref="JDA6"  Part="1"
-AR Path="/5D7F4208/BACB4F63" Ref="JDA6"  Part="1"
-F 0 "JDA6" H 2800 3510 59  0000 L BNN
+AR Path="/BACB4F63" Ref="JDA?"  Part="1"
+AR Path="/5D7F4208/BACB4F63" Ref="JDA2"  Part="1"
+F 0 "JDA2" H 2800 3510 59  0000 L BNN
 F 1 "THONKICONNNEW" H 2900 3350 50  0001 C CNN
 F 2 "topbreakout:WQP-PJ301M-12_JACK" H 2900 3350 50  0001 C CNN
@@
 $EndComp
 $Comp
-L TopBreakout-eagle-import:THONKICONNNEW JDA7
+L TopBreakout-eagle-import:THONKICONNNEW JDA?
 U 1 1 651AD31B
 P 2900 3900
-AR Path="/651AD31B" Ref="JDA7"  Part="1"
-AR Path="/5D7F4208/651AD31B" Ref="JDA7"  Part="1"
-F 0 "JDA7" H 2800 4060 59  0000 L BNN
+AR Path="/651AD31B" Ref="JDA?"  Part="1"
+AR Path="/5D7F4208/651AD31B" Ref="JDA3"  Part="1"
+F 0 "JDA3" H 2800 4060 59  0000 L BNN
 F 1 "THONKICONNNEW" H 2900 3900 50  0001 C CNN
 F 2 "topbreakout:WQP-PJ301M-12_JACK" H 2900 3900 50  0001 C CNN
@@
 $EndComp
 $Comp
-L TopBreakout-eagle-import:THONKICONNNEW JDA8
+L TopBreakout-eagle-import:THONKICONNNEW JDA?
 U 1 1 860915D8
 P 3000 4450
-AR Path="/860915D8" Ref="JDA8"  Part="1"
-AR Path="/5D7F4208/860915D8" Ref="JDA8"  Part="1"
-F 0 "JDA8" H 2900 4610 59  0000 L BNN
+AR Path="/860915D8" Ref="JDA?"  Part="1"
+AR Path="/5D7F4208/860915D8" Ref="JDA4"  Part="1"
+F 0 "JDA4" H 2900 4610 59  0000 L BNN
 F 1 "THONKICONNNEW" H 3000 4450 50  0001 C CNN
 F 2 "topbreakout:WQP-PJ301M-12_JACK" H 3000 4450 50  0001 C CNN
@@
 	2800 4550 2800 4650
 $Comp
-L power:GND #PWR0101
+L power:GND #PWR021
 U 1 1 5D8C8CCC
 P 2700 2950
-F 0 "#PWR0101" H 2700 2700 50  0001 C CNN
+F 0 "#PWR021" H 2700 2700 50  0001 C CNN
 F 1 "GND" H 2705 2777 50  0000 C CNN
 F 2 "" H 2700 2950 50  0001 C CNN
@@
 $EndComp
 $Comp
-L power:GND #PWR0102
+L power:GND #PWR022
 U 1 1 5D8C9140
 P 2700 3550
-F 0 "#PWR0102" H 2700 3300 50  0001 C CNN
+F 0 "#PWR022" H 2700 3300 50  0001 C CNN
 F 1 "GND" H 2705 3377 50  0000 C CNN
 F 2 "" H 2700 3550 50  0001 C CNN
@@
 $EndComp
 $Comp
-L power:GND #PWR0103
+L power:GND #PWR023
 U 1 1 5D8C9D18
 P 2700 4100
-F 0 "#PWR0103" H 2700 3850 50  0001 C CNN
+F 0 "#PWR023" H 2700 3850 50  0001 C CNN
 F 1 "GND" H 2705 3927 50  0000 C CNN
 F 2 "" H 2700 4100 50  0001 C CNN
@@
 $EndComp
 $Comp
-L power:GND #PWR0104
+L power:GND #PWR024
 U 1 1 5D8CA15E
 P 2800 4650
-F 0 "#PWR0104" H 2800 4400 50  0001 C CNN
+F 0 "#PWR024" H 2800 4400 50  0001 C CNN
 F 1 "GND" H 2805 4477 50  0000 C CNN
 F 2 "" H 2800 4650 50  0001 C CNN
@@
 GND
 $Comp
-L TopBreakout-eagle-import:THONKICONNNEW JDA3
+L TopBreakout-eagle-import:THONKICONNNEW JDA?
 U 1 1 8B6C1486
 P 7300 4050
-AR Path="/8B6C1486" Ref="JDA3"  Part="1"
-AR Path="/5D7F4208/8B6C1486" Ref="JDA3"  Part="1"
-F 0 "JDA3" H 7200 4210 59  0000 L BNN
+AR Path="/8B6C1486" Ref="JDA?"  Part="1"
+AR Path="/5D7F4208/8B6C1486" Ref="JDA6"  Part="1"
+F 0 "JDA6" H 7200 4210 59  0000 L BNN
 F 1 "THONKICONNNEW" H 7300 4050 50  0001 C CNN
 F 2 "topbreakout:WQP-PJ301M-12_JACK" H 7300 4050 50  0001 C CNN
@@
 $EndComp
 $Comp
-L TopBreakout-eagle-import:THONKICONNNEW JDA1
+L TopBreakout-eagle-import:THONKICONNNEW JDA?
 U 1 1 59910AC6
 P 8500 2800
-AR Path="/59910AC6" Ref="JDA1"  Part="1"
-AR Path="/5D7F4208/59910AC6" Ref="JDA1"  Part="1"
-F 0 "JDA1" H 8400 2960 59  0000 L BNN
+AR Path="/59910AC6" Ref="JDA?"  Part="1"
+AR Path="/5D7F4208/59910AC6" Ref="JDA8"  Part="1"
+F 0 "JDA8" H 8400 2960 59  0000 L BNN
 F 1 "THONKICONNNEW" H 8500 2800 50  0001 C CNN
 F 2 "topbreakout:WQP-PJ301M-12_JACK" H 8500 2800 50  0001 C CNN
@@
 $EndComp
 $Comp
-L TopBreakout-eagle-import:THONKICONNNEW JDA2
+L TopBreakout-eagle-import:THONKICONNNEW JDA?
 U 1 1 57C2BC44
 P 7900 3500
-AR Path="/57C2BC44" Ref="JDA2"  Part="1"
-AR Path="/5D7F4208/57C2BC44" Ref="JDA2"  Part="1"
-F 0 "JDA2" H 7800 3660 59  0000 L BNN
+AR Path="/57C2BC44" Ref="JDA?"  Part="1"
+AR Path="/5D7F4208/57C2BC44" Ref="JDA7"  Part="1"
+F 0 "JDA7" H 7800 3660 59  0000 L BNN
 F 1 "THONKICONNNEW" H 7900 3500 50  0001 C CNN
 F 2 "topbreakout:WQP-PJ301M-12_JACK" H 7900 3500 50  0001 C CNN
