File: hardware/boards/topbreakout/io_breakout-ver2.1_2.sch (KiCad schematic (older format))
At the start: 8 parts

Commit message: minor
Connections:
- net labels added: AD_V5, AD_V6, AD_V7, AD_V8
- net labels removed: TAGND
- wire segments 21 -> 25
Changed lines of the file:
@@
 Wire Wire Line
 	2600 3100 1300 3100
-Text GLabel 3500 3200 2    70   BiDi ~ 0
+Text GLabel 1300 3100 0    70   BiDi ~ 0
 AD_V2
 Wire Wire Line
@@
 Wire Wire Line
 	2500 3200 1300 3200
-Text GLabel 3500 3400 2    70   BiDi ~ 0
+Text GLabel 1300 3200 0    70   BiDi ~ 0
 AD_V3
 Wire Wire Line
@@
 Wire Wire Line
 	2400 3600 2400 3300
-Text GLabel 3500 3600 2    70   BiDi ~ 0
+Text GLabel 2400 3300 0    70   BiDi ~ 0
 AD_V4
 Wire Wire Line
 	8200 3700 8200 3800
-Wire Wire Line
-	8200 3800 8200 4000
-Connection ~ 8200 3800
-Text GLabel 8200 3900 2    70   BiDi ~ 0
-GND
 Wire Wire Line
 	8700 3500 8700 3600
@@
 Wire Wire Line
 	1300 3000 9800 3000
-Text GLabel 3500 3000 2    70   BiDi ~ 0
+Text GLabel 1300 3000 0    70   BiDi ~ 0
 AD_V1
 Wire Wire Line
 	7100 4100 7100 4200
 Wire Wire Line
-	7100 4200 7100 4300
-Connection ~ 7100 4200
-Text GLabel 7100 4300 2    70   BiDi ~ 0
-TAGND
-Wire Wire Line
 	7600 3900 7600 4000
-Wire Wire Line
-	7600 4000 7600 4100
-Connection ~ 7600 4000
-Text GLabel 7600 4100 2    70   BiDi ~ 0
-TAGND
 $Comp
-L TopBreakout-eagle-import:THONKICONNNEW JAD1
+L TopBreakout-eagle-import:THONKICONNNEW JAD?
 U 1 1 4CF81522
 P 10000 3100
-AR Path="/4CF81522" Ref="JAD1"  Part="1"
+AR Path="/4CF81522" Ref="JAD?"  Part="1"
 AR Path="/5D7F4281/4CF81522" Ref="JAD1"  Part="1"
 F 0 "JAD1" H 9900 3260 59  0000 L BNN
@@
 $EndComp
 $Comp
-L TopBreakout-eagle-import:THONKICONNNEW JAD2
+L TopBreakout-eagle-import:THONKICONNNEW JAD?
 U 1 1 EEF6290D
 P 9400 3300
-AR Path="/EEF6290D" Ref="JAD2"  Part="1"
+AR Path="/EEF6290D" Ref="JAD?"  Part="1"
 AR Path="/5D7F4281/EEF6290D" Ref="JAD2"  Part="1"
 F 0 "JAD2" H 9300 3460 59  0000 L BNN
@@
 $EndComp
 $Comp
-L TopBreakout-eagle-import:THONKICONNNEW JAD3
+L TopBreakout-eagle-import:THONKICONNNEW JAD?
 U 1 1 38B49BA0
 P 8900 3500
-AR Path="/38B49BA0" Ref="JAD3"  Part="1"
+AR Path="/38B49BA0" Ref="JAD?"  Part="1"
 AR Path="/5D7F4281/38B49BA0" Ref="JAD3"  Part="1"
 F 0 "JAD3" H 8800 3660 59  0000 L BNN
@@
 $EndComp
 $Comp
-L TopBreakout-eagle-import:THONKICONNNEW JAD4
+L TopBreakout-eagle-import:THONKICONNNEW JAD?
 U 1 1 0E8D2B61
 P 8400 3700
-AR Path="/0E8D2B61" Ref="JAD4"  Part="1"
+AR Path="/0E8D2B61" Ref="JAD?"  Part="1"
 AR Path="/5D7F4281/0E8D2B61" Ref="JAD4"  Part="1"
 F 0 "JAD4" H 8300 3860 59  0000 L BNN
@@
 $EndComp
 $Comp
-L TopBreakout-eagle-import:THONKICONNNEW JAD5
+L TopBreakout-eagle-import:THONKICONNNEW JAD?
 U 1 1 555B4C4E
 P 7800 3900
-AR Path="/555B4C4E" Ref="JAD5"  Part="1"
+AR Path="/555B4C4E" Ref="JAD?"  Part="1"
 AR Path="/5D7F4281/555B4C4E" Ref="JAD5"  Part="1"
 F 0 "JAD5" H 7700 4060 59  0000 L BNN
@@
 $EndComp
 $Comp
-L TopBreakout-eagle-import:THONKICONNNEW JAD6
+L TopBreakout-eagle-import:THONKICONNNEW JAD?
 U 1 1 893B2485
 P 7300 4100
-AR Path="/893B2485" Ref="JAD6"  Part="1"
+AR Path="/893B2485" Ref="JAD?"  Part="1"
 AR Path="/5D7F4281/893B2485" Ref="JAD6"  Part="1"
 F 0 "JAD6" H 7200 4260 59  0000 L BNN
@@
 $EndComp
 $Comp
-L TopBreakout-eagle-import:THONKICONNNEW JAD7
+L TopBreakout-eagle-import:THONKICONNNEW JAD?
 U 1 1 4CC294C2
 P 7300 4700
-AR Path="/4CC294C2" Ref="JAD7"  Part="1"
+AR Path="/4CC294C2" Ref="JAD?"  Part="1"
 AR Path="/5D7F4281/4CC294C2" Ref="JAD7"  Part="1"
 F 0 "JAD7" H 7200 4860 59  0000 L BNN
@@
 $EndComp
 $Comp
-L TopBreakout-eagle-import:THONKICONNNEW JAD8
+L TopBreakout-eagle-import:THONKICONNNEW JAD?
 U 1 1 AF2FA07E
 P 7300 5200
-AR Path="/AF2FA07E" Ref="JAD8"  Part="1"
+AR Path="/AF2FA07E" Ref="JAD?"  Part="1"
 AR Path="/5D7F4281/AF2FA07E" Ref="JAD8"  Part="1"
 F 0 "JAD8" H 7200 5360 59  0000 L BNN
@@
 	1    0    0    -1
 $EndComp
+Text GLabel 8200 3900 2    70   BiDi ~ 0
+GND
+Connection ~ 8200 3800
+Wire Wire Line
+	8200 3800 8200 3900
+Wire Wire Line
+	7100 4000 6150 4000
+Wire Wire Line
+	6150 4000 6150 4050
+Wire Wire Line
+	7600 3800 6200 3800
+Wire Wire Line
+	6200 3800 6200 3850
+Wire Wire Line
+	7100 4600 6100 4600
+Wire Wire Line
+	7100 5100 6100 5100
+Text GLabel 6200 3850 0    59   Input ~ 0
+AD_V5
+Text GLabel 6150 4050 0    59   Input ~ 0
+AD_V6
+Text GLabel 6100 4600 0    59   Input ~ 0
+AD_V7
+Text GLabel 6100 5100 0    59   Input ~ 0
+AD_V8
 $EndSCHEMATC

Commit message: imporvements
Connections:
- net GND: now also JAD5.P$2_SWITCH (SWITCH), JAD5.P$3_SLEEVE (SLEEVE), JAD6.P$2_SWITCH (SWITCH), JAD6.P$3_SLEEVE (SLEEVE), JAD7.P$2_SWITCH (SWITCH), JAD7.P$3_SLEEVE (SLEEVE), JAD8.P$2_SWITCH (SWITCH), JAD8.P$3_SLEEVE (SLEEVE)
Other:
- moved on the sheet: JAD5, JAD6, JAD7, JAD8
Changed lines of the file:
@@
 AD_V1
 Wire Wire Line
-	7100 4100 7100 4200
+	7500 5300 7500 5400
 Wire Wire Line
-	7600 3900 7600 4000
+	7600 4750 7600 4850
 $Comp
 L TopBreakout-eagle-import:THONKICONNNEW JAD?
@@
 L TopBreakout-eagle-import:THONKICONNNEW JAD?
 U 1 1 555B4C4E
-P 7800 3900
+P 7800 4750
 AR Path="/555B4C4E" Ref="JAD?"  Part="1"
 AR Path="/5D7F4281/555B4C4E" Ref="JAD5"  Part="1"
-F 0 "JAD5" H 7700 4060 59  0000 L BNN
-F 1 "THONKICONNNEW" H 7800 3900 50  0001 C CNN
-F 2 "topbreakout:WQP-PJ301M-12_JACK" H 7800 3900 50  0001 C CNN
-F 3 "" H 7800 3900 50  0001 C CNN
-	1    7800 3900
+F 0 "JAD5" H 7700 4910 59  0000 L BNN
+F 1 "THONKICONNNEW" H 7800 4750 50  0001 C CNN
+F 2 "topbreakout:WQP-PJ301M-12_JACK" H 7800 4750 50  0001 C CNN
+F 3 "" H 7800 4750 50  0001 C CNN
+	1    7800 4750
 	1    0    0    -1
 $EndComp
@@
 L TopBreakout-eagle-import:THONKICONNNEW JAD?
 U 1 1 893B2485
-P 7300 4100
+P 7700 5300
 AR Path="/893B2485" Ref="JAD?"  Part="1"
 AR Path="/5D7F4281/893B2485" Ref="JAD6"  Part="1"
-F 0 "JAD6" H 7200 4260 59  0000 L BNN
-F 1 "THONKICONNNEW" H 7300 4100 50  0001 C CNN
-F 2 "topbreakout:WQP-PJ301M-12_JACK" H 7300 4100 50  0001 C CNN
-F 3 "" H 7300 4100 50  0001 C CNN
-	1    7300 4100
+F 0 "JAD6" H 7600 5460 59  0000 L BNN
+F 1 "THONKICONNNEW" H 7700 5300 50  0001 C CNN
+F 2 "topbreakout:WQP-PJ301M-12_JACK" H 7700 5300 50  0001 C CNN
+F 3 "" H 7700 5300 50  0001 C CNN
+	1    7700 5300
 	1    0    0    -1
 $EndComp
@@
 L TopBreakout-eagle-import:THONKICONNNEW JAD?
 U 1 1 4CC294C2
-P 7300 4700
+P 7700 5900
 AR Path="/4CC294C2" Ref="JAD?"  Part="1"
 AR Path="/5D7F4281/4CC294C2" Ref="JAD7"  Part="1"
-F 0 "JAD7" H 7200 4860 59  0000 L BNN
-F 1 "THONKICONNNEW" H 7300 4700 50  0001 C CNN
-F 2 "topbreakout:WQP-PJ301M-12_JACK" H 7300 4700 50  0001 C CNN
-F 3 "" H 7300 4700 50  0001 C CNN
-	1    7300 4700
+F 0 "JAD7" H 7600 6060 59  0000 L BNN
+F 1 "THONKICONNNEW" H 7700 5900 50  0001 C CNN
+F 2 "topbreakout:WQP-PJ301M-12_JACK" H 7700 5900 50  0001 C CNN
+F 3 "" H 7700 5900 50  0001 C CNN
+	1    7700 5900
 	1    0    0    -1
 $EndComp
@@
 L TopBreakout-eagle-import:THONKICONNNEW JAD?
 U 1 1 AF2FA07E
-P 7300 5200
+P 7700 6400
 AR Path="/AF2FA07E" Ref="JAD?"  Part="1"
 AR Path="/5D7F4281/AF2FA07E" Ref="JAD8"  Part="1"
-F 0 "JAD8" H 7200 5360 59  0000 L BNN
-F 1 "THONKICONNNEW" H 7300 5200 50  0001 C CNN
-F 2 "topbreakout:WQP-PJ301M-12_JACK" H 7300 5200 50  0001 C CNN
-F 3 "" H 7300 5200 50  0001 C CNN
-	1    7300 5200
+F 0 "JAD8" H 7600 6560 59  0000 L BNN
+F 1 "THONKICONNNEW" H 7700 6400 50  0001 C CNN
+F 2 "topbreakout:WQP-PJ301M-12_JACK" H 7700 6400 50  0001 C CNN
+F 3 "" H 7700 6400 50  0001 C CNN
+	1    7700 6400
 	1    0    0    -1
 $EndComp
@@
 	8200 3800 8200 3900
 Wire Wire Line
-	7100 4000 6150 4000
+	7500 5200 6550 5200
 Wire Wire Line
-	6150 4000 6150 4050
+	6550 5200 6550 5250
 Wire Wire Line
-	7600 3800 6200 3800
+	7600 4650 6200 4650
 Wire Wire Line
-	6200 3800 6200 3850
+	6200 4650 6200 4700
 Wire Wire Line
-	7100 4600 6100 4600
+	7500 5800 6500 5800
 Wire Wire Line
-	7100 5100 6100 5100
-Text GLabel 6200 3850 0    59   Input ~ 0
+	7500 6300 6500 6300
+Text GLabel 6200 4700 0    59   Input ~ 0
 AD_V5
-Text GLabel 6150 4050 0    59   Input ~ 0
+Text GLabel 6550 5250 0    59   Input ~ 0
 AD_V6
-Text GLabel 6100 4600 0    59   Input ~ 0
+Text GLabel 6500 5800 0    59   Input ~ 0
 AD_V7
-Text GLabel 6100 5100 0    59   Input ~ 0
+Text GLabel 6500 6300 0    59   Input ~ 0
 AD_V8
+Text GLabel 7600 4850 0    70   BiDi ~ 0
+GND
+Text GLabel 7500 5400 0    70   BiDi ~ 0
+GND
+Text GLabel 7500 6000 0    70   BiDi ~ 0
+GND
+Text GLabel 7500 6500 0    70   BiDi ~ 0
+GND
+Wire Wire Line
+	7500 5900 7500 6000
+Wire Wire Line
+	7500 6400 7500 6500
 $EndSCHEMATC

Commit message: TopBreakout: v1.6
Connections:
- net GND renamed AD_AGND
Other:
- moved on the sheet: JAD1, JAD2, JAD3, JAD4, JAD5, JAD8
Changed lines of the file:
@@
 $EndDescr
 Wire Wire Line
-	2600 3200 9200 3200
+	7500 2950 7500 3050
 Wire Wire Line
-	2600 3200 2600 3100
-Wire Wire Line
-	2600 3100 1300 3100
-Text GLabel 1300 3100 0    70   BiDi ~ 0
-AD_V2
-Wire Wire Line
-	2500 3400 8700 3400
-Wire Wire Line
-	2500 3400 2500 3200
-Wire Wire Line
-	2500 3200 1300 3200
-Text GLabel 1300 3200 0    70   BiDi ~ 0
-AD_V3
-Wire Wire Line
-	2400 3600 8200 3600
-Wire Wire Line
-	2400 3600 2400 3300
-Text GLabel 2400 3300 0    70   BiDi ~ 0
-AD_V4
-Wire Wire Line
-	8200 3700 8200 3800
-Wire Wire Line
-	8700 3500 8700 3600
-Wire Wire Line
-	8700 3600 8700 3700
-Connection ~ 8700 3600
-Text GLabel 8700 3700 2    70   BiDi ~ 0
-GND
-Wire Wire Line
-	9200 3300 9200 3400
-Wire Wire Line
-	9200 3400 9200 3500
-Connection ~ 9200 3400
-Text GLabel 9200 3500 2    70   BiDi ~ 0
-GND
-Wire Wire Line
-	9800 3100 9800 3200
-Wire Wire Line
-	9800 3200 9800 3400
-Connection ~ 9800 3200
-Text GLabel 9800 3400 2    70   BiDi ~ 0
-GND
-Wire Wire Line
-	1300 3000 9800 3000
-Text GLabel 1300 3000 0    70   BiDi ~ 0
-AD_V1
+	7500 3050 6550 3050
+Connection ~ 7500 3050
 Wire Wire Line
 	7500 5300 7500 5400
 Wire Wire Line
-	7600 4750 7600 4850
+	7500 4750 7500 4850
 $Comp
 L TopBreakout-eagle-import:THONKICONNNEW JAD?
 U 1 1 4CF81522
-P 10000 3100
+P 7700 2350
 AR Path="/4CF81522" Ref="JAD?"  Part="1"
 AR Path="/5D7F4281/4CF81522" Ref="JAD1"  Part="1"
-F 0 "JAD1" H 9900 3260 59  0000 L BNN
-F 1 "THONKICONNNEW" H 10000 3100 50  0001 C CNN
-F 2 "topbreakout:WQP-PJ301M-12_JACK" H 10000 3100 50  0001 C CNN
-F 3 "" H 10000 3100 50  0001 C CNN
-	1    10000 3100
+F 0 "JAD1" H 7600 2510 59  0000 L BNN
+F 1 "THONKICONNNEW" H 7700 2350 50  0001 C CNN
+F 2 "topbreakout:WQP-PJ301M-12_JACK" H 7700 2350 50  0001 C CNN
+F 3 "" H 7700 2350 50  0001 C CNN
+	1    7700 2350
 	1    0    0    -1
 $EndComp
@@
 L TopBreakout-eagle-import:THONKICONNNEW JAD?
 U 1 1 EEF6290D
-P 9400 3300
+P 7700 2950
 AR Path="/EEF6290D" Ref="JAD?"  Part="1"
 AR Path="/5D7F4281/EEF6290D" Ref="JAD2"  Part="1"
-F 0 "JAD2" H 9300 3460 59  0000 L BNN
-F 1 "THONKICONNNEW" H 9400 3300 50  0001 C CNN
-F 2 "topbreakout:WQP-PJ301M-12_JACK" H 9400 3300 50  0001 C CNN
-F 3 "" H 9400 3300 50  0001 C CNN
-	1    9400 3300
+F 0 "JAD2" H 7600 3110 59  0000 L BNN
+F 1 "THONKICONNNEW" H 7700 2950 50  0001 C CNN
+F 2 "topbreakout:WQP-PJ301M-12_JACK" H 7700 2950 50  0001 C CNN
+F 3 "" H 7700 2950 50  0001 C CNN
+	1    7700 2950
 	1    0    0    -1
 $EndComp
@@
 L TopBreakout-eagle-import:THONKICONNNEW JAD?
 U 1 1 38B49BA0
-P 8900 3500
+P 7700 3600
 AR Path="/38B49BA0" Ref="JAD?"  Part="1"
 AR Path="/5D7F4281/38B49BA0" Ref="JAD3"  Part="1"
-F 0 "JAD3" H 8800 3660 59  0000 L BNN
-F 1 "THONKICONNNEW" H 8900 3500 50  0001 C CNN
-F 2 "topbreakout:WQP-PJ301M-12_JACK" H 8900 3500 50  0001 C CNN
-F 3 "" H 8900 3500 50  0001 C CNN
-	1    8900 3500
+F 0 "JAD3" H 7600 3760 59  0000 L BNN
+F 1 "THONKICONNNEW" H 7700 3600 50  0001 C CNN
+F 2 "topbreakout:WQP-PJ301M-12_JACK" H 7700 3600 50  0001 C CNN
+F 3 "" H 7700 3600 50  0001 C CNN
+	1    7700 3600
 	1    0    0    -1
 $EndComp
@@
 L TopBreakout-eagle-import:THONKICONNNEW JAD?
 U 1 1 0E8D2B61
-P 8400 3700
+P 7700 4150
 AR Path="/0E8D2B61" Ref="JAD?"  Part="1"
 AR Path="/5D7F4281/0E8D2B61" Ref="JAD4"  Part="1"
-F 0 "JAD4" H 8300 3860 59  0000 L BNN
-F 1 "THONKICONNNEW" H 8400 3700 50  0001 C CNN
-F 2 "topbreakout:WQP-PJ301M-12_JACK" H 8400 3700 50  0001 C CNN
-F 3 "" H 8400 3700 50  0001 C CNN
-	1    8400 3700
+F 0 "JAD4" H 7600 4310 59  0000 L BNN
+F 1 "THONKICONNNEW" H 7700 4150 50  0001 C CNN
+F 2 "topbreakout:WQP-PJ301M-12_JACK" H 7700 4150 50  0001 C CNN
+F 3 "" H 7700 4150 50  0001 C CNN
+	1    7700 4150
 	1    0    0    -1
 $EndComp
@@
 L TopBreakout-eagle-import:THONKICONNNEW JAD?
 U 1 1 555B4C4E
-P 7800 4750
+P 7700 4750
 AR Path="/555B4C4E" Ref="JAD?"  Part="1"
 AR Path="/5D7F4281/555B4C4E" Ref="JAD5"  Part="1"
-F 0 "JAD5" H 7700 4910 59  0000 L BNN
-F 1 "THONKICONNNEW" H 7800 4750 50  0001 C CNN
-F 2 "topbreakout:WQP-PJ301M-12_JACK" H 7800 4750 50  0001 C CNN
-F 3 "" H 7800 4750 50  0001 C CNN
-	1    7800 4750
+F 0 "JAD5" H 7600 4910 59  0000 L BNN
+F 1 "THONKICONNNEW" H 7700 4750 50  0001 C CNN
+F 2 "topbreakout:WQP-PJ301M-12_JACK" H 7700 4750 50  0001 C CNN
+F 3 "" H 7700 4750 50  0001 C CNN
+	1    7700 4750
 	1    0    0    -1
 $EndComp
@@
 L TopBreakout-eagle-import:THONKICONNNEW JAD?
 U 1 1 AF2FA07E
-P 7700 6400
+P 7700 6500
 AR Path="/AF2FA07E" Ref="JAD?"  Part="1"
 AR Path="/5D7F4281/AF2FA07E" Ref="JAD8"  Part="1"
-F 0 "JAD8" H 7600 6560 59  0000 L BNN
-F 1 "THONKICONNNEW" H 7700 6400 50  0001 C CNN
-F 2 "topbreakout:WQP-PJ301M-12_JACK" H 7700 6400 50  0001 C CNN
-F 3 "" H 7700 6400 50  0001 C CNN
-	1    7700 6400
+F 0 "JAD8" H 7600 6660 59  0000 L BNN
+F 1 "THONKICONNNEW" H 7700 6500 50  0001 C CNN
+F 2 "topbreakout:WQP-PJ301M-12_JACK" H 7700 6500 50  0001 C CNN
+F 3 "" H 7700 6500 50  0001 C CNN
+	1    7700 6500
 	1    0    0    -1
 $EndComp
-Text GLabel 8200 3900 2    70   BiDi ~ 0
-GND
-Connection ~ 8200 3800
-Wire Wire Line
-	8200 3800 8200 3900
 Wire Wire Line
 	7500 5200 6550 5200
 Wire Wire Line
-	6550 5200 6550 5250
-Wire Wire Line
-	7600 4650 6200 4650
-Wire Wire Line
-	6200 4650 6200 4700
+	7500 4650 6450 4650
 Wire Wire Line
 	7500 5800 6500 5800
 Wire Wire Line
-	7500 6300 6500 6300
-Text GLabel 6200 4700 0    59   Input ~ 0
+	7500 6400 6500 6400
+Text GLabel 6450 4650 0    59   Input ~ 0
 AD_V5
-Text GLabel 6550 5250 0    59   Input ~ 0
+Text GLabel 6550 5200 0    59   Input ~ 0
 AD_V6
 Text GLabel 6500 5800 0    59   Input ~ 0
 AD_V7
-Text GLabel 6500 6300 0    59   Input ~ 0
+Text GLabel 6500 6400 0    59   Input ~ 0
 AD_V8
-Text GLabel 7600 4850 0    70   BiDi ~ 0
-GND
-Text GLabel 7500 5400 0    70   BiDi ~ 0
-GND
-Text GLabel 7500 6000 0    70   BiDi ~ 0
-GND
-Text GLabel 7500 6500 0    70   BiDi ~ 0
-GND
 Wire Wire Line
 	7500 5900 7500 6000
 Wire Wire Line
-	7500 6400 7500 6500
+	7500 6500 7500 6600
+Wire Wire Line
+	6400 2850 7500 2850
+Text GLabel 6400 2850 0    70   BiDi ~ 0
+AD_V2
+Text GLabel 6550 3050 0    70   BiDi ~ 0
+AD_AGND
+Text GLabel 6650 4850 0    70   BiDi ~ 0
+AD_AGND
+Text GLabel 6750 5400 0    70   BiDi ~ 0
+AD_AGND
+Text GLabel 6800 6000 0    70   BiDi ~ 0
+AD_AGND
+Text GLabel 6750 6600 0    70   BiDi ~ 0
+AD_AGND
+Wire Wire Line
+	7500 4850 6650 4850
+Connection ~ 7500 4850
+Wire Wire Line
+	7500 5400 6750 5400
+Connection ~ 7500 5400
+Wire Wire Line
+	7500 6000 6800 6000
+Connection ~ 7500 6000
+Wire Wire Line
+	7500 6600 6750 6600
+Connection ~ 7500 6600
+Text GLabel 6600 3700 0    70   BiDi ~ 0
+AD_AGND
+Text GLabel 6500 4250 0    70   BiDi ~ 0
+AD_AGND
+Connection ~ 7500 3700
+Wire Wire Line
+	7500 3700 6600 3700
+Wire Wire Line
+	7500 3600 7500 3700
+Wire Wire Line
+	7500 4150 7500 4250
+Text GLabel 6350 4050 0    70   BiDi ~ 0
+AD_V4
+Wire Wire Line
+	6450 3500 7500 3500
+Wire Wire Line
+	6350 4050 7500 4050
+Text GLabel 6450 3500 0    70   BiDi ~ 0
+AD_V3
+Wire Wire Line
+	7500 4250 6500 4250
+Connection ~ 7500 4250
+Wire Wire Line
+	6400 2250 7500 2250
+Connection ~ 7500 2450
+Wire Wire Line
+	7500 2450 6550 2450
+Wire Wire Line
+	7500 2350 7500 2450
+Text GLabel 6400 2250 0    70   BiDi ~ 0
+AD_V1
+Text GLabel 6550 2450 0    70   BiDi ~ 0
+AD_AGND
 $EndSCHEMATC
