File: hardware/boards/topbreakout/io_breakout-ver2.1_3.sch (KiCad schematic (older format))
At the start: 5 parts, among them J1 WURTH_ELECTRONICS_61400413321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, J2 MOLEX_52892-3033MOLEX_52892-3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, J3 USB-A-S-X-X-VT

Commit message: TopBreakout: v1.6
Connections:
- no-connect marks 0 -> 10
Changed lines of the file:
@@
-$EndComp
-$Comp
-L TopBreakout-eagle-import:USB-A-S-X-X-VT J3
-U 1 1 83A3164B
-P 4750 3600
-AR Path="/83A3164B" Ref="J3"  Part="1"
-AR Path="/5D7F42FA/83A3164B" Ref="J3"  Part="1"
-F 0 "J3" H 4950 3731 42  0000 L BNN
-F 1 "USB-A-S-X-X-VT" H 4950 2820 42  0000 L BNN
-F 2 "topbreakout:USB-A-S-X-X-VT" H 4750 3600 50  0001 C CNN
-F 3 "" H 4750 3600 50  0001 C CNN
-	1    4750 3600
-	1    0    0    1
 $EndComp
 $Comp
@@
 Wire Wire Line
 	1400 5000 2350 5000
-Wire Wire Line
-	1400 5100 2350 5100
 Text GLabel 1800 6000 2    70   BiDi ~ 0
 GND
@@
 Text GLabel 1600 4400 2    70   BiDi ~ 0
 +3V3
+$Comp
+L TopBreakout-eagle-import:USB-A-S-X-X-VT J3
+U 1 1 83A3164B
+P 4750 3600
+AR Path="/83A3164B" Ref="J3"  Part="1"
+AR Path="/5D7F42FA/83A3164B" Ref="J3"  Part="1"
+F 0 "J3" H 4950 3731 42  0000 L BNN
+F 1 "USB-A-S-X-X-VT" H 4950 2820 42  0000 L BNN
+F 2 "topbreakout:USB-A-S-X-X-VT" H 4750 3600 50  0001 C CNN
+F 3 "" H 4750 3600 50  0001 C CNN
+	1    4750 3600
+	1    0    0    1
+$EndComp
+NoConn ~ 1700 900
+NoConn ~ 1700 1000
+NoConn ~ 2700 2000
+NoConn ~ 2700 2100
+NoConn ~ 2500 2800
+NoConn ~ 2500 2900
+NoConn ~ 1400 2900
+NoConn ~ 1400 2800
+NoConn ~ 4750 3100
+NoConn ~ 4750 3000
+Wire Wire Line
+	1400 5100 2350 5100
 $EndSCHEMATC

Commit message: mainboard v1.7
Parts:
- removed J2: MOLEX_52892-3033MOLEX_52892-3033_0_0, topbreakout:MOLEX_52892-3033_0, symbol TopBreakout-eagle-import:MOLEX_52892-3033MOLEX_52892-3033_0_0
- added J27, J28, J29, J30, J31, J32, J33, J34, J35, J36, J37, J38, J39, J40, J41, J42, J43, J44, J45, J46, J47, J48, J49, J50, J51, J52, J53, J54, J55, J56: Conn_01x01_Female, Connector_PinSocket_2.54mm:PinSocket_1x01_P2.54mm_Vertical, symbol Connector:Conn_01x01_Female
- renumbered J1 to J57, J3 to J58, U$1 to U$2, U$2 to U$3
Connections:
- wire segments 62 -> 63
