File: hardware/boards/topbreakout/io_breakout-ver2.1_5.sch (KiCad schematic (older format))
At the start: 15 parts, among them U1 ANALOG_DEVICES_AD7606BSTZANAL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

Commit message: minor
Parts:
- R10, R4, R7, R8, R9: footprint topbreakout:R0805 -> Resistors_SMD:R_0805
- R11: footprint topbreakout:R0805 -> Oddities:NetTie-I_Connected_SMD
Changed lines of the file:
@@
 Wire Wire Line
 	6700 2800 8500 2800
-Text Label 7300 2800 0    70   ~ 0
-AD_V5
 Wire Wire Line
 	6700 3000 8500 3000
-Text Label 7300 3000 0    70   ~ 0
-AD_V6
 Wire Wire Line
 	6700 3200 8500 3200
-Text Label 7300 3200 0    70   ~ 0
-AD_V7
 Wire Wire Line
 	6700 3400 8500 3400
-Text Label 7400 3400 0    70   ~ 0
-AD_V8
 Wire Wire Line
 	6700 4000 9000 4000
@@
 Wire Wire Line
 	4500 2500 4500 2600
-Text GLabel 4500 2000 2    70   BiDi ~ 0
-GND
-Text GLabel 4500 2100 2    70   BiDi ~ 0
-GND
-Text GLabel 4500 2200 2    70   BiDi ~ 0
+Text GLabel 4500 2000 0    70   BiDi ~ 0
+GND
+Text GLabel 4500 2100 0    70   BiDi ~ 0
+GND
+Text GLabel 4500 2200 0    70   BiDi ~ 0
 GND
 Connection ~ 4500 2100
-Text GLabel 4500 2300 2    70   BiDi ~ 0
+Text GLabel 4500 2300 0    70   BiDi ~ 0
 GND
 Connection ~ 4500 2200
-Text GLabel 4500 2400 2    70   BiDi ~ 0
+Text GLabel 4500 2400 0    70   BiDi ~ 0
 GND
 Connection ~ 4500 2300
-Text GLabel 4500 2500 2    70   BiDi ~ 0
+Text GLabel 4500 2500 0    70   BiDi ~ 0
 GND
 Connection ~ 4500 2400
-Text GLabel 4500 2600 2    70   BiDi ~ 0
+Text GLabel 4500 2600 0    70   BiDi ~ 0
 GND
 Connection ~ 4500 2500
@@
 Wire Wire Line
 	4500 2800 4500 2900
-Text GLabel 4500 2900 2    70   BiDi ~ 0
-GND
-Text GLabel 4500 3000 2    70   BiDi ~ 0
-GND
-Text GLabel 4500 3100 2    70   BiDi ~ 0
+Text GLabel 4500 2900 0    70   BiDi ~ 0
+GND
+Text GLabel 4500 3000 0    70   BiDi ~ 0
+GND
+Text GLabel 4500 3100 0    70   BiDi ~ 0
 GND
 Connection ~ 4500 3000
-Text GLabel 4500 3200 2    70   BiDi ~ 0
+Text GLabel 4500 3200 0    70   BiDi ~ 0
 GND
 Connection ~ 4500 3100
-Text GLabel 4500 3300 2    70   BiDi ~ 0
+Text GLabel 4500 3300 0    70   BiDi ~ 0
 GND
 Connection ~ 4500 3200
-Text GLabel 4500 3400 2    70   BiDi ~ 0
+Text GLabel 4500 3400 0    70   BiDi ~ 0
 GND
 Connection ~ 4500 3300
-Text GLabel 4500 3500 2    70   BiDi ~ 0
+Text GLabel 4500 3500 0    70   BiDi ~ 0
 GND
 Connection ~ 4500 3400
@@
 F 0 "R4" H 3000 4059 59  0000 L BNN
 F 1 "4.7k" H 3000 3870 59  0000 L BNN
-F 2 "topbreakout:R0805" H 3150 4000 50  0001 C CNN
+F 2 "Resistors_SMD:R_0805" H 3150 4000 50  0001 C CNN
 F 3 "" H 3150 4000 50  0001 C CNN
 	1    3150 4000
@@
 F 0 "R7" H 7400 4659 59  0000 L BNN
 F 1 "4.7k" H 7400 4470 59  0000 L BNN
-F 2 "topbreakout:R0805" H 7550 4600 50  0001 C CNN
+F 2 "Resistors_SMD:R_0805" H 7550 4600 50  0001 C CNN
 F 3 "" H 7550 4600 50  0001 C CNN
 	1    7550 4600
@@
 F 0 "R8" H 2500 3659 59  0000 L BNN
 F 1 "4.7k" H 2500 3470 59  0000 L BNN
-F 2 "topbreakout:R0805" H 2650 3600 50  0001 C CNN
+F 2 "Resistors_SMD:R_0805" H 2650 3600 50  0001 C CNN
 F 3 "" H 2650 3600 50  0001 C CNN
 	1    2650 3600
@@
 F 0 "R9" H 3350 3959 59  0000 L BNN
 F 1 "4.7k" H 3350 3770 59  0000 L BNN
-F 2 "topbreakout:R0805" H 3500 3900 50  0001 C CNN
+F 2 "Resistors_SMD:R_0805" H 3500 3900 50  0001 C CNN
 F 3 "" H 3500 3900 50  0001 C CNN
 	1    3500 3900
@@
 F 0 "R10" H 3850 3559 59  0000 L BNN
 F 1 "4.7k" H 3850 3370 59  0000 L BNN
-F 2 "topbreakout:R0805" H 4000 3500 50  0001 C CNN
+F 2 "Resistors_SMD:R_0805" H 4000 3500 50  0001 C CNN
 F 3 "" H 4000 3500 50  0001 C CNN
 	1    4000 3500
@@
 F 0 "R11" H 6950 6000 42  0000 L BNN
 F 1 "0" H 6950 5850 42  0000 L BNN
-F 2 "topbreakout:R0805" H 7100 5950 50  0001 C CNN
+F 2 "Oddities:NetTie-I_Connected_SMD" H 7100 5950 50  0001 C CNN
 F 3 "" H 7100 5950 50  0001 C CNN
 	1    7100 5950
@@
 Wire Wire Line
 	2150 5400 4900 5400
+Text GLabel 7300 2800 0    70   Input ~ 0
+AD_V5
+Text GLabel 7300 3000 0    70   Input ~ 0
+AD_V6
+Text GLabel 7300 3200 0    70   Input ~ 0
+AD_V7
+Text GLabel 7400 3400 0    70   Input ~ 0
+AD_V8
 $EndSCHEMATC

Commit message: routed, ERC checks success
Connections:
- net labels removed: AGND
Changed lines of the file:
@@
 Wire Wire Line
 	6700 2000 8500 2000
-Text GLabel 7300 2000 2    70   BiDi ~ 0
+Text GLabel 8500 2000 2    70   BiDi ~ 0
 AD_V1
 Wire Wire Line
 	6700 2200 8500 2200
-Text GLabel 7300 2200 2    70   BiDi ~ 0
+Text GLabel 8500 2200 2    70   BiDi ~ 0
 AD_V2
 Wire Wire Line
 	6700 2400 8500 2400
-Text GLabel 7300 2400 2    70   BiDi ~ 0
+Text GLabel 8500 2400 2    70   BiDi ~ 0
 AD_V3
 Wire Wire Line
 	6700 2600 8500 2600
-Text GLabel 7300 2600 2    70   BiDi ~ 0
+Text GLabel 8500 2600 2    70   BiDi ~ 0
 AD_V4
 Wire Wire Line
@@
 Connection ~ 3150 3300
 Wire Wire Line
-	7750 4600 8100 4600
-Text GLabel 7750 4600 2    70   BiDi ~ 0
+	7750 4600 7850 4600
+Text GLabel 7850 4600 2    70   BiDi ~ 0
 3V3
 Text GLabel 4600 5400 2    70   BiDi ~ 0
@@
 	9000 4400 9550 4400
 Connection ~ 9000 4400
-Text Label 9550 4400 0    70   ~ 0
-AGND
+Text Label 9550 4400 0    59   ~ 0
+AD_AGND
 Wire Wire Line
 	8350 4600 8350 4800
-Text Label 8350 4800 0    70   ~ 0
-AGND
+Text Label 8350 4800 0    59   ~ 0
+AD_AGND
 $Comp
 L TopBreakout-eagle-import:ANALOG_DEVICES_AD7606BSTZANALOG_DEVICES_AD7606BSTZ_0_2 U1
@@
 Wire Wire Line
 	2150 5400 4900 5400
-Text GLabel 7300 2800 0    70   Input ~ 0
+Text GLabel 8500 2800 2    70   Input ~ 0
 AD_V5
-Text GLabel 7300 3000 0    70   Input ~ 0
+Text GLabel 8500 3000 2    70   Input ~ 0
 AD_V6
-Text GLabel 7300 3200 0    70   Input ~ 0
+Text GLabel 8500 3200 2    70   Input ~ 0
 AD_V7
-Text GLabel 7400 3400 0    70   Input ~ 0
+Text GLabel 8500 3400 2    70   Input ~ 0
 AD_V8
 $EndSCHEMATC

Commit message: revision 1.4 changes
Parts:
- C5, C7, C8: footprint topbreakout:1206 -> Capacitor_SMD:C_0805_2012Metric
- R11: footprint Oddities:NetTie-I_Connected_SMD -> Mainboard:NetTie-I_Connected_SMD_small
Connections:
- net 3V3 renamed +3V3
Changed lines of the file:
@@
-EESchema Schematic File Version 4
-LIBS:TopBreakout-cache
+EESchema Schematic File Version 5
 EELAYER 30 0
 EELAYER END
@@
 Comment3 ""
 Comment4 ""
+Comment5 ""
+Comment6 ""
+Comment7 ""
+Comment8 ""
+Comment9 ""
 $EndDescr
 Text Label 4400 3700 0    70   ~ 0
@@
 	2650 3300 3150 3300
 Text GLabel 3500 3300 2    70   BiDi ~ 0
-3V3
++3V3
 Connection ~ 3500 3300
 Connection ~ 3150 3300
@@
 	7750 4600 7850 4600
 Text GLabel 7850 4600 2    70   BiDi ~ 0
-3V3
-Text GLabel 4600 5400 2    70   BiDi ~ 0
-3V3
-Text GLabel 4600 5400 2    70   BiDi ~ 0
-3V3
++3V3
 Text GLabel 2200 5400 0    70   BiDi ~ 0
-3V3
++3V3
 Wire Wire Line
 	3200 5800 3200 6100
@@
 	4000 6000 4000 6100
 Connection ~ 3600 6100
-Text GLabel 3200 5800 2    70   BiDi ~ 0
-GND
 Connection ~ 4000 6100
 Wire Wire Line
@@
 Wire Wire Line
 	7100 6100 7100 6350
-Text GLabel 7100 6350 2    70   BiDi ~ 0
-GND
 Wire Wire Line
 	3200 5500 4900 5500
@@
 F 0 "C5" H 9060 4315 70  0000 L BNN
 F 1 "1.0uF" H 9060 4115 70  0000 L BNN
-F 2 "topbreakout:1206" H 9000 4200 50  0001 C CNN
+F 2 "Capacitor_SMD:C_0805_2012Metric" H 9000 4200 50  0001 C CNN
 F 3 "" H 9000 4200 50  0001 C CNN
 	1    9000 4200
@@
 F 0 "C7" H 8660 4415 70  0000 L BNN
 F 1 "1.0uF" H 8660 4215 70  0000 L BNN
-F 2 "topbreakout:1206" H 8600 4300 50  0001 C CNN
+F 2 "Capacitor_SMD:C_0805_2012Metric" H 8600 4300 50  0001 C CNN
 F 3 "" H 8600 4300 50  0001 C CNN
 	1    8600 4300
@@
 F 0 "C8" H 8410 4615 70  0000 L BNN
 F 1 "10uF" H 8360 4415 70  0000 L BNN
-F 2 "topbreakout:1206" H 8350 4500 50  0001 C CNN
+F 2 "Capacitor_SMD:C_0805_2012Metric" H 8350 4500 50  0001 C CNN
 F 3 "" H 8350 4500 50  0001 C CNN
 	1    8350 4500
@@
 F 0 "R11" H 6950 6000 42  0000 L BNN
 F 1 "0" H 6950 5850 42  0000 L BNN
-F 2 "Oddities:NetTie-I_Connected_SMD" H 7100 5950 50  0001 C CNN
+F 2 "Mainboard:NetTie-I_Connected_SMD_small" H 7100 5950 50  0001 C CNN
 F 3 "" H 7100 5950 50  0001 C CNN
 	1    7100 5950
@@
 Text GLabel 8500 3400 2    70   Input ~ 0
 AD_V8
+$Comp
+L power:GND #PWR0107
+U 1 1 5DB92978
+P 3600 6100
+F 0 "#PWR0107" H 3600 5850 50  0001 C CNN
+F 1 "GND" H 3605 5927 50  0000 C CNN
+F 2 "" H 3600 6100 50  0001 C CNN
+F 3 "" H 3600 6100 50  0001 C CNN
+	1    3600 6100
+	1    0    0    -1
+$EndComp
+$Comp
+L power:GND #PWR0108
+U 1 1 5DB98F82
+P 7100 6350
+F 0 "#PWR0108" H 7100 6100 50  0001 C CNN
+F 1 "GND" H 7105 6177 50  0000 C CNN
+F 2 "" H 7100 6350 50  0001 C CNN
+F 3 "" H 7100 6350 50  0001 C CNN
+	1    7100 6350
+	1    0    0    -1
+$EndComp
 $EndSCHEMATC

Commit message: TopBreakout: v1.6
Parts:
- added TP2, TP4, TP5, TP6, TP7, TP8, TP9: TEST-POINT3X5, topbreakout:PAD.03X.05, symbol TopBreakout-eagle-import:TEST-POINT3X5
Connections:
- net +3V3: now also TP4.P$1 (1)
- net AD_CONVST: now also TP6.P$1 (1)
- net AD_CS: now also TP2.P$1 (1)
- net AD_REFINOUT: now also TP9.P$1 (1)
- net AD_RESET: now also TP7.P$1 (1)
- net SPI0_MISO: now also TP5.P$1 (1)
- net SPI0_SCK: now also TP8.P$1 (1)
- no-connect marks 0 -> 1
Changed lines of the file:
@@
 Text GLabel 3100 5000 0    70   BiDi ~ 0
-AD_CONVST
-Text GLabel 4200 4900 2    70   BiDi ~ 0
 AD_CONVST
 Wire Wire Line
@@
 AD_RESET
 Wire Wire Line
-	4900 4300 1300 4300
-Text GLabel 4400 4300 2    70   BiDi ~ 0
-SPI0_SCK
-Text GLabel 1300 4300 0    70   BiDi ~ 0
-SPI0_SCK
+	4900 4300 3950 4300
 Wire Wire Line
 	4900 4400 2300 4400
-Text GLabel 4000 4400 2    70   BiDi ~ 0
-AD_CS
-Text GLabel 4000 4400 2    70   BiDi ~ 0
-AD_CS
-Text GLabel 4000 4400 2    70   BiDi ~ 0
-AD_CS
 Text GLabel 2300 4400 0    70   BiDi ~ 0
 AD_CS
@@
 Text GLabel 4300 5100 0    70   BiDi ~ 0
 AD_BUSY
-Wire Wire Line
-	4900 2700 4500 2700
-Text GLabel 4500 2700 0    70   BiDi ~ 0
+Text GLabel 2950 2700 0    70   BiDi ~ 0
 SPI0_MISO
 Wire Wire Line
@@
 Wire Wire Line
 	2650 3300 3150 3300
-Text GLabel 3500 3300 2    70   BiDi ~ 0
+Text GLabel 3500 3300 1    70   BiDi ~ 0
 +3V3
 Connection ~ 3500 3300
@@
 Text GLabel 7850 4600 2    70   BiDi ~ 0
 +3V3
-Text GLabel 2200 5400 0    70   BiDi ~ 0
-+3V3
 Wire Wire Line
 	3200 5800 3200 6100
@@
 Wire Wire Line
 	4900 3800 4050 3800
-Text GLabel 4400 3900 2    70   BiDi ~ 0
-GND
-Text GLabel 4500 3800 2    70   BiDi ~ 0
+Text GLabel 4050 3800 0    70   BiDi ~ 0
 GND
 Wire Wire Line
@@
 Wire Wire Line
 	8000 3300 8000 3500
-Text Label 8000 2100 0    70   ~ 0
-AD_AGND
 Connection ~ 8000 2300
 Connection ~ 8000 2500
@@
 AR Path="/5D7F4383/5459D6DE" Ref="TP1"  Part="1"
 F 0 "TP1" H 1300 5600 70  0001 L BNN
-F 1 "TEST-POINT3X5" V 1300 5500 70  0000 R TNN
+F 1 "TEST-POINT3X5" V 1300 5500 70  0001 R TNN
 F 2 "topbreakout:PAD.03X.05" H 1400 5500 50  0001 C CNN
 F 3 "" H 1400 5500 50  0001 C CNN
@@
 Wire Wire Line
 	4000 3700 4900 3700
-Wire Wire Line
-	2150 5400 4900 5400
 Text GLabel 8500 2800 2    70   Input ~ 0
 AD_V5
@@
 	1    0    0    -1
 $EndComp
+Text GLabel 8000 2100 2    70   Input ~ 0
+AD_AGND
+Text GLabel 3950 4300 0    70   BiDi ~ 0
+SPI0_SCK
+$Comp
+L TopBreakout-eagle-import:TEST-POINT3X5 TP?
+U 1 1 5E007168
+P 7300 4800
+AR Path="/5E007168" Ref="TP?"  Part="1"
+AR Path="/5D7F4383/5E007168" Ref="TP9"  Part="1"
+F 0 "TP9" H 7200 4900 70  0001 L BNN
+F 1 "TEST-POINT3X5" V 7200 4800 70  0001 R TNN
+F 2 "topbreakout:PAD.03X.05" H 7300 4800 50  0001 C CNN
+F 3 "" H 7300 4800 50  0001 C CNN
+	1    7300 4800
+	1    0    0    -1
+$EndComp
+NoConn ~ 4900 5200
+$Comp
+L TopBreakout-eagle-import:TEST-POINT3X5 TP?
+U 1 1 5E012602
+P 2950 2700
+AR Path="/5E012602" Ref="TP?"  Part="1"
+AR Path="/5D7F4383/5E012602" Ref="TP5"  Part="1"
+F 0 "TP5" H 2850 2800 70  0001 L BNN
+F 1 "TEST-POINT3X5" V 2850 2700 70  0001 R TNN
+F 2 "topbreakout:PAD.03X.05" H 2950 2700 50  0001 C CNN
+F 3 "" H 2950 2700 50  0001 C CNN
+	1    2950 2700
+	0    -1   -1   0
+$EndComp
+Wire Wire Line
+	2950 2700 4900 2700
+$Comp
+L TopBreakout-eagle-import:TEST-POINT3X5 TP?
+U 1 1 5E01E21D
+P 2300 4400
+AR Path="/5E01E21D" Ref="TP?"  Part="1"
+AR Path="/5D7F4383/5E01E21D" Ref="TP2"  Part="1"
+F 0 "TP2" H 2200 4500 70  0001 L BNN
+F 1 "TEST-POINT3X5" V 2200 4400 70  0001 R TNN
+F 2 "topbreakout:PAD.03X.05" H 2300 4400 50  0001 C CNN
+F 3 "" H 2300 4400 50  0001 C CNN
+	1    2300 4400
+	0    -1   -1   0
+$EndComp
+$Comp
+L TopBreakout-eagle-import:TEST-POINT3X5 TP?
+U 1 1 5E020685
+P 3700 4700
+AR Path="/5E020685" Ref="TP?"  Part="1"
+AR Path="/5D7F4383/5E020685" Ref="TP7"  Part="1"
+F 0 "TP7" H 3600 4800 70  0001 L BNN
+F 1 "TEST-POINT3X5" V 3600 4700 70  0001 R TNN
+F 2 "topbreakout:PAD.03X.05" H 3700 4700 50  0001 C CNN
+F 3 "" H 3700 4700 50  0001 C CNN
+	1    3700 4700
+	0    -1   -1   0
+$EndComp
+$Comp
+L TopBreakout-eagle-import:TEST-POINT3X5 TP?
+U 1 1 5E0225F0
+P 3100 5000
+AR Path="/5E0225F0" Ref="TP?"  Part="1"
+AR Path="/5D7F4383/5E0225F0" Ref="TP6"  Part="1"
+F 0 "TP6" H 3000 5100 70  0001 L BNN
+F 1 "TEST-POINT3X5" V 3000 5000 70  0001 R TNN
+F 2 "topbreakout:PAD.03X.05" H 3100 5000 50  0001 C CNN
+F 3 "" H 3100 5000 50  0001 C CNN
+	1    3100 5000
+	0    -1   -1   0
+$EndComp
+Connection ~ 3100 5000
+Text GLabel 2200 5400 0    70   BiDi ~ 0
++3V3
+Wire Wire Line
+	2200 5400 2300 5400
+$Comp
+L TopBreakout-eagle-import:TEST-POINT3X5 TP?
+U 1 1 5E0290F9
+P 2300 5400
+AR Path="/5E0290F9" Ref="TP?"  Part="1"
+AR Path="/5D7F4383/5E0290F9" Ref="TP4"  Part="1"
+F 0 "TP4" H 2200 5500 70  0001 L BNN
+F 1 "TEST-POINT3X5" V 2200 5400 70  0001 R TNN
+F 2 "topbreakout:PAD.03X.05" H 2300 5400 50  0001 C CNN
+F 3 "" H 2300 5400 50  0001 C CNN
+	1    2300 5400
+	0    -1   -1   0
+$EndComp
+Connection ~ 2300 5400
+Wire Wire Line
+	2300 5400 4900 5400
+$Comp
+L TopBreakout-eagle-import:TEST-POINT3X5 TP?
+U 1 1 5E02DC53
+P 3950 4300
+AR Path="/5E02DC53" Ref="TP?"  Part="1"
+AR Path="/5D7F4383/5E02DC53" Ref="TP8"  Part="1"
+F 0 "TP8" H 3850 4400 70  0001 L BNN
+F 1 "TEST-POINT3X5" V 3850 4300 70  0001 R TNN
+F 2 "topbreakout:PAD.03X.05" H 3950 4300 50  0001 C CNN
+F 3 "" H 3950 4300 50  0001 C CNN
+	1    3950 4300
+	0    -1   -1   0
+$EndComp
 $EndSCHEMATC

Commit message: mainboard v1.7
Parts:
- removed TP2, TP4, TP5, TP6, TP7, TP8, TP9: TEST-POINT3X5, topbreakout:PAD.03X.05, symbol TopBreakout-eagle-import:TEST-POINT3X5
- renumbered C1 to C21, C2 to C22, C3 to C23, C4 to C24, C8 to C25, C7 to C26, C5 to C27, R8 to R32, R4 to R33, R9 to R34, R10 to R35, R11 to R36, R7 to R37, U1 to U3
Connections:
- net AVIN renamed VIN
- no-connect marks 1 -> 2
