File: hardware/boards/knobs-controller/knobs_2.sch (KiCad schematic (older format))
At the start: 11 parts, among them U2 MK1_ZERO_AP7215-33YG-13, U3 MK1_ZERO_ATSAMD21G18A-48

Commit message: redo migrate from eagle
Parts:
- C10, C19, C27, C28, C29, C30, C32, C8: footprint KnobsController_v1.1:RESISTOR-NICK_C0805 -> knobs:RESISTOR-NICK_C0805; symbol KnobsController_v1.1-eagle-import:RESISTOR-NICK_C-EUC0805 -> knobs-eagle-import:RESISTOR-NICK_C-EUC0805
- L6: footprint KnobsController_v1.1:MK1_ZERO_0603-1608X90N -> knobs:MK1_ZERO_0603-1608X90N; symbol KnobsController_v1.1-eagle-import:MK1_ZERO_BLM18PG471SN1D -> knobs-eagle-import:MK1_ZERO_BLM18PG471SN1D
- U2: footprint KnobsController_v1.1:MK1_ZERO_SOT150P400X160-3N -> knobs:MK1_ZERO_SOT150P400X160-3N; symbol KnobsController_v1.1-eagle-import:MK1_ZERO_AP7215-33YG-13 -> knobs-eagle-import:MK1_ZERO_AP7215-33YG-13
- U3: footprint KnobsController_v1.1:MK1_ZERO_QFN50P700X700X90-49XN-EPSQ515 -> knobs:MK1_ZERO_QFN50P700X700X90-49XN-EPSQ515; symbol KnobsController_v1.1-eagle-import:MK1_ZERO_ATSAMD21G18A-48 -> knobs-eagle-import:MK1_ZERO_ATSAMD21G18A-48

Commit message: minor cleanup
Parts:
- L6: value MK1_ZERO_BLM18PG471SN1D -> BLM18PG471SN1D
- U2: value MK1_ZERO_AP7215-33YG-13 -> AP7215-33YG-13
- U3: value MK1_ZERO_ATSAMD21G18A-48 -> ATSAMD21G18A-48
Connections:
- removed net GND: C10.2, C19.2, C27.2, C29.2, C30.2, C32.2, C8.2, U2.1 (GND), U3.18 (GND@1), U3.35 (GND@2), U3.42 (GND@3), U3.49 (EP), U3.5 (GNDANA)
- new net: C29.2, U3.35 (GND@2)
- new net: C27.2, C30.2, U3.5 (GNDANA)
- new net: C19.2, U3.18 (GND@1)
- new net: C32.2, U3.42 (GND@3)
Other:
- note removed: "Arturo Guadalupi"

Commit message: routed
Connections:
- net VUSB renamed VIN
Changed lines of the file:
@@
 	4800 4200 4800 4300
-Wire Wire Line
-	7700 1000 7900 1000
-Wire Wire Line
-	7900 1000 7900 1200
-Wire Wire Line
-	7900 1000 7900 900
-Connection ~ 7900 1000
 Wire Wire Line
 	4200 4900 4200 4800
@@
 Connection ~ 4200 4800
 Connection ~ 4800 4800
-Wire Wire Line
-	6400 1200 6400 1000
-Wire Wire Line
-	6400 1000 6400 900
-Wire Wire Line
-	6400 900  6200 900
-Wire Wire Line
-	6700 1000 6400 1000
-Connection ~ 6400 1000
-Text GLabel 6200 900  0    70   BiDi ~ 0
-VUSB
 $Comp
 L knobs-eagle-import:MK1_ZERO_ATSAMD21G18A-48 U3
@@
 $EndComp
 $Comp
-L power:+3V3 #PWR?
+L power:+3V3 #PWR0115
 U 1 1 5D87F590
 P 4200 3800
-F 0 "#PWR?" H 4200 3650 50  0001 C CNN
+F 0 "#PWR0115" H 4200 3650 50  0001 C CNN
 F 1 "+3V3" H 4215 3973 50  0000 C CNN
 F 2 "" H 4200 3800 50  0001 C CNN
@@
 $EndComp
 $Comp
-L power:+3V3 #PWR?
+L power:+3V3 #PWR0116
 U 1 1 5D8806AC
 P 4800 4200
-F 0 "#PWR?" H 4800 4050 50  0001 C CNN
+F 0 "#PWR0116" H 4800 4050 50  0001 C CNN
 F 1 "+3V3" H 4815 4373 50  0000 C CNN
 F 2 "" H 4800 4200 50  0001 C CNN
@@
 $EndComp
 $Comp
-L power:+3V3 #PWR?
+L power:+3V3 #PWR0117
 U 1 1 5D880E3E
 P 2600 3800
-F 0 "#PWR?" H 2600 3650 50  0001 C CNN
+F 0 "#PWR0117" H 2600 3650 50  0001 C CNN
 F 1 "+3V3" H 2615 3973 50  0000 C CNN
 F 2 "" H 2600 3800 50  0001 C CNN
@@
 $EndComp
 $Comp
-L power:+3V3 #PWR?
+L power:+3V3 #PWR0118
 U 1 1 5D88183D
 P 7900 900
-F 0 "#PWR?" H 7900 750 50  0001 C CNN
+F 0 "#PWR0118" H 7900 750 50  0001 C CNN
 F 1 "+3V3" H 7915 1073 50  0000 C CNN
 F 2 "" H 7900 900 50  0001 C CNN
@@
 $EndComp
 $Comp
-L knobs-eagle-import:GND #GND?
+L knobs-eagle-import:GND #GND0101
 U 1 1 5D883034
 P 2600 4500
-F 0 "#GND?" H 2600 4500 50  0001 C CNN
+F 0 "#GND0101" H 2600 4500 50  0001 C CNN
 F 1 "GND" H 2600 4379 59  0000 C CNN
 F 2 "" H 2600 4500 50  0001 C CNN
@@
 	2600 5300 2600 5200
 $Comp
-L knobs-eagle-import:GND #GND?
+L knobs-eagle-import:GND #GND0102
 U 1 1 5D883C4A
 P 2600 5400
-F 0 "#GND?" H 2600 5400 50  0001 C CNN
+F 0 "#GND0102" H 2600 5400 50  0001 C CNN
 F 1 "GND" H 2600 5279 59  0000 C CNN
 F 2 "" H 2600 5400 50  0001 C CNN
@@
 $EndComp
 $Comp
-L knobs-eagle-import:GND #GND?
+L knobs-eagle-import:GND #GND0103
 U 1 1 5D8841C2
 P 2600 6200
-F 0 "#GND?" H 2600 6200 50  0001 C CNN
+F 0 "#GND0103" H 2600 6200 50  0001 C CNN
 F 1 "GND" H 2600 6079 59  0000 C CNN
 F 2 "" H 2600 6200 50  0001 C CNN
@@
 $EndComp
 $Comp
-L knobs-eagle-import:GND #GND?
+L knobs-eagle-import:GND #GND0104
 U 1 1 5D884790
 P 4200 5900
-F 0 "#GND?" H 4200 5900 50  0001 C CNN
+F 0 "#GND0104" H 4200 5900 50  0001 C CNN
 F 1 "GND" H 4200 5779 59  0000 C CNN
 F 2 "" H 4200 5900 50  0001 C CNN
@@
 $EndComp
 $Comp
-L knobs-eagle-import:GND #GND?
+L knobs-eagle-import:GND #GND0105
 U 1 1 5D884C3C
 P 4200 5400
-F 0 "#GND?" H 4200 5400 50  0001 C CNN
+F 0 "#GND0105" H 4200 5400 50  0001 C CNN
 F 1 "GND" H 4200 5279 59  0000 C CNN
 F 2 "" H 4200 5400 50  0001 C CNN
@@
 $EndComp
 $Comp
-L knobs-eagle-import:GND #GND?
+L knobs-eagle-import:GND #GND0106
 U 1 1 5D88525E
 P 4200 4500
-F 0 "#GND?" H 4200 4500 50  0001 C CNN
+F 0 "#GND0106" H 4200 4500 50  0001 C CNN
 F 1 "GND" H 4200 4379 59  0000 C CNN
 F 2 "" H 4200 4500 50  0001 C CNN
@@
 $EndComp
 $Comp
-L knobs-eagle-import:GND #GND?
+L knobs-eagle-import:GND #GND0107
 U 1 1 5D88564F
 P 6400 1700
-F 0 "#GND?" H 6400 1700 50  0001 C CNN
+F 0 "#GND0107" H 6400 1700 50  0001 C CNN
 F 1 "GND" H 6400 1579 59  0000 C CNN
 F 2 "" H 6400 1700 50  0001 C CNN
@@
 $EndComp
 $Comp
-L knobs-eagle-import:GND #GND?
+L knobs-eagle-import:GND #GND0108
 U 1 1 5D885B2E
 P 7200 1700
-F 0 "#GND?" H 7200 1700 50  0001 C CNN
+F 0 "#GND0108" H 7200 1700 50  0001 C CNN
 F 1 "GND" H 7200 1579 59  0000 C CNN
 F 2 "" H 7200 1700 50  0001 C CNN
@@
 $EndComp
 $Comp
-L knobs-eagle-import:GND #GND?
+L knobs-eagle-import:GND #GND0109
 U 1 1 5D885ECA
 P 7900 1700
-F 0 "#GND?" H 7900 1700 50  0001 C CNN
+F 0 "#GND0109" H 7900 1700 50  0001 C CNN
 F 1 "GND" H 7900 1579 59  0000 C CNN
 F 2 "" H 7900 1700 50  0001 C CNN
@@
 	4100 3900 4200 3900
 $Comp
-L power:+3V3 #PWR?
+L power:+3V3 #PWR0119
 U 1 1 5D88CD3D
 P 2350 5600
-F 0 "#PWR?" H 2350 5450 50  0001 C CNN
+F 0 "#PWR0119" H 2350 5450 50  0001 C CNN
 F 1 "+3V3" H 2365 5773 50  0000 C CNN
 F 2 "" H 2350 5600 50  0001 C CNN
@@
 Wire Wire Line
 	2700 4300 2600 4300
+Wire Wire Line
+	7700 1000 7900 1000
+Wire Wire Line
+	7900 1000 7900 900
+Wire Wire Line
+	7900 1000 7900 1200
+Connection ~ 7900 1000
+Wire Wire Line
+	6400 1200 6400 1000
+Wire Wire Line
+	6400 1000 6700 1000
+Text GLabel 6400 1000 0    50   Input ~ 0
+VIN
 $EndSCHEMATC

Commit message: mainboard v1.7
Parts:
- renumbered C19 to C13, C32 to C14, C28 to C15, C29 to C16, C30 to C17, C27 to C18, C8 to C19, C10 to C20, L6 to L2, U3 to U1
Changed lines of the file:
@@
 Connection ~ 4800 4800
 $Comp
-L knobs-eagle-import:MK1_ZERO_ATSAMD21G18A-48 U3
+L knobs-eagle-import:MK1_ZERO_ATSAMD21G18A-48 U?
 U 2 1 5C954573
 P 3400 4800
-AR Path="/5C954573" Ref="U3"  Part="2"
-AR Path="/5D866797/5C954573" Ref="U3"  Part="2"
-F 0 "U3" H 2800 5820 59  0000 L BNN
+AR Path="/5C954573" Ref="U?"  Part="2"
+AR Path="/5D866797/5C954573" Ref="U1"  Part="2"
+F 0 "U1" H 2800 5820 59  0000 L BNN
 F 1 "ATSAMD21G18A-48" H 2800 3780 59  0000 L TNN
 F 2 "knobs:MK1_ZERO_QFN50P700X700X90-49XN-EPSQ515" H 3400 4800 50  0001 C CNN
@@
 $EndComp
 $Comp
-L knobs-eagle-import:RESISTOR-NICK_C-EUC0805 C19
+L knobs-eagle-import:RESISTOR-NICK_C-EUC0805 C?
 U 1 1 FC039302
 P 2600 4100
-AR Path="/FC039302" Ref="C19"  Part="1"
-AR Path="/5D866797/FC039302" Ref="C19"  Part="1"
-F 0 "C19" H 2480 4115 59  0000 R BNN
+AR Path="/FC039302" Ref="C?"  Part="1"
+AR Path="/5D866797/FC039302" Ref="C13"  Part="1"
+F 0 "C13" H 2480 4115 59  0000 R BNN
 F 1 "100nF" H 2480 4085 59  0000 R TNN
 F 2 "knobs:RESISTOR-NICK_C0805" H 2600 4100 50  0001 C CNN
@@
 $EndComp
 $Comp
-L knobs-eagle-import:RESISTOR-NICK_C-EUC0805 C30
+L knobs-eagle-import:RESISTOR-NICK_C-EUC0805 C?
 U 1 1 0E4FA8E4
 P 4200 5000
-AR Path="/0E4FA8E4" Ref="C30"  Part="1"
-AR Path="/5D866797/0E4FA8E4" Ref="C30"  Part="1"
-F 0 "C30" H 4320 5015 59  0000 L BNN
+AR Path="/0E4FA8E4" Ref="C?"  Part="1"
+AR Path="/5D866797/0E4FA8E4" Ref="C17"  Part="1"
+F 0 "C17" H 4320 5015 59  0000 L BNN
 F 1 "100nF" H 4320 4985 59  0000 L TNN
 F 2 "knobs:RESISTOR-NICK_C0805" H 4200 5000 50  0001 C CNN
@@
 $EndComp
 $Comp
-L knobs-eagle-import:RESISTOR-NICK_C-EUC0805 C32
+L knobs-eagle-import:RESISTOR-NICK_C-EUC0805 C?
 U 1 1 7F00266C
 P 2600 5000
-AR Path="/7F00266C" Ref="C32"  Part="1"
-AR Path="/5D866797/7F00266C" Ref="C32"  Part="1"
-F 0 "C32" H 2480 5015 59  0000 R BNN
+AR Path="/7F00266C" Ref="C?"  Part="1"
+AR Path="/5D866797/7F00266C" Ref="C14"  Part="1"
+F 0 "C14" H 2480 5015 59  0000 R BNN
 F 1 "1uF" H 2480 4985 59  0000 R TNN
 F 2 "knobs:RESISTOR-NICK_C0805" H 2600 5000 50  0001 C CNN
@@
 $EndComp
 $Comp
-L knobs-eagle-import:RESISTOR-NICK_C-EUC0805 C28
+L knobs-eagle-import:RESISTOR-NICK_C-EUC0805 C?
 U 1 1 87859B6F
 P 2600 5900
-AR Path="/87859B6F" Ref="C28"  Part="1"
-AR Path="/5D866797/87859B6F" Ref="C28"  Part="1"
-F 0 "C28" H 2480 5915 59  0000 R BNN
+AR Path="/87859B6F" Ref="C?"  Part="1"
+AR Path="/5D866797/87859B6F" Ref="C15"  Part="1"
+F 0 "C15" H 2480 5915 59  0000 R BNN
 F 1 "100nF" H 2480 5885 59  0000 R TNN
 F 2 "knobs:RESISTOR-NICK_C0805" H 2600 5900 50  0001 C CNN
@@
 $EndComp
 $Comp
-L knobs-eagle-import:RESISTOR-NICK_C-EUC0805 C29
+L knobs-eagle-import:RESISTOR-NICK_C-EUC0805 C?
 U 1 1 1E55062F
 P 4200 4100
-AR Path="/1E55062F" Ref="C29"  Part="1"
-AR Path="/5D866797/1E55062F" Ref="C29"  Part="1"
-F 0 "C29" H 4320 4115 59  0000 L BNN
+AR Path="/1E55062F" Ref="C?"  Part="1"
+AR Path="/5D866797/1E55062F" Ref="C16"  Part="1"
+F 0 "C16" H 4320 4115 59  0000 L BNN
 F 1 "100nF" H 4320 4075 59  0000 L TNN
 F 2 "knobs:RESISTOR-NICK_C0805" H 4200 4100 50  0001 C CNN
@@
 $EndComp
 $Comp
-L knobs-eagle-import:RESISTOR-NICK_C-EUC0805 C27
+L knobs-eagle-import:RESISTOR-NICK_C-EUC0805 C?
 U 1 1 26DD9C79
 P 4800 5000
-AR Path="/26DD9C79" Ref="C27"  Part="1"
-AR Path="/5D866797/26DD9C79" Ref="C27"  Part="1"
-F 0 "C27" H 4920 5015 59  0000 L BNN
+AR Path="/26DD9C79" Ref="C?"  Part="1"
+AR Path="/5D866797/26DD9C79" Ref="C18"  Part="1"
+F 0 "C18" H 4920 5015 59  0000 L BNN
 F 1 "4.7uF" H 4920 4985 59  0000 L TNN
 F 2 "knobs:RESISTOR-NICK_C0805" H 4800 5000 50  0001 C CNN
@@
 $EndComp
 $Comp
-L knobs-eagle-import:MK1_ZERO_BLM18PG471SN1D L6
+L knobs-eagle-import:MK1_ZERO_BLM18PG471SN1D L?
 U 1 1 529BA6EE
 P 4800 4500
-AR Path="/529BA6EE" Ref="L6"  Part="1"
-AR Path="/5D866797/529BA6EE" Ref="L6"  Part="1"
-F 0 "L6" V 4780 4600 59  0000 L BNN
+AR Path="/529BA6EE" Ref="L?"  Part="1"
+AR Path="/5D866797/529BA6EE" Ref="L2"  Part="1"
+F 0 "L2" V 4780 4600 59  0000 L BNN
 F 1 "BLM18PG471SN1D" V 4820 4600 59  0000 L TNN
 F 2 "knobs:MK1_ZERO_0603-1608X90N" H 4800 4500 50  0001 C CNN
@@
 $EndComp
 $Comp
-L knobs-eagle-import:RESISTOR-NICK_C-EUC0805 C8
+L knobs-eagle-import:RESISTOR-NICK_C-EUC0805 C?
 U 1 1 049ED488
 P 6400 1300
-AR Path="/049ED488" Ref="C8"  Part="1"
-AR Path="/5D866797/049ED488" Ref="C8"  Part="1"
-F 0 "C8" H 6500 1390 59  0000 L CNN
+AR Path="/049ED488" Ref="C?"  Part="1"
+AR Path="/5D866797/049ED488" Ref="C19"  Part="1"
+F 0 "C19" H 6500 1390 59  0000 L CNN
 F 1 "1uF" H 6500 1300 59  0000 L CNN
 F 2 "knobs:RESISTOR-NICK_C0805" H 6400 1300 50  0001 C CNN
@@
 $EndComp
 $Comp
-L knobs-eagle-import:MK1_ZERO_AP7215-33YG-13 U2
+L knobs-eagle-import:MK1_ZERO_AP7215-33YG-13 U?
 U 1 1 455EE6D3
 P 7200 1100
-AR Path="/455EE6D3" Ref="U2"  Part="1"
+AR Path="/455EE6D3" Ref="U?"  Part="1"
 AR Path="/5D866797/455EE6D3" Ref="U2"  Part="1"
 F 0 "U2" H 6800 1420 59  0000 L BNN
@@
 $EndComp
 $Comp
-L knobs-eagle-import:RESISTOR-NICK_C-EUC0805 C10
+L knobs-eagle-import:RESISTOR-NICK_C-EUC0805 C?
 U 1 1 214B8673
 P 7900 1300
-AR Path="/214B8673" Ref="C10"  Part="1"
-AR Path="/5D866797/214B8673" Ref="C10"  Part="1"
-F 0 "C10" H 8000 1390 59  0000 L CNN
+AR Path="/214B8673" Ref="C?"  Part="1"
+AR Path="/5D866797/214B8673" Ref="C20"  Part="1"
+F 0 "C20" H 8000 1390 59  0000 L CNN
 F 1 "1uF" H 8000 1300 59  0000 L CNN
 F 2 "knobs:RESISTOR-NICK_C0805" H 7900 1300 50  0001 C CNN
@@
 $EndComp
 $Comp
-L power:+3V3 #PWR0115
+L power:+3V3 #PWR018
 U 1 1 5D87F590
 P 4200 3800
-F 0 "#PWR0115" H 4200 3650 50  0001 C CNN
+F 0 "#PWR018" H 4200 3650 50  0001 C CNN
 F 1 "+3V3" H 4215 3973 50  0000 C CNN
 F 2 "" H 4200 3800 50  0001 C CNN
@@
 $EndComp
 $Comp
-L power:+3V3 #PWR0116
+L power:+3V3 #PWR019
 U 1 1 5D8806AC
 P 4800 4200
-F 0 "#PWR0116" H 4800 4050 50  0001 C CNN
+F 0 "#PWR019" H 4800 4050 50  0001 C CNN
 F 1 "+3V3" H 4815 4373 50  0000 C CNN
 F 2 "" H 4800 4200 50  0001 C CNN
@@
 $EndComp
 $Comp
-L power:+3V3 #PWR0117
+L power:+3V3 #PWR017
 U 1 1 5D880E3E
 P 2600 3800
-F 0 "#PWR0117" H 2600 3650 50  0001 C CNN
+F 0 "#PWR017" H 2600 3650 50  0001 C CNN
 F 1 "+3V3" H 2615 3973 50  0000 C CNN
 F 2 "" H 2600 3800 50  0001 C CNN
@@
 $EndComp
 $Comp
-L power:+3V3 #PWR0118
+L power:+3V3 #PWR020
 U 1 1 5D88183D
 P 7900 900
-F 0 "#PWR0118" H 7900 750 50  0001 C CNN
+F 0 "#PWR020" H 7900 750 50  0001 C CNN
 F 1 "+3V3" H 7915 1073 50  0000 C CNN
 F 2 "" H 7900 900 50  0001 C CNN
@@
 $EndComp
 $Comp
-L knobs-eagle-import:GND #GND0101
+L knobs-eagle-import:GND #GND019
 U 1 1 5D883034
 P 2600 4500
-F 0 "#GND0101" H 2600 4500 50  0001 C CNN
+F 0 "#GND019" H 2600 4500 50  0001 C CNN
 F 1 "GND" H 2600 4379 59  0000 C CNN
 F 2 "" H 2600 4500 50  0001 C CNN
@@
 	2600 5300 2600 5200
 $Comp
-L knobs-eagle-import:GND #GND0102
+L knobs-eagle-import:GND #GND020
 U 1 1 5D883C4A
 P 2600 5400
-F 0 "#GND0102" H 2600 5400 50  0001 C CNN
+F 0 "#GND020" H 2600 5400 50  0001 C CNN
 F 1 "GND" H 2600 5279 59  0000 C CNN
 F 2 "" H 2600 5400 50  0001 C CNN
@@
 $EndComp
 $Comp
-L knobs-eagle-import:GND #GND0103
+L knobs-eagle-import:GND #GND021
 U 1 1 5D8841C2
 P 2600 6200
-F 0 "#GND0103" H 2600 6200 50  0001 C CNN
+F 0 "#GND021" H 2600 6200 50  0001 C CNN
 F 1 "GND" H 2600 6079 59  0000 C CNN
 F 2 "" H 2600 6200 50  0001 C CNN
@@
 $EndComp
 $Comp
-L knobs-eagle-import:GND #GND0104
+L knobs-eagle-import:GND #GND024
 U 1 1 5D884790
 P 4200 5900
-F 0 "#GND0104" H 4200 5900 50  0001 C CNN
+F 0 "#GND024" H 4200 5900 50  0001 C CNN
 F 1 "GND" H 4200 5779 59  0000 C CNN
 F 2 "" H 4200 5900 50  0001 C CNN
@@
 $EndComp
 $Comp
-L knobs-eagle-import:GND #GND0105
+L knobs-eagle-import:GND #GND023
 U 1 1 5D884C3C
 P 4200 5400
-F 0 "#GND0105" H 4200 5400 50  0001 C CNN
+F 0 "#GND023" H 4200 5400 50  0001 C CNN
 F 1 "GND" H 4200 5279 59  0000 C CNN
 F 2 "" H 4200 5400 50  0001 C CNN
@@
 $EndComp
 $Comp
-L knobs-eagle-import:GND #GND0106
+L knobs-eagle-import:GND #GND022
 U 1 1 5D88525E
 P 4200 4500
-F 0 "#GND0106" H 4200 4500 50  0001 C CNN
+F 0 "#GND022" H 4200 4500 50  0001 C CNN
 F 1 "GND" H 4200 4379 59  0000 C CNN
 F 2 "" H 4200 4500 50  0001 C CNN
@@
 $EndComp
 $Comp
-L knobs-eagle-import:GND #GND0107
+L knobs-eagle-import:GND #GND025
 U 1 1 5D88564F
 P 6400 1700
-F 0 "#GND0107" H 6400 1700 50  0001 C CNN
+F 0 "#GND025" H 6400 1700 50  0001 C CNN
 F 1 "GND" H 6400 1579 59  0000 C CNN
 F 2 "" H 6400 1700 50  0001 C CNN
@@
 $EndComp
 $Comp
-L knobs-eagle-import:GND #GND0108
+L knobs-eagle-import:GND #GND026
 U 1 1 5D885B2E
 P 7200 1700
-F 0 "#GND0108" H 7200 1700 50  0001 C CNN
+F 0 "#GND026" H 7200 1700 50  0001 C CNN
 F 1 "GND" H 7200 1579 59  0000 C CNN
 F 2 "" H 7200 1700 50  0001 C CNN
@@
 $EndComp
 $Comp
-L knobs-eagle-import:GND #GND0109
+L knobs-eagle-import:GND #GND027
 U 1 1 5D885ECA
 P 7900 1700
-F 0 "#GND0109" H 7900 1700 50  0001 C CNN
+F 0 "#GND027" H 7900 1700 50  0001 C CNN
 F 1 "GND" H 7900 1579 59  0000 C CNN
 F 2 "" H 7900 1700 50  0001 C CNN
@@
 	4100 3900 4200 3900
 $Comp
-L power:+3V3 #PWR0119
+L power:+3V3 #PWR016
 U 1 1 5D88CD3D
 P 2350 5600
-F 0 "#PWR0119" H 2350 5450 50  0001 C CNN
+F 0 "#PWR016" H 2350 5450 50  0001 C CNN
 F 1 "+3V3" H 2365 5773 50  0000 C CNN
 F 2 "" H 2350 5600 50  0001 C CNN
