File: hardware/boards/knobs-controller/knobs_2.sch (KiCad schematic (older format))
At the start: 11 parts, among them U1 ATSAMD21G18A-48, U2 AP7215-33YG-13

Commit message: 1.8 work-in-progress
Parts:
- C13, C14, C15, C16, C17, C18, C19, C20: footprint footprints:RESISTOR-NICK_C0805 -> Capacitor_SMD:C_0805_2012Metric
Changed lines of the file:
@@
 F 0 "C13" H 2480 4115 59  0000 R BNN
 F 1 "100nF" H 2480 4085 59  0000 R TNN
-F 2 "footprints:RESISTOR-NICK_C0805" H 2600 4100 50  0001 C CNN
+F 2 "Capacitor_SMD:C_0805_2012Metric" H 2600 4100 50  0001 C CNN
 F 3 "" H 2600 4100 50  0001 C CNN
 	1    2600 4100
@@
 F 0 "C17" H 4320 5015 59  0000 L BNN
 F 1 "100nF" H 4320 4985 59  0000 L TNN
-F 2 "footprints:RESISTOR-NICK_C0805" H 4200 5000 50  0001 C CNN
+F 2 "Capacitor_SMD:C_0805_2012Metric" H 4200 5000 50  0001 C CNN
 F 3 "" H 4200 5000 50  0001 C CNN
 	1    4200 5000
@@
 F 0 "C14" H 2480 5015 59  0000 R BNN
 F 1 "1uF" H 2480 4985 59  0000 R TNN
-F 2 "footprints:RESISTOR-NICK_C0805" H 2600 5000 50  0001 C CNN
+F 2 "Capacitor_SMD:C_0805_2012Metric" H 2600 5000 50  0001 C CNN
 F 3 "" H 2600 5000 50  0001 C CNN
 	1    2600 5000
@@
 F 0 "C15" H 2480 5915 59  0000 R BNN
 F 1 "100nF" H 2480 5885 59  0000 R TNN
-F 2 "footprints:RESISTOR-NICK_C0805" H 2600 5900 50  0001 C CNN
+F 2 "Capacitor_SMD:C_0805_2012Metric" H 2600 5900 50  0001 C CNN
 F 3 "" H 2600 5900 50  0001 C CNN
 	1    2600 5900
@@
 F 0 "C16" H 4320 4115 59  0000 L BNN
 F 1 "100nF" H 4320 4075 59  0000 L TNN
-F 2 "footprints:RESISTOR-NICK_C0805" H 4200 4100 50  0001 C CNN
+F 2 "Capacitor_SMD:C_0805_2012Metric" H 4200 4100 50  0001 C CNN
 F 3 "" H 4200 4100 50  0001 C CNN
 	1    4200 4100
@@
 F 0 "C18" H 4920 5015 59  0000 L BNN
 F 1 "4.7uF" H 4920 4985 59  0000 L TNN
-F 2 "footprints:RESISTOR-NICK_C0805" H 4800 5000 50  0001 C CNN
+F 2 "Capacitor_SMD:C_0805_2012Metric" H 4800 5000 50  0001 C CNN
 F 3 "" H 4800 5000 50  0001 C CNN
 	1    4800 5000
@@
 F 0 "C19" H 6500 1390 59  0000 L CNN
 F 1 "1uF" H 6500 1300 59  0000 L CNN
-F 2 "footprints:RESISTOR-NICK_C0805" H 6400 1300 50  0001 C CNN
+F 2 "Capacitor_SMD:C_0805_2012Metric" H 6400 1300 50  0001 C CNN
 F 3 "" H 6400 1300 50  0001 C CNN
 F 4 "25V" H 6500 1210 59  0001 L CNN "VOLTAGE"
@@
 F 0 "C20" H 8000 1390 59  0000 L CNN
 F 1 "1uF" H 8000 1300 59  0000 L CNN
-F 2 "footprints:RESISTOR-NICK_C0805" H 7900 1300 50  0001 C CNN
+F 2 "Capacitor_SMD:C_0805_2012Metric" H 7900 1300 50  0001 C CNN
 F 3 "" H 7900 1300 50  0001 C CNN
 F 4 "25V" H 8000 1210 59  0001 L CNN "VOLTAGE"

Commit message: 100nF changed to 0.1uF
Parts:
- C13, C15, C16, C17: value 100nF -> 0.1uF
Changed lines of the file:
@@
 AR Path="/5D866797/FC039302" Ref="C13"  Part="1"
 F 0 "C13" H 2480 4115 59  0000 R BNN
-F 1 "100nF" H 2480 4085 59  0000 R TNN
+F 1 "0.1uF" H 2480 4085 59  0000 R TNN
 F 2 "Capacitor_SMD:C_0805_2012Metric" H 2600 4100 50  0001 C CNN
 F 3 "" H 2600 4100 50  0001 C CNN
@@
 AR Path="/5D866797/0E4FA8E4" Ref="C17"  Part="1"
 F 0 "C17" H 4320 5015 59  0000 L BNN
-F 1 "100nF" H 4320 4985 59  0000 L TNN
+F 1 "0.1uF" H 4320 4985 59  0000 L TNN
 F 2 "Capacitor_SMD:C_0805_2012Metric" H 4200 5000 50  0001 C CNN
 F 3 "" H 4200 5000 50  0001 C CNN
@@
 AR Path="/5D866797/87859B6F" Ref="C15"  Part="1"
 F 0 "C15" H 2480 5915 59  0000 R BNN
-F 1 "100nF" H 2480 5885 59  0000 R TNN
+F 1 "0.1uF" H 2480 5885 59  0000 R TNN
 F 2 "Capacitor_SMD:C_0805_2012Metric" H 2600 5900 50  0001 C CNN
 F 3 "" H 2600 5900 50  0001 C CNN
@@
 AR Path="/5D866797/1E55062F" Ref="C16"  Part="1"
 F 0 "C16" H 4320 4115 59  0000 L BNN
-F 1 "100nF" H 4320 4075 59  0000 L TNN
+F 1 "0.1uF" H 4320 4075 59  0000 L TNN
 F 2 "Capacitor_SMD:C_0805_2012Metric" H 4200 4100 50  0001 C CNN
 F 3 "" H 4200 4100 50  0001 C CNN

Commit message: changed c6 to 0805, updates to footprints to simplify BOM
Parts:
- C13, C14, C15, C16, C17, C18, C19, C20: symbol knobs-eagle-import:RESISTOR-NICK_C-EUC0805 -> knobs-eagle-import:C-EUC0805
Changed lines of the file:
@@
 $EndComp
 $Comp
-L knobs-eagle-import:RESISTOR-NICK_C-EUC0805 C?
+L knobs-eagle-import:C-EUC0805 C?
 U 1 1 FC039302
 P 2600 4100
@@
 $EndComp
 $Comp
-L knobs-eagle-import:RESISTOR-NICK_C-EUC0805 C?
+L knobs-eagle-import:C-EUC0805 C?
 U 1 1 0E4FA8E4
 P 4200 5000
@@
 $EndComp
 $Comp
-L knobs-eagle-import:RESISTOR-NICK_C-EUC0805 C?
+L knobs-eagle-import:C-EUC0805 C?
 U 1 1 7F00266C
 P 2600 5000
@@
 $EndComp
 $Comp
-L knobs-eagle-import:RESISTOR-NICK_C-EUC0805 C?
+L knobs-eagle-import:C-EUC0805 C?
 U 1 1 87859B6F
 P 2600 5900
@@
 $EndComp
 $Comp
-L knobs-eagle-import:RESISTOR-NICK_C-EUC0805 C?
+L knobs-eagle-import:C-EUC0805 C?
 U 1 1 1E55062F
 P 4200 4100
@@
 $EndComp
 $Comp
-L knobs-eagle-import:RESISTOR-NICK_C-EUC0805 C?
+L knobs-eagle-import:C-EUC0805 C?
 U 1 1 26DD9C79
 P 4800 5000
@@
 $EndComp
 $Comp
-L knobs-eagle-import:RESISTOR-NICK_C-EUC0805 C?
+L knobs-eagle-import:C-EUC0805 C?
 U 1 1 049ED488
 P 6400 1300
@@
 $EndComp
 $Comp
-L knobs-eagle-import:RESISTOR-NICK_C-EUC0805 C?
+L knobs-eagle-import:C-EUC0805 C?
 U 1 1 214B8673
 P 7900 1300
