File: hardware/boards/knobs-controller/MIDI.sch (KiCad schematic (older format))
At the start: 8 parts

Commit message: 1.8 work-in-progress
Connections:
- net MIDI_IN_PIN4: now also R39.1; no longer D3.2 (A), U$4.3 (C)
- net MIDI_IN_PIN5: now also D3.2 (A), U$4.3 (C); no longer R39.1
- net MIDI_OUT_PIN4: now also R38.1; no longer R40.1
- net MIDI_OUT_PIN5: now also R40.1; no longer R38.1
Changed lines of the file:
@@
 Connection ~ 6000 3700
 Text GLabel 4800 3700 0    70   BiDi ~ 0
-MIDI_IN_PIN4
+MIDI_IN_PIN5
 Wire Wire Line
 	6000 5500 6500 5500
@@
 	5500 5300 4500 5300
 Text GLabel 4500 5300 0    70   BiDi ~ 0
-MIDI_OUT_PIN5
+MIDI_OUT_PIN4
 Wire Wire Line
 	5600 5500 4500 5500
 Text GLabel 4500 5500 0    70   BiDi ~ 0
-MIDI_OUT_PIN4
+MIDI_OUT_PIN5
 Wire Wire Line
 	5500 3300 4800 3300
 Text GLabel 4800 3300 0    70   BiDi ~ 0
-MIDI_IN_PIN5
+MIDI_IN_PIN4
 $Comp
 L Mainboard-eagle-import:R-US_R0805 R?
