File: hardware/boards/knobs-controller/io_breakout-ver2.1_6.sch (KiCad schematic (older format))
At the start: 8 parts, among them U4 ANALOG_DEVICES_AD5754BREZANAL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, U5 MICROCHIP_MCP1700T-2502E-TTMI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

Commit message: changed c6 to 0805, updates to footprints to simplify BOM
Parts:
- C28, C29: footprint Capacitors_SMD:C_0805 -> Capacitor_SMD:C_0805_2012Metric; symbol TopBreakout-eagle-import:C-EUC1206 -> knobs-eagle-import:C-EUC0805
- C30, C31: symbol TopBreakout-eagle-import:C-EUC1206 -> knobs-eagle-import:C-EUC0805
Changed lines of the file:
@@
 $EndComp
 $Comp
-L TopBreakout-eagle-import:C-EUC1206 C?
+L knobs-eagle-import:C-EUC0805 C?
 U 1 1 FDFA29AC
 P 7800 2300
@@
 $EndComp
 $Comp
-L TopBreakout-eagle-import:C-EUC1206 C?
+L knobs-eagle-import:C-EUC0805 C?
 U 1 1 5BE03534
 P 8300 2300
@@
 $EndComp
 $Comp
-L TopBreakout-eagle-import:C-EUC1206 C?
+L knobs-eagle-import:C-EUC0805 C?
 U 1 1 E5C7F153
 P 2600 2300
@@
 F 0 "C28" V 2400 2250 59  0000 C CNN
 F 1 "0.1uF" V 2750 2250 59  0000 C CNN
-F 2 "Capacitors_SMD:C_0805" H 2600 2300 50  0001 C CNN
+F 2 "Capacitor_SMD:C_0805_2012Metric" H 2600 2300 50  0001 C CNN
 F 3 "" H 2600 2300 50  0001 C CNN
 	1    2600 2300
@@
 $EndComp
 $Comp
-L TopBreakout-eagle-import:C-EUC1206 C?
+L knobs-eagle-import:C-EUC0805 C?
 U 1 1 608006B0
 P 3100 2300
@@
 F 0 "C29" V 2950 2250 59  0000 C CNN
 F 1 "0.1uF" V 3250 2250 59  0000 C CNN
-F 2 "Capacitors_SMD:C_0805" H 3100 2300 50  0001 C CNN
+F 2 "Capacitor_SMD:C_0805_2012Metric" H 3100 2300 50  0001 C CNN
 F 3 "" H 3100 2300 50  0001 C CNN
 	1    3100 2300
