File: hardware/boards/mainboard/Audio-in.sch (KiCad schematic (older format))
At the start: 9 parts

Commit message: mainboard 1.8.1 cleanup
Parts:
- C27, C28, C29, C30: footprint Capacitors_SMD:C_0805_HandSoldering -> Capacitor_SMD:C_0805_2012Metric_Pad1.15x1.40mm_HandSolder; symbol Audio-in-eagle-import:C-EUC0805 -> Mainboard-eagle-import:C-EUC0805K
- R5, R6, R7, R8: footprint Resistors_SMD:R_0805_HandSoldering -> Resistor_SMD:R_0805_2012Metric_Pad1.15x1.40mm_HandSolder
Changed lines of the file:
@@
 $Descr A4 11693 8268
 encoding utf-8
-Sheet 7 12
+Sheet 6 12
 Title ""
 Date ""
@@
 Comment9 ""
 $EndDescr
-Text Label 7900 4450 0    70   ~ 0
-V_IN
-Text Label 7900 4450 0    70   ~ 0
-V_IN
 Wire Wire Line
 	5200 3750 5300 3750
@@
 AR Path="/5D773153/5D7E3898/81A18C18" Ref="R9"  Part="1"
 AR Path="/5D773153/5D7EAAD7/81A18C18" Ref="R13"  Part="1"
-F 0 "R9" H 5050 4009 59  0000 L BNN
+F 0 "R13" H 5050 4009 59  0000 L BNN
 F 1 "100K" H 5050 3820 59  0000 L BNN
-F 2 "Resistors_SMD:R_0805_HandSoldering" H 5200 3950 50  0001 C CNN
+F 2 "Resistor_SMD:R_0805_2012Metric_Pad1.15x1.40mm_HandSolder" H 5200 3950 50  0001 C CNN
 F 3 "" H 5200 3950 50  0001 C CNN
 	1    5200 3950
@@
 AR Path="/5D773153/5D7E3898/9C9FFFCA" Ref="R10"  Part="1"
 AR Path="/5D773153/5D7EAAD7/9C9FFFCA" Ref="R14"  Part="1"
-F 0 "R10" H 5350 3809 59  0000 L BNN
+F 0 "R14" H 5350 3809 59  0000 L BNN
 F 1 "150" H 5350 3620 59  0000 L BNN
-F 2 "Resistors_SMD:R_0805_HandSoldering" H 5500 3750 50  0001 C CNN
+F 2 "Resistor_SMD:R_0805_2012Metric_Pad1.15x1.40mm_HandSolder" H 5500 3750 50  0001 C CNN
 F 3 "" H 5500 3750 50  0001 C CNN
 	1    5500 3750
@@
 $EndComp
 $Comp
-L Audio-in-eagle-import:C-EUC0805 C27
+L Mainboard-eagle-import:C-EUC0805K C27
 U 1 1 4294FF20
 P 6000 3750
@@
 AR Path="/5D773153/5D7E3898/4294FF20" Ref="C31"  Part="1"
 AR Path="/5D773153/5D7EAAD7/4294FF20" Ref="C35"  Part="1"
-F 0 "C31" H 6060 3765 59  0000 L BNN
+F 0 "C35" H 6060 3765 59  0000 L BNN
 F 1 "10uF" H 6060 3565 59  0000 L BNN
-F 2 "Capacitors_SMD:C_0805_HandSoldering" H 6000 3750 50  0001 C CNN
+F 2 "Capacitor_SMD:C_0805_2012Metric_Pad1.15x1.40mm_HandSolder" H 6000 3750 50  0001 C CNN
 F 3 "" H 6000 3750 50  0001 C CNN
 	1    6000 3750
@@
 $EndComp
 $Comp
-L Audio-in-eagle-import:C-EUC0805 C28
+L Mainboard-eagle-import:C-EUC0805K C28
 U 1 1 FB49CEF8
 P 6200 4300
@@
 AR Path="/5D773153/5D7E3898/FB49CEF8" Ref="C32"  Part="1"
 AR Path="/5D773153/5D7EAAD7/FB49CEF8" Ref="C36"  Part="1"
-F 0 "C32" H 6260 4315 59  0000 L BNN
+F 0 "C36" H 6260 4315 59  0000 L BNN
 F 1 "2700pF" H 6260 4115 59  0000 L BNN
-F 2 "Capacitors_SMD:C_0805_HandSoldering" H 6200 4300 50  0001 C CNN
+F 2 "Capacitor_SMD:C_0805_2012Metric_Pad1.15x1.40mm_HandSolder" H 6200 4300 50  0001 C CNN
 F 3 "" H 6200 4300 50  0001 C CNN
 	1    6200 4300
@@
 AR Path="/5D773153/5D7E3898/B915E54E" Ref="R11"  Part="1"
 AR Path="/5D773153/5D7EAAD7/B915E54E" Ref="R15"  Part="1"
-F 0 "R11" H 7350 4309 59  0000 L BNN
+F 0 "R15" H 7350 4309 59  0000 L BNN
 F 1 "100K" H 7350 4120 59  0000 L BNN
-F 2 "Resistors_SMD:R_0805_HandSoldering" H 7500 4250 50  0001 C CNN
+F 2 "Resistor_SMD:R_0805_2012Metric_Pad1.15x1.40mm_HandSolder" H 7500 4250 50  0001 C CNN
 F 3 "" H 7500 4250 50  0001 C CNN
 	1    7500 4250
@@
 AR Path="/5D773153/5D7E3898/3A24EE69" Ref="R12"  Part="1"
 AR Path="/5D773153/5D7EAAD7/3A24EE69" Ref="R16"  Part="1"
-F 0 "R12" H 7650 4109 59  0000 L BNN
+F 0 "R16" H 7650 4109 59  0000 L BNN
 F 1 "150" H 7650 3920 59  0000 L BNN
-F 2 "Resistors_SMD:R_0805_HandSoldering" H 7800 4050 50  0001 C CNN
+F 2 "Resistor_SMD:R_0805_2012Metric_Pad1.15x1.40mm_HandSolder" H 7800 4050 50  0001 C CNN
 F 3 "" H 7800 4050 50  0001 C CNN
 	1    7800 4050
@@
 $EndComp
 $Comp
-L Audio-in-eagle-import:C-EUC0805 C29
+L Mainboard-eagle-import:C-EUC0805K C29
 U 1 1 03B11DE5
 P 8100 4050
@@
 AR Path="/5D773153/5D7E3898/03B11DE5" Ref="C33"  Part="1"
 AR Path="/5D773153/5D7EAAD7/03B11DE5" Ref="C37"  Part="1"
-F 0 "C33" H 8160 4065 59  0000 L BNN
+F 0 "C37" H 8160 4065 59  0000 L BNN
 F 1 "10uF" H 8160 3865 59  0000 L BNN
-F 2 "Capacitors_SMD:C_0805_HandSoldering" H 8100 4050 50  0001 C CNN
+F 2 "Capacitor_SMD:C_0805_2012Metric_Pad1.15x1.40mm_HandSolder" H 8100 4050 50  0001 C CNN
 F 3 "" H 8100 4050 50  0001 C CNN
 	1    8100 4050
@@
 $EndComp
 $Comp
-L Audio-in-eagle-import:C-EUC0805 C30
+L Mainboard-eagle-import:C-EUC0805K C30
 U 1 1 5D940E46
 P 8300 4300
@@
 AR Path="/5D773153/5D7E3898/5D940E46" Ref="C34"  Part="1"
 AR Path="/5D773153/5D7EAAD7/5D940E46" Ref="C38"  Part="1"
-F 0 "C34" H 8360 4315 59  0000 L BNN
+F 0 "C38" H 8360 4315 59  0000 L BNN
 F 1 "2700pF" H 8360 4115 59  0000 L BNN
-F 2 "Capacitors_SMD:C_0805_HandSoldering" H 8300 4300 50  0001 C CNN
+F 2 "Capacitor_SMD:C_0805_2012Metric_Pad1.15x1.40mm_HandSolder" H 8300 4300 50  0001 C CNN
 F 3 "" H 8300 4300 50  0001 C CNN
 	1    8300 4300
@@
 AR Path="/5D773153/5D7E3898/5D940E45" Ref="U$3"  Part="1"
 AR Path="/5D773153/5D7EAAD7/5D940E45" Ref="U$4"  Part="1"
-F 0 "U$3" H 3750 4550 50  0001 C CNN
+F 0 "U$4" H 3750 4550 50  0001 C CNN
 F 1 "ACJS-MV-5" H 3750 4550 50  0001 C CNN
 F 2 "footprints:ACJS-MV5" H 3750 4550 50  0001 C CNN

Commit message: cleanup, silkscreen improvements
Changed lines of the file:
@@
 AR Path="/5D773153/5D7E3898/81A18C18" Ref="R9"  Part="1"
 AR Path="/5D773153/5D7EAAD7/81A18C18" Ref="R13"  Part="1"
-F 0 "R13" H 5050 4009 59  0000 L BNN
+F 0 "R5" H 5050 4009 59  0000 L BNN
 F 1 "100K" H 5050 3820 59  0000 L BNN
 F 2 "Resistor_SMD:R_0805_2012Metric_Pad1.15x1.40mm_HandSolder" H 5200 3950 50  0001 C CNN
@@
 AR Path="/5D773153/5D7E3898/9C9FFFCA" Ref="R10"  Part="1"
 AR Path="/5D773153/5D7EAAD7/9C9FFFCA" Ref="R14"  Part="1"
-F 0 "R14" H 5350 3809 59  0000 L BNN
+F 0 "R6" H 5350 3809 59  0000 L BNN
 F 1 "150" H 5350 3620 59  0000 L BNN
 F 2 "Resistor_SMD:R_0805_2012Metric_Pad1.15x1.40mm_HandSolder" H 5500 3750 50  0001 C CNN
@@
 AR Path="/5D773153/5D7E3898/4294FF20" Ref="C31"  Part="1"
 AR Path="/5D773153/5D7EAAD7/4294FF20" Ref="C35"  Part="1"
-F 0 "C35" H 6060 3765 59  0000 L BNN
+F 0 "C27" H 6060 3765 59  0000 L BNN
 F 1 "10uF" H 6060 3565 59  0000 L BNN
 F 2 "Capacitor_SMD:C_0805_2012Metric_Pad1.15x1.40mm_HandSolder" H 6000 3750 50  0001 C CNN
@@
 AR Path="/5D773153/5D7E3898/FB49CEF8" Ref="C32"  Part="1"
 AR Path="/5D773153/5D7EAAD7/FB49CEF8" Ref="C36"  Part="1"
-F 0 "C36" H 6260 4315 59  0000 L BNN
+F 0 "C28" H 6260 4315 59  0000 L BNN
 F 1 "2700pF" H 6260 4115 59  0000 L BNN
 F 2 "Capacitor_SMD:C_0805_2012Metric_Pad1.15x1.40mm_HandSolder" H 6200 4300 50  0001 C CNN
@@
 AR Path="/5D773153/5D7E3898/B915E54E" Ref="R11"  Part="1"
 AR Path="/5D773153/5D7EAAD7/B915E54E" Ref="R15"  Part="1"
-F 0 "R15" H 7350 4309 59  0000 L BNN
+F 0 "R7" H 7350 4309 59  0000 L BNN
 F 1 "100K" H 7350 4120 59  0000 L BNN
 F 2 "Resistor_SMD:R_0805_2012Metric_Pad1.15x1.40mm_HandSolder" H 7500 4250 50  0001 C CNN
@@
 AR Path="/5D773153/5D7E3898/3A24EE69" Ref="R12"  Part="1"
 AR Path="/5D773153/5D7EAAD7/3A24EE69" Ref="R16"  Part="1"
-F 0 "R16" H 7650 4109 59  0000 L BNN
+F 0 "R8" H 7650 4109 59  0000 L BNN
 F 1 "150" H 7650 3920 59  0000 L BNN
 F 2 "Resistor_SMD:R_0805_2012Metric_Pad1.15x1.40mm_HandSolder" H 7800 4050 50  0001 C CNN
@@
 AR Path="/5D773153/5D7E3898/03B11DE5" Ref="C33"  Part="1"
 AR Path="/5D773153/5D7EAAD7/03B11DE5" Ref="C37"  Part="1"
-F 0 "C37" H 8160 4065 59  0000 L BNN
+F 0 "C29" H 8160 4065 59  0000 L BNN
 F 1 "10uF" H 8160 3865 59  0000 L BNN
 F 2 "Capacitor_SMD:C_0805_2012Metric_Pad1.15x1.40mm_HandSolder" H 8100 4050 50  0001 C CNN
@@
 AR Path="/5D773153/5D7E3898/5D940E46" Ref="C34"  Part="1"
 AR Path="/5D773153/5D7EAAD7/5D940E46" Ref="C38"  Part="1"
-F 0 "C38" H 8360 4315 59  0000 L BNN
+F 0 "C30" H 8360 4315 59  0000 L BNN
 F 1 "2700pF" H 8360 4115 59  0000 L BNN
 F 2 "Capacitor_SMD:C_0805_2012Metric_Pad1.15x1.40mm_HandSolder" H 8300 4300 50  0001 C CNN
@@
 AR Path="/5D773153/5D7E3898/5D940E45" Ref="U$3"  Part="1"
 AR Path="/5D773153/5D7EAAD7/5D940E45" Ref="U$4"  Part="1"
-F 0 "U$4" H 3750 4550 50  0001 C CNN
+F 0 "U$2" H 3750 4550 50  0001 C CNN
 F 1 "ACJS-MV-5" H 3750 4550 50  0001 C CNN
 F 2 "footprints:ACJS-MV5" H 3750 4550 50  0001 C CNN
