File: hardware/boards/mainboard/Audio-out.sch (KiCad schematic (older format))
At the start: 9 parts

Commit message: mainboard
Changed lines of the file:
@@
 $Descr A4 11693 8268
 encoding utf-8
-Sheet 10 13
+Sheet 9 12
 Title ""
 Date ""
@@
 Wire Wire Line
 	5600 4000 5600 4100
-Text Label 4500 4100 0    70   ~ 0
-AGND
 Connection ~ 7000 4100
 Connection ~ 6100 4100
@@
 Wire Wire Line
 	5700 4750 4300 4750
-Text Label 4500 4750 0    70   ~ 0
-AGND
-Wire Wire Line
-	3300 3700 3750 3700
-Text Label 3300 3700 0    70   ~ 0
-LEFT
-Text Label 3300 3700 2    70   ~ 0
-LEFT
 Wire Wire Line
 	4050 3700 4300 3700
@@
 Wire Wire Line
 	3750 4350 3250 4350
-Text Label 3250 4350 2    70   ~ 0
-RIGHT
 Wire Wire Line
 	5700 4450 5700 4350
@@
 AR Path="/5D773153/5D8B335A/E0EA0F9E" Ref="R25"  Part="1"
 AR Path="/5D773153/5D8BB03A/E0EA0F9E" Ref="R29"  Part="1"
-F 0 "R21" H 4150 3959 59  0000 L BNN
+F 0 "R29" H 4150 3959 59  0000 L BNN
 F 1 "10K" H 4150 3770 59  0000 L BNN
 F 2 "Resistors_SMD:R_0805_HandSoldering" H 4300 3900 50  0001 C CNN
@@
 AR Path="/5D773153/5D8B335A/4B69501E" Ref="R27"  Part="1"
 AR Path="/5D773153/5D8BB03A/4B69501E" Ref="R31"  Part="1"
-F 0 "R23" H 4500 3759 59  0000 L BNN
+F 0 "R31" H 4500 3759 59  0000 L BNN
 F 1 "560" H 4500 3570 59  0000 L BNN
 F 2 "Resistors_SMD:R_0805_HandSoldering" H 4650 3700 50  0001 C CNN
@@
 AR Path="/5D773153/5D8B335A/D85E66C8" Ref="R26"  Part="1"
 AR Path="/5D773153/5D8BB03A/D85E66C8" Ref="R30"  Part="1"
-F 0 "R22" H 4150 4609 59  0000 L BNN
+F 0 "R30" H 4150 4609 59  0000 L BNN
 F 1 "10K" H 4150 4420 59  0000 L BNN
 F 2 "Resistors_SMD:R_0805_HandSoldering" H 4300 4550 50  0001 C CNN
@@
 AR Path="/5D773153/5D8B335A/EDD241BD" Ref="R28"  Part="1"
 AR Path="/5D773153/5D8BB03A/EDD241BD" Ref="R32"  Part="1"
-F 0 "R24" H 4500 4409 59  0000 L BNN
+F 0 "R32" H 4500 4409 59  0000 L BNN
 F 1 "560" H 4500 4220 59  0000 L BNN
 F 2 "Resistors_SMD:R_0805_HandSoldering" H 4650 4350 50  0001 C CNN
@@
 AR Path="/5D773153/5D8B335A/6F308249" Ref="J_OUT3"  Part="1"
 AR Path="/5D773153/5D8BB03A/6F308249" Ref="J_OUT4"  Part="1"
-F 0 "J_OUT2" H 7300 3500 50  0001 C CNN
+F 0 "J_OUT4" H 7300 3500 50  0001 C CNN
 F 1 "ACJS-MV-5" H 7300 3500 50  0001 C CNN
 F 2 "Mainboard:ACJS-MV5" H 7300 3500 50  0001 C CNN
@@
 AR Path="/5D773153/5D8B335A/D3DD9420" Ref="C48"  Part="1"
 AR Path="/5D773153/5D8BB03A/D3DD9420" Ref="C52"  Part="1"
-F 0 "C44" H 4010 3715 59  0000 L BNN
+F 0 "C52" H 4010 3715 59  0000 L BNN
 F 1 "4.7uF" H 4010 3515 59  0000 L BNN
 F 2 "Capacitors_SMD:C_0805_HandSoldering" H 3950 3700 50  0001 C CNN
@@
 AR Path="/5D773153/5D8B335A/BAA6A02E" Ref="C47"  Part="1"
 AR Path="/5D773153/5D8BB03A/BAA6A02E" Ref="C51"  Part="1"
-F 0 "C43" H 3910 4365 59  0000 L BNN
+F 0 "C51" H 3910 4365 59  0000 L BNN
 F 1 "4.7uF" H 3910 4165 59  0000 L BNN
 F 2 "Capacitors_SMD:C_0805_HandSoldering" H 3850 4350 50  0001 C CNN
@@
 AR Path="/5D773153/5D8B335A/57CFC50E" Ref="C50"  Part="1"
 AR Path="/5D773153/5D8BB03A/57CFC50E" Ref="C54"  Part="1"
-F 0 "C46" H 5760 4565 59  0000 L BNN
+F 0 "C54" H 5760 4565 59  0000 L BNN
 F 1 "2700pF" H 5760 4365 59  0000 L BNN
 F 2 "Capacitors_SMD:C_0805_HandSoldering" H 5700 4550 50  0001 C CNN
@@
 AR Path="/5D773153/5D8B335A/D3171833" Ref="C49"  Part="1"
 AR Path="/5D773153/5D8BB03A/D3171833" Ref="C53"  Part="1"
-F 0 "C45" H 5660 3815 59  0000 L BNN
+F 0 "C53" H 5660 3815 59  0000 L BNN
 F 1 "2700pF" H 5660 3615 59  0000 L BNN
 F 2 "Capacitors_SMD:C_0805_HandSoldering" H 5600 3800 50  0001 C CNN
@@
 	1    0    0    -1
 $EndComp
+Wire Wire Line
+	3300 3700 3750 3700
+Text HLabel 3300 3700 0    70   Input ~ 0
+LEFT
+Text HLabel 3250 4350 0    70   Input ~ 0
+RIGHT
+Text HLabel 4500 4750 0    70   Input ~ 0
+AGND
+Text HLabel 4500 4100 0    70   Input ~ 0
+AGND
 $EndSCHEMATC

Commit message: mainboard v1.7
Changed lines of the file:
@@
-EESchema Schematic File Version 5
+EESchema Schematic File Version 4
 EELAYER 30 0
 EELAYER END
 $Descr A4 11693 8268
 encoding utf-8
-Sheet 12 12
+Sheet 9 12
 Title ""
 Date ""
@@
 Comment3 ""
 Comment4 ""
-Comment5 ""
-Comment6 ""
-Comment7 ""
-Comment8 ""
-Comment9 ""
 $EndDescr
 Wire Wire Line
@@
 AR Path="/5D773153/5D8B335A/E0EA0F9E" Ref="R25"  Part="1"
 AR Path="/5D773153/5D8BB03A/E0EA0F9E" Ref="R29"  Part="1"
-F 0 "R29" H 4150 3959 59  0000 L BNN
+F 0 "R17" H 4150 3959 59  0000 L BNN
 F 1 "10K" H 4150 3770 59  0000 L BNN
 F 2 "Resistors_SMD:R_0805_HandSoldering" H 4300 3900 50  0001 C CNN
@@
 AR Path="/5D773153/5D8B335A/4B69501E" Ref="R27"  Part="1"
 AR Path="/5D773153/5D8BB03A/4B69501E" Ref="R31"  Part="1"
-F 0 "R31" H 4500 3759 59  0000 L BNN
+F 0 "R19" H 4500 3759 59  0000 L BNN
 F 1 "560" H 4500 3570 59  0000 L BNN
 F 2 "Resistors_SMD:R_0805_HandSoldering" H 4650 3700 50  0001 C CNN
@@
 AR Path="/5D773153/5D8B335A/D85E66C8" Ref="R26"  Part="1"
 AR Path="/5D773153/5D8BB03A/D85E66C8" Ref="R30"  Part="1"
-F 0 "R30" H 4150 4609 59  0000 L BNN
+F 0 "R18" H 4150 4609 59  0000 L BNN
 F 1 "10K" H 4150 4420 59  0000 L BNN
 F 2 "Resistors_SMD:R_0805_HandSoldering" H 4300 4550 50  0001 C CNN
@@
 AR Path="/5D773153/5D8B335A/EDD241BD" Ref="R28"  Part="1"
 AR Path="/5D773153/5D8BB03A/EDD241BD" Ref="R32"  Part="1"
-F 0 "R32" H 4500 4409 59  0000 L BNN
+F 0 "R20" H 4500 4409 59  0000 L BNN
 F 1 "560" H 4500 4220 59  0000 L BNN
 F 2 "Resistors_SMD:R_0805_HandSoldering" H 4650 4350 50  0001 C CNN
@@
 AR Path="/5D773153/5D8B335A/6F308249" Ref="J_OUT3"  Part="1"
 AR Path="/5D773153/5D8BB03A/6F308249" Ref="J_OUT4"  Part="1"
-F 0 "J_OUT4" H 7300 3500 50  0001 C CNN
+F 0 "J_OUT1" H 7300 3500 50  0001 C CNN
 F 1 "ACJS-MV-5" H 7300 3500 50  0001 C CNN
 F 2 "Mainboard:ACJS-MV5" H 7300 3500 50  0001 C CNN
@@
 AR Path="/5D773153/5D8B335A/D3DD9420" Ref="C48"  Part="1"
 AR Path="/5D773153/5D8BB03A/D3DD9420" Ref="C52"  Part="1"
-F 0 "C52" H 4010 3715 59  0000 L BNN
+F 0 "C40" H 4010 3715 59  0000 L BNN
 F 1 "4.7uF" H 4010 3515 59  0000 L BNN
 F 2 "Capacitors_SMD:C_0805_HandSoldering" H 3950 3700 50  0001 C CNN
@@
 AR Path="/5D773153/5D8B335A/BAA6A02E" Ref="C47"  Part="1"
 AR Path="/5D773153/5D8BB03A/BAA6A02E" Ref="C51"  Part="1"
-F 0 "C51" H 3910 4365 59  0000 L BNN
+F 0 "C39" H 3910 4365 59  0000 L BNN
 F 1 "4.7uF" H 3910 4165 59  0000 L BNN
 F 2 "Capacitors_SMD:C_0805_HandSoldering" H 3850 4350 50  0001 C CNN
@@
 AR Path="/5D773153/5D8B335A/57CFC50E" Ref="C50"  Part="1"
 AR Path="/5D773153/5D8BB03A/57CFC50E" Ref="C54"  Part="1"
-F 0 "C54" H 5760 4565 59  0000 L BNN
+F 0 "C42" H 5760 4565 59  0000 L BNN
 F 1 "2700pF" H 5760 4365 59  0000 L BNN
 F 2 "Capacitors_SMD:C_0805_HandSoldering" H 5700 4550 50  0001 C CNN
@@
 AR Path="/5D773153/5D8B335A/D3171833" Ref="C49"  Part="1"
 AR Path="/5D773153/5D8BB03A/D3171833" Ref="C53"  Part="1"
-F 0 "C53" H 5660 3815 59  0000 L BNN
+F 0 "C41" H 5660 3815 59  0000 L BNN
 F 1 "2700pF" H 5660 3615 59  0000 L BNN
 F 2 "Capacitors_SMD:C_0805_HandSoldering" H 5600 3800 50  0001 C CNN
