File: hardware/boards/mainboard/Mainboard.sch (KiCad schematic (older format))
At the start: 0 parts

Commit message: mainboard
Parts:
- added J2: JST---S4B-PH-SM4-TB(LF)(SN)_JST_S4B-PH-SM4-TB_LF_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, knobs:JST---S4B-PH-SM4-TB(LF)(SN)_JST_S4B-PH-SM4-TB_LF_SN_0, symbol knobs-eagle-import:JST---S4B-PH-SM4-TB(LF)(SN)_JST_S4B-PH-SM4-TB_LF_SNJST_S4B-P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
Connections:
- new net GND: J2.1
- new net KC_TEENSY_RX: J2.2
- new net KC_TEENSY_TX: J2.3
- new net VIN: J2.4
- no-connect marks 0 -> 2
Changed lines of the file:
@@
 $Descr A4 11693 8268
 encoding utf-8
-Sheet 1 13
+Sheet 1 12
 Title ""
 Date ""
@@
 F1 "codec.sch" 50
 $EndSheet
-$Sheet
-S 9000 1000 500  150
-U 5D773307
-F0 "Midi" 50
-F1 "Midi.sch" 50
-$EndSheet
+$Comp
+L power:GND #PWR0102
+U 1 1 5D8F3899
+P 6650 3350
+F 0 "#PWR0102" H 6650 3100 50  0001 C CNN
+F 1 "GND" H 6655 3177 50  0000 C CNN
+F 2 "" H 6650 3350 50  0001 C CNN
+F 3 "" H 6650 3350 50  0001 C CNN
+	1    6650 3350
+	1    0    0    -1
+$EndComp
+Wire Wire Line
+	6400 3350 6650 3350
+Text GLabel 6400 3950 2    50   Input ~ 0
+VIN
+Text GLabel 7500 3550 2    70   Output ~ 0
+KC_TEENSY_RX
+Wire Wire Line
+	6400 3550 7500 3550
+Text GLabel 7500 3750 2    70   Input ~ 0
+KC_TEENSY_TX
+$Comp
+L knobs-eagle-import:JST---S4B-PH-SM4-TB(LF)(SN)_JST_S4B-PH-SM4-TB_LF_SNJST_S4B-PH-SM4-TB_LF_SN_0_0 J2
+U 1 1 5D8FCBBF
+P 5600 2950
+F 0 "J2" H 6540 2850 85  0000 C CNN
+F 1 "JST---S4B-PH-SM4-TB(LF)(SN)_JST_S4B-PH-SM4-TB_LF_SNJST_S4B-PH-SM4-TB_LF_SN_0_0" H 5600 2950 50  0001 C CNN
+F 2 "knobs:JST---S4B-PH-SM4-TB(LF)(SN)_JST_S4B-PH-SM4-TB_LF_SN_0" H 5600 2950 50  0001 C CNN
+F 3 "" H 5600 2950 50  0001 C CNN
+	1    5600 2950
+	1    0    0    -1
+$EndComp
+Wire Wire Line
+	6400 3750 7500 3750
+NoConn ~ 6400 4350
+NoConn ~ 6400 4150
 $EndSCHEMATC

Commit message: mainboard v1.7
Parts:
- removed J2: JST---S4B-PH-SM4-TB(LF)(SN)_JST_S4B-PH-SM4-TB_LF_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, knobs:JST---S4B-PH-SM4-TB(LF)(SN)_JST_S4B-PH-SM4-TB_LF_SN_0, symbol knobs-eagle-import:JST---S4B-PH-SM4-TB(LF)(SN)_JST_S4B-PH-SM4-TB_LF_SNJST_S4B-P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
Connections:
- no-connect marks 2 -> 0
Changed lines of the file:
@@
-EESchema Schematic File Version 5
+EESchema Schematic File Version 4
 EELAYER 30 0
 EELAYER END
@@
 Comment3 ""
 Comment4 ""
-Comment5 ""
-Comment6 ""
-Comment7 ""
-Comment8 ""
-Comment9 ""
 $EndDescr
 $Sheet
@@
 F1 "codec.sch" 50
 $EndSheet
-$Comp
-L power:GND #PWR0102
-U 1 1 5D8F3899
-P 6650 3350
-F 0 "#PWR0102" H 6650 3100 50  0001 C CNN
-F 1 "GND" H 6655 3177 50  0000 C CNN
-F 2 "" H 6650 3350 50  0001 C CNN
-F 3 "" H 6650 3350 50  0001 C CNN
-	1    6650 3350
-	1    0    0    -1
-$EndComp
-Wire Wire Line
-	6400 3350 6650 3350
-Text GLabel 6400 3950 2    50   Input ~ 0
-VIN
-Text GLabel 7500 3550 2    70   Output ~ 0
-KC_TEENSY_RX
-Wire Wire Line
-	6400 3550 7500 3550
-Text GLabel 7500 3750 2    70   Input ~ 0
-KC_TEENSY_TX
-$Comp
-L knobs-eagle-import:JST---S4B-PH-SM4-TB(LF)(SN)_JST_S4B-PH-SM4-TB_LF_SNJST_S4B-PH-SM4-TB_LF_SN_0_0 J2
-U 1 1 5D8FCBBF
-P 5600 2950
-F 0 "J2" H 6540 2850 85  0000 C CNN
-F 1 "JST---S4B-PH-SM4-TB(LF)(SN)_JST_S4B-PH-SM4-TB_LF_SNJST_S4B-PH-SM4-TB_LF_SN_0_0" H 5600 2950 50  0001 C CNN
-F 2 "knobs:JST---S4B-PH-SM4-TB(LF)(SN)_JST_S4B-PH-SM4-TB_LF_SN_0" H 5600 2950 50  0001 C CNN
-F 3 "" H 5600 2950 50  0001 C CNN
-	1    5600 2950
-	1    0    0    -1
-$EndComp
-Wire Wire Line
-	6400 3750 7500 3750
-NoConn ~ 6400 4350
-NoConn ~ 6400 4150
 $EndSCHEMATC
