File: hardware/boards/mainboard/kryon-ver2.1-final_2.sch (KiCad schematic (older format))
At the start: 13 parts, among them IC1 LM340?-MP

Commit message: mainboard
Connections:
- net GND: no longer C1.2, C4.2
- net 3V3 renamed +3V3
- new net: C1.2, C4.2
Changed lines of the file:
@@
 $Descr A4 11693 8268
 encoding utf-8
-Sheet 3 13
+Sheet 3 12
 Title ""
 Date ""
@@
 	5600 2400 6100 2400
 Text GLabel 6100 2400 2    70   BiDi ~ 0
-3V3
++3V3
 Wire Wire Line
 	5600 2700 5800 2700
@@
 	5800 2700 6100 2700
 Connection ~ 5800 2700
-Text GLabel 5600 2700 0    10   BiDi ~ 0
-GND
 Wire Wire Line
 	5600 3500 6000 3500

Commit message: mainboard v1.6
Parts:
- added JM1, JM2, JS1, JS2: Conn_01x02_Male, Connector_PinHeader_2.54mm:PinHeader_1x02_P2.54mm_Vertical, symbol Connector:Conn_01x02_Male
- added JP2: PINHD-1X2, Mainboard:1X02, symbol Mainboard-eagle-import:PINHD-1X2
- SV1: footprint Mainboard:EURO_POWER_HEADER -> Connector_PinHeader_2.54mm:PinHeader_2x08_P2.54mm_Vertical
Connections:
- net VIN: now also JP2.2
- net PWR_5V: now reaches SV1.11
- net PWR_5V: now also SV1.12, JP2.1
- net MASTER_TX: now reaches SV1.13
- net MASTER_TX: now also SV1.14, JM2.1 (Pin_1), JS2.1 (Pin_1)
- net MASTER_RX: now reaches SV1.15
- net MASTER_RX: now also SV1.16, JM1.2 (Pin_2), JS1.2 (Pin_2)
- new net BUS_TEENSY_RX: JM1.1 (Pin_1), JS2.2 (Pin_2)
- new net BUS_TEENSY_TX: JM2.2 (Pin_2), JS1.1 (Pin_1)
Other:
- note added: "Master"
- note added: "Slave"
Changed lines of the file:
@@
 	5900 5400 5900 5800
 Wire Wire Line
-	5900 5800 6400 5800
+	5900 5800 6250 5800
 Wire Wire Line
 	5900 5400 6200 5400
@@
 F 0 "SV1" H 3550 4330 59  0000 L BNN
 F 1 "EURO_POWER_HEADERREGULAR" H 3550 3600 59  0000 L BNN
-F 2 "Mainboard:EURO_POWER_HEADER" H 3700 4000 50  0001 C CNN
+F 2 "Connector_PinHeader_2.54mm:PinHeader_2x08_P2.54mm_Vertical" H 3700 4000 50  0001 C CNN
 F 3 "" H 3700 4000 50  0001 C CNN
 	1    3700 4000
@@
 Text GLabel 8100 3900 2    70   Input ~ 0
 AVSS
+Wire Wire Line
+	3400 3600 4000 3600
+Wire Wire Line
+	3400 3500 4000 3500
+$Comp
+L Connector:Conn_01x02_Male JM2
+U 1 1 5DF8E104
+P 3750 2700
+F 0 "JM2" H 3800 2500 50  0000 C CNN
+F 1 "Conn_01x02_Male" H 4050 2400 50  0000 C CNN
+F 2 "Connector_PinHeader_2.54mm:PinHeader_1x02_P2.54mm_Vertical" H 3750 2700 50  0001 C CNN
+F 3 "~" H 3750 2700 50  0001 C CNN
+	1    3750 2700
+	1    0    0    -1
+$EndComp
+$Comp
+L Connector:Conn_01x02_Male JM1
+U 1 1 5DF8F180
+P 3650 2800
+F 0 "JM1" H 3800 2900 50  0000 R CNN
+F 1 "Conn_01x02_Male" H 4300 3000 50  0000 R CNN
+F 2 "Connector_PinHeader_2.54mm:PinHeader_1x02_P2.54mm_Vertical" H 3650 2800 50  0001 C CNN
+F 3 "~" H 3650 2800 50  0001 C CNN
+	1    3650 2800
+	-1   0    0    1
+$EndComp
+$Comp
+L Connector:Conn_01x02_Male JS1
+U 1 1 5DF9340C
+P 3600 2150
+F 0 "JS1" H 3750 2250 50  0000 R CNN
+F 1 "Conn_01x02_Male" H 4250 1900 50  0000 R CNN
+F 2 "Connector_PinHeader_2.54mm:PinHeader_1x02_P2.54mm_Vertical" H 3600 2150 50  0001 C CNN
+F 3 "~" H 3600 2150 50  0001 C CNN
+	1    3600 2150
+	-1   0    0    1
+$EndComp
+Text Label 4000 3600 0    50   ~ 0
+MASTER_TX
+Text Label 4000 3500 0    50   ~ 0
+MASTER_RX
+Text Label 4350 2700 0    50   ~ 0
+MASTER_TX
+Text Label 3450 2700 2    50   ~ 0
+MASTER_RX
+Text Label 4350 2050 0    50   ~ 0
+MASTER_TX
+Text Label 3400 2050 2    50   ~ 0
+MASTER_RX
+Text GLabel 4350 2150 2    50   Input ~ 0
+BUS_TEENSY_RX
+$Comp
+L Connector:Conn_01x02_Male JS2
+U 1 1 5DF97449
+P 3750 2050
+F 0 "JS2" H 3800 1850 50  0000 C CNN
+F 1 "Conn_01x02_Male" H 4100 2200 50  0000 C CNN
+F 2 "Connector_PinHeader_2.54mm:PinHeader_1x02_P2.54mm_Vertical" H 3750 2050 50  0001 C CNN
+F 3 "~" H 3750 2050 50  0001 C CNN
+	1    3750 2050
+	1    0    0    -1
+$EndComp
+Wire Wire Line
+	4350 2150 3950 2150
+Text GLabel 3400 2150 0    50   Input ~ 0
+BUS_TEENSY_TX
+Wire Wire Line
+	3950 2050 4350 2050
+Wire Notes Line
+	2950 1850 5050 1850
+Wire Notes Line
+	5050 1850 5050 2450
+Wire Notes Line
+	5050 2450 2950 2450
+Wire Notes Line
+	2950 1850 2950 2450
+Text Notes 2950 1850 0    50   ~ 0
+Slave
+Text GLabel 3450 2800 0    50   Input ~ 0
+BUS_TEENSY_RX
+Text GLabel 4350 2800 2    50   Input ~ 0
+BUS_TEENSY_TX
+Wire Wire Line
+	3950 2700 4350 2700
+Wire Wire Line
+	4350 2800 3950 2800
+Wire Notes Line
+	5050 2600 5050 3100
+Wire Notes Line
+	5050 3100 3000 3100
+Wire Notes Line
+	3000 3100 3000 2600
+Wire Notes Line
+	3000 2600 5050 2600
+Text Notes 3000 2600 0    50   ~ 0
+Master
+$Comp
+L Mainboard-eagle-import:PINHD-1X2 JP2
+U 1 1 5DFECC19
+P 7050 5400
+F 0 "JP2" H 6800 5625 59  0000 L BNN
+F 1 "PINHD-1X2" H 6800 5100 59  0000 L BNN
+F 2 "Mainboard:1X02" H 7050 5400 50  0001 C CNN
+F 3 "" H 7050 5400 50  0001 C CNN
+	1    7050 5400
+	1    0    0    -1
+$EndComp
+Wire Wire Line
+	6950 5400 6950 5600
+Wire Wire Line
+	6950 5600 6250 5600
+Wire Wire Line
+	6250 5600 6250 5800
+Connection ~ 6250 5800
+Wire Wire Line
+	6250 5800 6400 5800
+Wire Wire Line
+	3400 3700 4000 3700
+Text Label 4000 3700 0    50   ~ 0
+PWR_5V
+Wire Wire Line
+	6950 5300 6600 5300
+Wire Wire Line
+	6600 5300 6600 5250
+Text Label 6600 5250 0    50   ~ 0
+PWR_5V
 $EndSCHEMATC
