File: hardware/boards/teensy-eurorack.sch (KiCad schematic (older format))
At the start: 75 parts, among them J1 Conn_01x08, J11 AudioJack2_SwitchT, J12 AudioJack2_SwitchT, J13 AudioJack2_SwitchT, J14 AudioJack2_SwitchT, J15 AudioJack2_SwitchT, J16 AudioJack2_SwitchT, J17 AudioJack2_SwitchT, J18 AudioJack2_SwitchT, J19 AudioJack2_SwitchT, J2 Conn_02x08_Odd_Even, J20 AudioJack2_SwitchT, J21 AudioJack2_SwitchT, J22 AudioJack2_SwitchT, J23 AudioJack2_SwitchT, J24 AudioJack2_SwitchT, J25 AudioJack2_SwitchT, J26 AudioJack2_SwitchT, J3 Conn_02x08_Odd_Even, U1 CS42448, U2 ANALOG_DEVICES_AD5754BREZANAL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, U3 ANALOG_DEVICES_AD5754BREZANAL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, U4 Teensy4.1, U5 MCP1700-2502E_SOT23, U6 ANALOG_DEVICES_AD7606BSTZANAL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

Commit message: work in progress
Parts:
- added J?: Conn_02x08_Odd_Even, symbol Connector_Generic:Conn_02x08_Odd_Even
- added J?: Conn_01x02, symbol Connector_Generic:Conn_01x02
- added J? (x2): DIN-5, symbol Connector:DIN-5
- added RV? (x4): R_POT, symbol Device:R_POT
- added SW? (x3): Rotary_Encoder_Switch, symbol Device:Rotary_Encoder_Switch
- added U?: 6N138, symbol Isolator:6N138
Connections:
- net +12V: now also J?.10 (Pin_10), J?.9 (Pin_9)
- net +5V: now also U6.37 (2_AVCC), J?.1 (Pin_1)
- net -12V: now also J?.1 (Pin_1), J?.2 (Pin_2)
- net ADC_BUSY: now also U4.5 (3_LRCLK2)
- net ADC_CONVST: now also U4.7 (5_IN2)
- net ADC_CS: now also U4.12 (10_CS_MQSR)
- net DAC_SDOUT: now also U4.33 (41_A1_MIS01)
- net DAC_SYNC: now also U4.38 (16_A2_RX4_SCL1)
- net GND: now also U2.18 (1_DAC_GND), U2.19 (2_DAC_GND), U2.21 (2_SIG_GND), U3.18 (1_DAC_GND), U3.19 (2_DAC_GND), U3.21 (2_SIG_GND), U6.17 (DB1), U6.18 (DB2), U6.19 (DB3), U6.2 (1_AGND), U6.20 (DB4), U6.21 (DB5), U6.26 (2_AGND), U6.27 (DB9), U6.28 (DB10), U6.29 (DB11), U6.30 (DB12), U6.31 (DB13), U6.32 (DB14/HBEN), U6.35 (3_AGND), U6.4 (OS1), U6.40 (4_AGND), U6.41 (5_AGND), U6.46 (2_REFGND)
- net MIDI_RX: now reaches U4.2 (0_RX1_CRX2_CS1)
- net MIDI_TX: now reaches U4.3 (1_TX1_CTX2_MISO1)
- new net: J?.11 (Pin_11), J?.12 (Pin_12), J?.2 (Pin_2)
- new net: J?.3 (Pin_3), J?.5 (Pin_5), J?.7 (Pin_7)
- new net: J?.4 (Pin_4), J?.6 (Pin_6), J?.8 (Pin_8)
Other:
- moved on the sheet: C19, C20, C21, C22, C23, C24, C25, C26, C27, C28, C29, C30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

Commit message: footprints
Parts:
- added J31, J32: Conn_01x20, Connector_PinSocket_2.54mm:PinSocket_1x20_P2.54mm_Vertical, symbol Connector_Generic:Conn_01x20
- added J33, J34: Conn_01x20, Connector_PinHeader_2.54mm:PinHeader_1x20_P2.54mm_Vertical, symbol Connector_Generic:Conn_01x20
- J27: renamed from J?; footprint (none) -> Connector_PinHeader_2.54mm:PinHeader_1x02_P2.54mm_Vertical
- J28: renamed from J?; footprint (none) -> Connector_PinHeader_2.54mm:PinHeader_2x08_P2.54mm_Vertical
- RV1, RV2, RV3, RV4: renamed from RV?; footprint (none) -> footprints:9MM_SNAP-IN_POT
- U7: renamed from U?; footprint (none) -> footprints:6N138S
- gave numbers to parts that had none: 5
Connections:
- new net: J31.20 (Pin_20), J33.20 (Pin_20)
- new net: J32.20 (Pin_20), J34.20 (Pin_20)
Changed lines of the file:
@@
 DAC_SDOUT
 $Comp
-L Connector_Generic:Conn_02x08_Odd_Even J?
+L Connector_Generic:Conn_02x08_Odd_Even J28
 U 1 1 5EE93454
 P 1350 8850
-F 0 "J?" H 1400 9367 50  0000 C CNN
+F 0 "J28" H 1400 9367 50  0000 C CNN
 F 1 "Conn_02x08_Odd_Even" H 1400 9276 50  0000 C CNN
-F 2 "" H 1350 8850 50  0001 C CNN
+F 2 "Connector_PinHeader_2.54mm:PinHeader_2x08_P2.54mm_Vertical" H 1350 8850 50  0001 C CNN
 F 3 "~" H 1350 8850 50  0001 C CNN
 	1    1350 8850
@@
 $EndComp
 $Comp
-L power:-12V #PWR?
+L power:-12V #PWR0101
 U 1 1 5EE9CB27
 P 1800 8550
-F 0 "#PWR?" H 1800 8650 50  0001 C CNN
+F 0 "#PWR0101" H 1800 8650 50  0001 C CNN
 F 1 "-12V" H 1815 8723 50  0000 C CNN
 F 2 "" H 1800 8550 50  0001 C CNN
@@
 $EndComp
 $Comp
-L power:-12V #PWR?
+L power:-12V #PWR0122
 U 1 1 5EE9E974
 P 900 8550
-F 0 "#PWR?" H 900 8650 50  0001 C CNN
+F 0 "#PWR0122" H 900 8650 50  0001 C CNN
 F 1 "-12V" H 915 8723 50  0000 C CNN
 F 2 "" H 900 8550 50  0001 C CNN
@@
 Connection ~ 1650 8750
 $Comp
-L power:+12V #PWR?
+L power:+12V #PWR0123
 U 1 1 5EED4414
 P 900 8950
-F 0 "#PWR?" H 900 8800 50  0001 C CNN
+F 0 "#PWR0123" H 900 8800 50  0001 C CNN
 F 1 "+12V" H 915 9123 50  0000 C CNN
 F 2 "" H 900 8950 50  0001 C CNN
@@
 $EndComp
 $Comp
-L power:+12V #PWR?
+L power:+12V #PWR0124
 U 1 1 5EED521B
 P 1800 8950
-F 0 "#PWR?" H 1800 8800 50  0001 C CNN
+F 0 "#PWR0124" H 1800 8800 50  0001 C CNN
 F 1 "+12V" H 1815 9123 50  0000 C CNN
 F 2 "" H 1800 8950 50  0001 C CNN
@@
 	1150 9050 1650 9050
 $Comp
-L Connector_Generic:Conn_01x02 J?
+L Connector_Generic:Conn_01x02 J27
 U 1 1 5EEEAE16
 P 700 9250
-F 0 "J?" V 572 9062 50  0000 R CNN
+F 0 "J27" V 572 9062 50  0000 R CNN
 F 1 "Conn_01x02" V 663 9062 50  0000 R CNN
-F 2 "" H 700 9250 50  0001 C CNN
+F 2 "Connector_PinHeader_2.54mm:PinHeader_1x02_P2.54mm_Vertical" H 700 9250 50  0001 C CNN
 F 3 "~" H 700 9250 50  0001 C CNN
 	1    700  9250
@@
 $EndComp
 $Comp
-L power:+5V #PWR?
+L power:+5V #PWR0125
 U 1 1 5EEF2D0F
 P 700 9050
-F 0 "#PWR?" H 700 8900 50  0001 C CNN
+F 0 "#PWR0125" H 700 8900 50  0001 C CNN
 F 1 "+5V" H 715 9223 50  0000 C CNN
 F 2 "" H 700 9050 50  0001 C CNN
@@
 	18600 16100 18650 16100
 $Comp
-L Device:Rotary_Encoder_Switch SW?
+L Device:Rotary_Encoder_Switch SW1
 U 1 1 5F03F2CF
 P 6850 8400
-F 0 "SW?" H 6850 8767 50  0000 C CNN
+F 0 "SW1" H 6850 8767 50  0000 C CNN
 F 1 "Rotary_Encoder_Switch" H 6850 8676 50  0000 C CNN
 F 2 "" H 6700 8560 50  0001 C CNN
@@
 $EndComp
 $Comp
-L Device:Rotary_Encoder_Switch SW?
+L Device:Rotary_Encoder_Switch SW2
 U 1 1 5F041FB0
 P 6850 9050
-F 0 "SW?" H 6850 9417 50  0000 C CNN
+F 0 "SW2" H 6850 9417 50  0000 C CNN
 F 1 "Rotary_Encoder_Switch" H 6850 9326 50  0000 C CNN
 F 2 "" H 6700 9210 50  0001 C CNN
@@
 $EndComp
 $Comp
-L Device:Rotary_Encoder_Switch SW?
+L Device:Rotary_Encoder_Switch SW3
 U 1 1 5F044C02
 P 6850 9700
-F 0 "SW?" H 6850 10067 50  0000 C CNN
+F 0 "SW3" H 6850 10067 50  0000 C CNN
 F 1 "Rotary_Encoder_Switch" H 6850 9976 50  0000 C CNN
 F 2 "" H 6700 9860 50  0001 C CNN
@@
 	6400 7750 6400 10000
 $Comp
-L Device:R_POT RV?
+L Device:R_POT RV3
 U 1 1 5F06BA2B
 P 6000 8350
-F 0 "RV?" H 5931 8396 50  0000 R CNN
+F 0 "RV3" H 5931 8396 50  0000 R CNN
 F 1 "R_POT" H 5931 8305 50  0000 R CNN
-F 2 "" H 6000 8350 50  0001 C CNN
+F 2 "footprints:9MM_SNAP-IN_POT" H 6000 8350 50  0001 C CNN
 F 3 "~" H 6000 8350 50  0001 C CNN
 	1    6000 8350
@@
 $EndComp
 $Comp
-L Device:R_POT RV?
+L Device:R_POT RV4
 U 1 1 5F06C67E
 P 6000 9200
-F 0 "RV?" H 5931 9246 50  0000 R CNN
+F 0 "RV4" H 5931 9246 50  0000 R CNN
 F 1 "R_POT" H 5931 9155 50  0000 R CNN
-F 2 "" H 6000 9200 50  0001 C CNN
+F 2 "footprints:9MM_SNAP-IN_POT" H 6000 9200 50  0001 C CNN
 F 3 "~" H 6000 9200 50  0001 C CNN
 	1    6000 9200
@@
 $EndComp
 $Comp
-L Device:R_POT RV?
+L Device:R_POT RV2
 U 1 1 5F06CD44
 P 5350 9200
-F 0 "RV?" H 5281 9246 50  0000 R CNN
+F 0 "RV2" H 5281 9246 50  0000 R CNN
 F 1 "R_POT" H 5281 9155 50  0000 R CNN
-F 2 "" H 5350 9200 50  0001 C CNN
+F 2 "footprints:9MM_SNAP-IN_POT" H 5350 9200 50  0001 C CNN
 F 3 "~" H 5350 9200 50  0001 C CNN
 	1    5350 9200
@@
 $EndComp
 $Comp
-L Device:R_POT RV?
+L Device:R_POT RV1
 U 1 1 5F06D518
 P 5350 8350
-F 0 "RV?" H 5281 8396 50  0000 R CNN
+F 0 "RV1" H 5281 8396 50  0000 R CNN
 F 1 "R_POT" H 5281 8305 50  0000 R CNN
-F 2 "" H 5350 8350 50  0001 C CNN
+F 2 "footprints:9MM_SNAP-IN_POT" H 5350 8350 50  0001 C CNN
 F 3 "~" H 5350 8350 50  0001 C CNN
 	1    5350 8350
@@
 	4950 7750 4950 10000
 $Comp
-L Connector:DIN-5 J?
+L Connector:DIN-5 J29
 U 1 1 5F082697
 P 3300 8400
-F 0 "J?" H 3300 8033 50  0000 C CNN
+F 0 "J29" H 3300 8033 50  0000 C CNN
 F 1 "DIN-5" H 3300 8124 50  0000 C CNN
 F 2 "" H 3300 8400 50  0001 C CNN
@@
 $EndComp
 $Comp
-L Connector:DIN-5 J?
+L Connector:DIN-5 J30
 U 1 1 5F0833EE
 P 3300 9350
-F 0 "J?" H 3300 8983 50  0000 C CNN
+F 0 "J30" H 3300 8983 50  0000 C CNN
 F 1 "DIN-5" H 3300 9074 50  0000 C CNN
 F 2 "" H 3300 9350 50  0001 C CNN
@@
 $EndComp
 $Comp
-L Isolator:6N138 U?
+L Isolator:6N138 U7
 U 1 1 5F0A4598
 P 4150 8400
-F 0 "U?" H 4150 8867 50  0000 C CNN
+F 0 "U7" H 4150 8867 50  0000 C CNN
 F 1 "6N138" H 4150 8776 50  0000 C CNN
-F 2 "" H 4440 8100 50  0001 C CNN
+F 2 "footprints:6N138S" H 4440 8100 50  0001 C CNN
 F 3 "http://www.onsemi.com/pub/Collateral/HCPL2731-D.pdf" H 4440 8100 50  0001 C CNN
 	1    4150 8400
 	1    0    0    -1
 $EndComp
+$Comp
+L Connector_Generic:Conn_01x20 J31
+U 1 1 5F0E9788
+P 13100 3750
+F 0 "J31" H 13018 2525 50  0000 C CNN
+F 1 "Conn_01x20" H 13018 2616 50  0000 C CNN
+F 2 "Connector_PinSocket_2.54mm:PinSocket_1x20_P2.54mm_Vertical" H 13100 3750 50  0001 C CNN
+F 3 "~" H 13100 3750 50  0001 C CNN
+	1    13100 3750
+	-1   0    0    1
+$EndComp
+$Comp
+L Connector_Generic:Conn_01x20 J33
+U 1 1 5F0F1E7B
+P 14450 3750
+F 0 "J33" H 14368 2525 50  0000 C CNN
+F 1 "Conn_01x20" H 14368 2616 50  0000 C CNN
+F 2 "Connector_PinHeader_2.54mm:PinHeader_1x20_P2.54mm_Vertical" H 14450 3750 50  0001 C CNN
+F 3 "~" H 14450 3750 50  0001 C CNN
+	1    14450 3750
+	1    0    0    1
+$EndComp
+Wire Wire Line
+	13300 2750 14250 2750
+$Comp
+L Connector_Generic:Conn_01x20 J32
+U 1 1 5F1200B8
+P 13100 6200
+F 0 "J32" H 13018 4975 50  0000 C CNN
+F 1 "Conn_01x20" H 13018 5066 50  0000 C CNN
+F 2 "Connector_PinSocket_2.54mm:PinSocket_1x20_P2.54mm_Vertical" H 13100 6200 50  0001 C CNN
+F 3 "~" H 13100 6200 50  0001 C CNN
+	1    13100 6200
+	-1   0    0    1
+$EndComp
+$Comp
+L Connector_Generic:Conn_01x20 J34
+U 1 1 5F122D19
+P 14450 6200
+F 0 "J34" H 14368 4975 50  0000 C CNN
+F 1 "Conn_01x20" H 14368 5066 50  0000 C CNN
+F 2 "Connector_PinHeader_2.54mm:PinHeader_1x20_P2.54mm_Vertical" H 14450 6200 50  0001 C CNN
+F 3 "~" H 14450 6200 50  0001 C CNN
+	1    14450 6200
+	1    0    0    1
+$EndComp
+Wire Wire Line
+	13300 5200 14250 5200
 $EndSCHEMATC

Commit message: pcb w-i-p
Parts:
- J1: footprint Connector_PinHeader_2.54mm:PinHeader_1x08_P2.54mm_Vertical -> footprints:ST7735
- MIDI_IN1: renamed from J29; footprint (none) -> footprints:OG-MIDI_SD-50BV
- MIDI_OUT1: renamed from J30; footprint (none) -> footprints:OG-MIDI_SD-50BV
- SW1, SW2, SW3: footprint (none) -> Rotary_Encoder:RotaryEncoder_Alps_EC12E-Switch_Vertical_H20mm_CircularMountingHoles
- renumbered J33 to JB1, J34 to JB2, J11 to JIN1, J13 to JIN2, J15 to JIN3, J17 to JIN4, J19 to JIN5, J21 to JIN6, J23 to JIN7, J25 to JIN8, J31 to JM1, J32 to JM2, J12 to JOUT1, J14 to JOUT2, J16 to JOUT3, J18 to JOUT4, J20 to JOUT5, J22 to JOUT6, J24 to JOUT7, J26 to JOUT8
Changed lines of the file:
@@
 F 0 "J1" H 13650 1900 50  0000 L CNN
 F 1 "Conn_01x08" H 13400 1800 50  0000 L CNN
-F 2 "Connector_PinHeader_2.54mm:PinHeader_1x08_P2.54mm_Vertical" H 13700 1400 50  0001 C CNN
+F 2 "footprints:ST7735" H 13700 1400 50  0001 C CNN
 F 3 "~" H 13700 1400 50  0001 C CNN
 	1    13700 1400
@@
 	7300 7750 450  7750
 $Comp
-L Connector:AudioJack2_SwitchT J11
+L Connector:AudioJack2_SwitchT JIN1
 U 1 1 5F9E4DCE
 P 1150 14400
-F 0 "J11" H 1182 14725 50  0000 C CNN
+F 0 "JIN1" H 1182 14725 50  0000 C CNN
 F 1 "AudioJack2_SwitchT" H 1182 14634 50  0000 C CNN
 F 2 "footprints:WQP-PJ301M-12_JACK" H 1150 14400 50  0001 C CNN
@@
 $EndComp
 $Comp
-L Connector:AudioJack2_SwitchT J13
+L Connector:AudioJack2_SwitchT JIN2
 U 1 1 5F9E6243
 P 1900 14400
-F 0 "J13" H 1932 14725 50  0000 C CNN
+F 0 "JIN2" H 1932 14725 50  0000 C CNN
 F 1 "AudioJack2_SwitchT" H 1932 14634 50  0000 C CNN
 F 2 "footprints:WQP-PJ301M-12_JACK" H 1900 14400 50  0001 C CNN
@@
 $EndComp
 $Comp
-L Connector:AudioJack2_SwitchT J15
+L Connector:AudioJack2_SwitchT JIN3
 U 1 1 5F9E717F
 P 2650 14400
-F 0 "J15" H 2682 14725 50  0000 C CNN
+F 0 "JIN3" H 2682 14725 50  0000 C CNN
 F 1 "AudioJack2_SwitchT" H 2682 14634 50  0000 C CNN
 F 2 "footprints:WQP-PJ301M-12_JACK" H 2650 14400 50  0001 C CNN
@@
 $EndComp
 $Comp
-L Connector:AudioJack2_SwitchT J17
+L Connector:AudioJack2_SwitchT JIN4
 U 1 1 5F9E7A07
 P 3400 14400
-F 0 "J17" H 3432 14725 50  0000 C CNN
+F 0 "JIN4" H 3432 14725 50  0000 C CNN
 F 1 "AudioJack2_SwitchT" H 3432 14634 50  0000 C CNN
 F 2 "footprints:WQP-PJ301M-12_JACK" H 3400 14400 50  0001 C CNN
@@
 $EndComp
 $Comp
-L Connector:AudioJack2_SwitchT J21
+L Connector:AudioJack2_SwitchT JIN6
 U 1 1 5F9E920D
 P 5000 14400
-F 0 "J21" H 5032 14725 50  0000 C CNN
+F 0 "JIN6" H 5032 14725 50  0000 C CNN
 F 1 "AudioJack2_SwitchT" H 5032 14634 50  0000 C CNN
 F 2 "footprints:WQP-PJ301M-12_JACK" H 5000 14400 50  0001 C CNN
@@
 $EndComp
 $Comp
-L Connector:AudioJack2_SwitchT J23
+L Connector:AudioJack2_SwitchT JIN7
 U 1 1 5F9E9D8C
 P 5800 14400
-F 0 "J23" H 5832 14725 50  0000 C CNN
+F 0 "JIN7" H 5832 14725 50  0000 C CNN
 F 1 "AudioJack2_SwitchT" H 5832 14634 50  0000 C CNN
 F 2 "footprints:WQP-PJ301M-12_JACK" H 5800 14400 50  0001 C CNN
@@
 $EndComp
 $Comp
-L Connector:AudioJack2_SwitchT J25
+L Connector:AudioJack2_SwitchT JIN8
 U 1 1 5F9EA698
 P 6600 14400
-F 0 "J25" H 6632 14725 50  0000 C CNN
+F 0 "JIN8" H 6632 14725 50  0000 C CNN
 F 1 "AudioJack2_SwitchT" H 6632 14634 50  0000 C CNN
 F 2 "footprints:WQP-PJ301M-12_JACK" H 6600 14400 50  0001 C CNN
@@
 $EndComp
 $Comp
-L Connector:AudioJack2_SwitchT J12
+L Connector:AudioJack2_SwitchT JOUT1
 U 1 1 5F9F799A
 P 1150 15350
-F 0 "J12" H 1182 15675 50  0000 C CNN
+F 0 "JOUT1" H 1182 15675 50  0000 C CNN
 F 1 "AudioJack2_SwitchT" H 1182 15584 50  0000 C CNN
 F 2 "footprints:WQP-PJ301M-12_JACK" H 1150 15350 50  0001 C CNN
@@
 $EndComp
 $Comp
-L Connector:AudioJack2_SwitchT J14
+L Connector:AudioJack2_SwitchT JOUT2
 U 1 1 5F9F79A0
 P 1900 15350
-F 0 "J14" H 1932 15675 50  0000 C CNN
+F 0 "JOUT2" H 1932 15675 50  0000 C CNN
 F 1 "AudioJack2_SwitchT" H 1932 15584 50  0000 C CNN
 F 2 "footprints:WQP-PJ301M-12_JACK" H 1900 15350 50  0001 C CNN
@@
 $EndComp
 $Comp
-L Connector:AudioJack2_SwitchT J16
+L Connector:AudioJack2_SwitchT JOUT3
 U 1 1 5F9F79A6
 P 2650 15350
-F 0 "J16" H 2682 15675 50  0000 C CNN
+F 0 "JOUT3" H 2682 15675 50  0000 C CNN
 F 1 "AudioJack2_SwitchT" H 2682 15584 50  0000 C CNN
 F 2 "footprints:WQP-PJ301M-12_JACK" H 2650 15350 50  0001 C CNN
@@
 $EndComp
 $Comp
-L Connector:AudioJack2_SwitchT J18
+L Connector:AudioJack2_SwitchT JOUT4
 U 1 1 5F9F79AC
 P 3400 15350
-F 0 "J18" H 3432 15675 50  0000 C CNN
+F 0 "JOUT4" H 3432 15675 50  0000 C CNN
 F 1 "AudioJack2_SwitchT" H 3432 15584 50  0000 C CNN
 F 2 "footprints:WQP-PJ301M-12_JACK" H 3400 15350 50  0001 C CNN
@@
 $EndComp
 $Comp
-L Connector:AudioJack2_SwitchT J20
+L Connector:AudioJack2_SwitchT JOUT5
 U 1 1 5F9F79B2
 P 4200 15350
-F 0 "J20" H 4232 15675 50  0000 C CNN
+F 0 "JOUT5" H 4232 15675 50  0000 C CNN
 F 1 "AudioJack2_SwitchT" H 4232 15584 50  0000 C CNN
 F 2 "footprints:WQP-PJ301M-12_JACK" H 4200 15350 50  0001 C CNN
@@
 $EndComp
 $Comp
-L Connector:AudioJack2_SwitchT J22
+L Connector:AudioJack2_SwitchT JOUT6
 U 1 1 5F9F79B8
 P 5000 15350
-F 0 "J22" H 5032 15675 50  0000 C CNN
+F 0 "JOUT6" H 5032 15675 50  0000 C CNN
 F 1 "AudioJack2_SwitchT" H 5032 15584 50  0000 C CNN
 F 2 "footprints:WQP-PJ301M-12_JACK" H 5000 15350 50  0001 C CNN
@@
 $EndComp
 $Comp
-L Connector:AudioJack2_SwitchT J24
+L Connector:AudioJack2_SwitchT JOUT7
 U 1 1 5F9F79BE
 P 5800 15350
-F 0 "J24" H 5832 15675 50  0000 C CNN
+F 0 "JOUT7" H 5832 15675 50  0000 C CNN
 F 1 "AudioJack2_SwitchT" H 5832 15584 50  0000 C CNN
 F 2 "footprints:WQP-PJ301M-12_JACK" H 5800 15350 50  0001 C CNN
@@
 $EndComp
 $Comp
-L Connector:AudioJack2_SwitchT J26
+L Connector:AudioJack2_SwitchT JOUT8
 U 1 1 5F9F79C4
 P 6600 15350
-F 0 "J26" H 6632 15675 50  0000 C CNN
+F 0 "JOUT8" H 6632 15675 50  0000 C CNN
 F 1 "AudioJack2_SwitchT" H 6632 15584 50  0000 C CNN
 F 2 "footprints:WQP-PJ301M-12_JACK" H 6600 15350 50  0001 C CNN
@@
 VIN4
 $Comp
-L Connector:AudioJack2_SwitchT J19
+L Connector:AudioJack2_SwitchT JIN5
 U 1 1 5F9E8103
 P 4200 14400
-F 0 "J19" H 4232 14725 50  0000 C CNN
+F 0 "JIN5" H 4232 14725 50  0000 C CNN
 F 1 "AudioJack2_SwitchT" H 4232 14634 50  0000 C CNN
 F 2 "footprints:WQP-PJ301M-12_JACK" H 4200 14400 50  0001 C CNN
@@
 F 0 "SW1" H 6850 8767 50  0000 C CNN
 F 1 "Rotary_Encoder_Switch" H 6850 8676 50  0000 C CNN
-F 2 "" H 6700 8560 50  0001 C CNN
+F 2 "Rotary_Encoder:RotaryEncoder_Alps_EC12E-Switch_Vertical_H20mm_CircularMountingHoles" H 6700 8560 50  0001 C CNN
 F 3 "~" H 6850 8660 50  0001 C CNN
 	1    6850 8400
@@
 F 0 "SW2" H 6850 9417 50  0000 C CNN
 F 1 "Rotary_Encoder_Switch" H 6850 9326 50  0000 C CNN
-F 2 "" H 6700 9210 50  0001 C CNN
+F 2 "Rotary_Encoder:RotaryEncoder_Alps_EC12E-Switch_Vertical_H20mm_CircularMountingHoles" H 6700 9210 50  0001 C CNN
 F 3 "~" H 6850 9310 50  0001 C CNN
 	1    6850 9050
@@
 F 0 "SW3" H 6850 10067 50  0000 C CNN
 F 1 "Rotary_Encoder_Switch" H 6850 9976 50  0000 C CNN
-F 2 "" H 6700 9860 50  0001 C CNN
+F 2 "Rotary_Encoder:RotaryEncoder_Alps_EC12E-Switch_Vertical_H20mm_CircularMountingHoles" H 6700 9860 50  0001 C CNN
 F 3 "~" H 6850 9960 50  0001 C CNN
 	1    6850 9700
@@
 	4950 7750 4950 10000
 $Comp
-L Connector:DIN-5 J29
+L Connector:DIN-5 MIDI_IN1
 U 1 1 5F082697
 P 3300 8400
-F 0 "J29" H 3300 8033 50  0000 C CNN
+F 0 "MIDI_IN1" H 3300 8033 50  0000 C CNN
 F 1 "DIN-5" H 3300 8124 50  0000 C CNN
-F 2 "" H 3300 8400 50  0001 C CNN
+F 2 "footprints:OG-MIDI_SD-50BV" H 3300 8400 50  0001 C CNN
 F 3 "http://www.mouser.com/ds/2/18/40_c091_abd_e-75918.pdf" H 3300 8400 50  0001 C CNN
 	1    3300 8400
@@
 $EndComp
 $Comp
-L Connector:DIN-5 J30
+L Connector:DIN-5 MIDI_OUT1
 U 1 1 5F0833EE
 P 3300 9350
-F 0 "J30" H 3300 8983 50  0000 C CNN
+F 0 "MIDI_OUT1" H 3300 8983 50  0000 C CNN
 F 1 "DIN-5" H 3300 9074 50  0000 C CNN
-F 2 "" H 3300 9350 50  0001 C CNN
+F 2 "footprints:OG-MIDI_SD-50BV" H 3300 9350 50  0001 C CNN
 F 3 "http://www.mouser.com/ds/2/18/40_c091_abd_e-75918.pdf" H 3300 9350 50  0001 C CNN
 	1    3300 9350
@@
 $EndComp
 $Comp
-L Connector_Generic:Conn_01x20 J31
+L Connector_Generic:Conn_01x20 JM1
 U 1 1 5F0E9788
 P 13100 3750
-F 0 "J31" H 13018 2525 50  0000 C CNN
+F 0 "JM1" H 13018 2525 50  0000 C CNN
 F 1 "Conn_01x20" H 13018 2616 50  0000 C CNN
 F 2 "Connector_PinSocket_2.54mm:PinSocket_1x20_P2.54mm_Vertical" H 13100 3750 50  0001 C CNN
@@
 $EndComp
 $Comp
-L Connector_Generic:Conn_01x20 J33
+L Connector_Generic:Conn_01x20 JB1
 U 1 1 5F0F1E7B
 P 14450 3750
-F 0 "J33" H 14368 2525 50  0000 C CNN
+F 0 "JB1" H 14368 2525 50  0000 C CNN
 F 1 "Conn_01x20" H 14368 2616 50  0000 C CNN
 F 2 "Connector_PinHeader_2.54mm:PinHeader_1x20_P2.54mm_Vertical" H 14450 3750 50  0001 C CNN
@@
 	13300 2750 14250 2750
 $Comp
-L Connector_Generic:Conn_01x20 J32
+L Connector_Generic:Conn_01x20 JM2
 U 1 1 5F1200B8
 P 13100 6200
-F 0 "J32" H 13018 4975 50  0000 C CNN
+F 0 "JM2" H 13018 4975 50  0000 C CNN
 F 1 "Conn_01x20" H 13018 5066 50  0000 C CNN
 F 2 "Connector_PinSocket_2.54mm:PinSocket_1x20_P2.54mm_Vertical" H 13100 6200 50  0001 C CNN
@@
 $EndComp
 $Comp
-L Connector_Generic:Conn_01x20 J34
+L Connector_Generic:Conn_01x20 JB2
 U 1 1 5F122D19
 P 14450 6200
-F 0 "J34" H 14368 4975 50  0000 C CNN
+F 0 "JB2" H 14368 4975 50  0000 C CNN
 F 1 "Conn_01x20" H 14368 5066 50  0000 C CNN
 F 2 "Connector_PinHeader_2.54mm:PinHeader_1x20_P2.54mm_Vertical" H 14450 6200 50  0001 C CNN

Commit message: pcb w-i-p
Parts:
- removed J2, J3: Conn_02x08_Odd_Even, Connector_PinHeader_2.00mm:PinHeader_2x08_P2.00mm_Vertical, symbol Connector_Generic:Conn_02x08_Odd_Even
Changed lines of the file:
@@
-	1    0    0    -1
-$EndComp
-$Comp
-L Connector_Generic:Conn_02x08_Odd_Even J3
-U 1 1 5EEB9163
-P 15450 1400
-F 0 "J3" H 15500 1917 50  0000 C CNN
-F 1 "Conn_02x08_Odd_Even" H 15500 1826 50  0000 C CNN
-F 2 "Connector_PinHeader_2.00mm:PinHeader_2x08_P2.00mm_Vertical" H 15450 1400 50  0001 C CNN
-F 3 "~" H 15450 1400 50  0001 C CNN
-	1    15450 1400
 	1    0    0    -1
 $EndComp
@@
 Text Label 17050 12850 0    50   ~ 0
 VGND8
-Text Label 15250 1100 2    50   ~ 0
-VIN1
-Text Label 15250 1200 2    50   ~ 0
-VIN2
-Text Label 15250 1300 2    50   ~ 0
-VIN3
-Text Label 15250 1400 2    50   ~ 0
-VIN4
-Text Label 15250 1500 2    50   ~ 0
-VIN5
-Text Label 15250 1600 2    50   ~ 0
-VIN6
-Text Label 15250 1700 2    50   ~ 0
-VIN7
-Text Label 15250 1800 2    50   ~ 0
-VIN8
-Text Label 15750 1100 0    50   ~ 0
-VGND1
-Text Label 15750 1200 0    50   ~ 0
-VGND2
-Text Label 15750 1300 0    50   ~ 0
-VGND3
-Text Label 15750 1400 0    50   ~ 0
-VGND4
-Text Label 15750 1500 0    50   ~ 0
-VGND5
-Text Label 15750 1600 0    50   ~ 0
-VGND6
-Text Label 15750 1700 0    50   ~ 0
-VGND7
-Text Label 15750 1800 0    50   ~ 0
-VGND8
 $Comp
 L power:GND #PWR0100
@@
 	1    0    0    -1
 $EndComp
-$Comp
-L Connector_Generic:Conn_02x08_Odd_Even J2
-U 1 1 5F07602D
-P 14400 1400
-F 0 "J2" H 14450 1917 50  0000 C CNN
-F 1 "Conn_02x08_Odd_Even" H 14450 1826 50  0000 C CNN
-F 2 "Connector_PinHeader_2.00mm:PinHeader_2x08_P2.00mm_Vertical" H 14400 1400 50  0001 C CNN
-F 3 "~" H 14400 1400 50  0001 C CNN
-	1    14400 1400
-	1    0    0    -1
-$EndComp
 Text Label 11600 10400 0    50   ~ 0
 VOUT1
@@
 Text Label 11600 13450 0    50   ~ 0
 DAC_REF2V5
-Text Label 14200 1100 2    50   ~ 0
-VOUT1
-Text Label 14200 1200 2    50   ~ 0
-VOUT2
-Text Label 14200 1300 2    50   ~ 0
-VOUT3
-Text Label 14200 1400 2    50   ~ 0
-VOUT4
-Text Label 14200 1500 2    50   ~ 0
-VOUT5
-Text Label 14200 1600 2    50   ~ 0
-VOUT6
-Text Label 14200 1700 2    50   ~ 0
-VOUT7
-Text Label 14200 1800 2    50   ~ 0
-VOUT8
-$Comp
-L power:GND #PWR096
-U 1 1 5F088F79
-P 14700 1800
-F 0 "#PWR096" H 14700 1550 50  0001 C CNN
-F 1 "GND" H 14705 1627 50  0001 C CNN
-F 2 "" H 14700 1800 50  0001 C CNN
-F 3 "" H 14700 1800 50  0001 C CNN
-	1    14700 1800
-	1    0    0    -1
-$EndComp
-Wire Wire Line
-	14700 1800 14700 1700
-Connection ~ 14700 1800
-Wire Wire Line
-	14700 1700 14700 1600
-Connection ~ 14700 1700
-Wire Wire Line
-	14700 1500 14700 1600
-Connection ~ 14700 1600
-Wire Wire Line
-	14700 1500 14700 1400
-Connection ~ 14700 1500
-Wire Wire Line
-	14700 1400 14700 1300
-Connection ~ 14700 1400
-Wire Wire Line
-	14700 1300 14700 1200
-Connection ~ 14700 1300
-Wire Wire Line
-	14700 1200 14700 1100
-Connection ~ 14700 1200
 $Sheet
 S 6200 2000 750  400

Commit message: pcb w-i-p
Parts:
- added D?: D, symbol Device:D
- added R? (x3): 220, Resistor_SMD:R_0805_2012Metric, symbol Device:R
Connections:
- net +3V3: now also RV1.1, RV2.1, RV3.1, RV4.1, U7.8 (VCC), R?.2
- net GND: now also RV1.3, RV2.3, RV3.3, RV4.3, SW1.C, SW1.S2, SW2.C, SW2.S2, SW3.C, SW3.S2, U7.5 (GND)
- net MIDI_RX: now also U7.6 (VO2)
- net MIDI_TX: now also R?.1
- net E1A: now reaches SW1.A
- net E1B: now reaches SW1.B
- net ES1: now reaches SW1.S1
- net E2A: now reaches SW2.A
- net E2B: now reaches SW2.B
- net ES2: now reaches SW2.S1
- net E3A: now reaches SW3.A
- net E3B: now reaches SW3.B
- net ES3: now reaches SW3.S1
- net P3: now reaches RV3.2
- net P4: now reaches RV4.2
- net P2: now reaches RV2.2
- net P1: now reaches RV1.2
- net at MIDI_IN1.2: now also R?.2
- net at MIDI_IN1.4: now also U7.3 (C2), D?.2 (A)
- net at MIDI_OUT1.2: now also R?.1
- net at MIDI_OUT1.4: now also R?.2
- net at U7.2 (C1): now also D?.1 (K), R?.1
- no-connect marks 26 -> 32
Other:
- moved on the sheet: MIDI_IN1, MIDI_OUT1, RV1, RV2, RV3, RV4, U7
