File: hardware/boards/teensy-eurorack.sch (KiCad schematic (older format))
At the start: 93 parts, among them J1 Conn_01x08, J27 Conn_01x02, J28 Conn_02x08_Odd_Even, SW1 Rotary_Encoder_Switch, SW2 Rotary_Encoder_Switch, SW3 Rotary_Encoder_Switch, U1 CS42448, U2 ANALOG_DEVICES_AD5754BREZANAL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, U3 ANALOG_DEVICES_AD5754BREZANAL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, U4 Teensy4.1, U5 MCP1700-2502E_SOT23, U6 ANALOG_DEVICES_AD7606BSTZANAL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, U7 6N138

Commit message: wip
Parts:
- U4: footprint footprints:Teensy41 -> footprints:Teensy41_tht; symbol teensy-eurorack:Teensy4.1 -> teensy-eurorack:Teensy4.1_tht
- gave numbers to parts that had none: 4
Connections:
- net TFT_CLK is gone; now on net TFT_SCK: U4.35 (13_SCK_CRX1_LED)
- net +5V: now also JB2.16 (Pin_16), JM2.16 (Pin_16)
- net ADC_BUSY: now also JB1.20 (Pin_20), JM1.20 (Pin_20)
- net GND: now also JB1.1 (Pin_1), JB2.1 (Pin_1), JM1.1 (Pin_1)
- net MIDI_RX: now also JB1.3 (Pin_3), JM1.3 (Pin_3)
- net MIDI_TX: now also JB1.2 (Pin_2), JM1.2 (Pin_2)
- net TFT_CS: now also JB2.20 (Pin_20), JM2.20 (Pin_20)
- net TFT_DC: now also JB2.19 (Pin_19), JM2.19 (Pin_19)
- net TFT_MOSI: now also JB2.18 (Pin_18), JM2.18 (Pin_18)
- net TFT_SCK: now also JB2.17 (Pin_17), JM2.17 (Pin_17)
- net at JM1.17 (Pin_17): now also JB1.17 (Pin_17)
- net at JM1.18 (Pin_18): now also JB1.18 (Pin_18)
- net at JM1.19 (Pin_19): now also JB1.19 (Pin_19)
- net at JM2.12 (Pin_12): now also JB2.12 (Pin_12)
- net at JM2.13 (Pin_13): now also JB2.13 (Pin_13)
- net at JM2.14 (Pin_14): now also JB2.14 (Pin_14)
- net at JM2.15 (Pin_15): now also JB2.15 (Pin_15)
Changed lines of the file:
@@
 $EndDescr
 $Comp
-L teensy-eurorack:Teensy4.1 U4
+L teensy-eurorack:Teensy4.1_tht U4
 U 1 1 5ECE9695
 P 10050 3600
 F 0 "U4" H 10050 6165 50  0000 C CNN
 F 1 "Teensy4.1" H 10050 6074 50  0000 C CNN
-F 2 "footprints:Teensy41" H 9650 4000 50  0001 C CNN
+F 2 "footprints:Teensy41_tht" H 9650 4000 50  0001 C CNN
 F 3 "" H 9650 4000 50  0001 C CNN
 	1    10050 3600
@@
 TFT_MOSI
 Text Label 11150 2750 0    49   ~ 0
-TFT_CLK
+TFT_SCK
 Text Label 8950 1750 2    49   ~ 0
 TFT_DC
@@
 	13300 5200 14250 5200
 $Comp
-L Device:R R?
+L Device:R R37
 U 1 1 5F095AF2
 P 3200 8250
-F 0 "R?" V 2993 8250 50  0000 C CNN
+F 0 "R37" V 2993 8250 50  0000 C CNN
 F 1 "220" V 3084 8250 50  0000 C CNN
 F 2 "Resistor_SMD:R_0805_2012Metric" V 3130 8250 50  0001 C CNN
@@
 $EndComp
 $Comp
-L Device:D D?
+L Device:D D1
 U 1 1 5F099A44
 P 3350 8400
-F 0 "D?" V 3304 8480 50  0000 L CNN
+F 0 "D1" V 3304 8480 50  0000 L CNN
 F 1 "D" V 3395 8480 50  0000 L CNN
 F 2 "" H 3350 8400 50  0001 C CNN
@@
 Connection ~ 3350 8550
 $Comp
-L Device:R R?
+L Device:R R38
 U 1 1 5F0C1340
 P 3950 9400
-F 0 "R?" V 3743 9400 50  0000 C CNN
+F 0 "R38" V 3743 9400 50  0000 C CNN
 F 1 "220" V 3834 9400 50  0000 C CNN
 F 2 "Resistor_SMD:R_0805_2012Metric" V 3880 9400 50  0001 C CNN
@@
 $EndComp
 $Comp
-L power:+3V3 #PWR?
+L power:+3V3 #PWR0126
 U 1 1 5F0C1B5A
 P 3950 9250
-F 0 "#PWR?" H 3950 9100 50  0001 C CNN
+F 0 "#PWR0126" H 3950 9100 50  0001 C CNN
 F 1 "+3V3" H 3800 9350 50  0000 C CNN
 F 2 "" H 3950 9250 50  0001 C CNN
@@
 	3100 9700 2750 9700
 $Comp
-L Device:R R?
+L Device:R R36
 U 1 1 5F0D5AD0
 P 2600 9700
-F 0 "R?" V 2393 9700 50  0000 C CNN
+F 0 "R36" V 2393 9700 50  0000 C CNN
 F 1 "220" V 2484 9700 50  0000 C CNN
 F 2 "Resistor_SMD:R_0805_2012Metric" V 2530 9700 50  0001 C CNN
@@
 NoConn ~ 3400 9900
 $Comp
-L power:+3V3 #PWR?
+L power:+3V3 #PWR0127
 U 1 1 5F10C1FA
 P 4450 8200
-F 0 "#PWR?" H 4450 8050 50  0001 C CNN
+F 0 "#PWR0127" H 4450 8050 50  0001 C CNN
 F 1 "+3V3" H 4300 8300 50  0000 C CNN
 F 2 "" H 4450 8200 50  0001 C CNN
@@
 MIDI_RX
 $Comp
-L power:GND #PWR?
+L power:GND #PWR0128
 U 1 1 5F118B6C
 P 4250 8600
-F 0 "#PWR?" H 4250 8350 50  0001 C CNN
+F 0 "#PWR0128" H 4250 8350 50  0001 C CNN
 F 1 "GND" H 4255 8427 50  0000 C CNN
 F 2 "" H 4250 8600 50  0001 C CNN
@@
 $EndComp
 $Comp
-L power:+3V3 #PWR?
+L power:+3V3 #PWR0129
 U 1 1 5F11AC8F
 P 5100 8250
-F 0 "#PWR?" H 5100 8100 50  0001 C CNN
+F 0 "#PWR0129" H 5100 8100 50  0001 C CNN
 F 1 "+3V3" H 4950 8350 50  0000 C CNN
 F 2 "" H 5100 8250 50  0001 C CNN
@@
 $EndComp
 $Comp
-L power:+3V3 #PWR?
+L power:+3V3 #PWR0130
 U 1 1 5F11B855
 P 5750 8250
-F 0 "#PWR?" H 5750 8100 50  0001 C CNN
+F 0 "#PWR0130" H 5750 8100 50  0001 C CNN
 F 1 "+3V3" H 5600 8350 50  0000 C CNN
 F 2 "" H 5750 8250 50  0001 C CNN
@@
 $EndComp
 $Comp
-L power:+3V3 #PWR?
+L power:+3V3 #PWR0131
 U 1 1 5F11BC4A
 P 5750 9100
-F 0 "#PWR?" H 5750 8950 50  0001 C CNN
+F 0 "#PWR0131" H 5750 8950 50  0001 C CNN
 F 1 "+3V3" H 5600 9200 50  0000 C CNN
 F 2 "" H 5750 9100 50  0001 C CNN
@@
 $EndComp
 $Comp
-L power:+3V3 #PWR?
+L power:+3V3 #PWR0132
 U 1 1 5F11BFB5
 P 5100 9100
-F 0 "#PWR?" H 5100 8950 50  0001 C CNN
+F 0 "#PWR0132" H 5100 8950 50  0001 C CNN
 F 1 "+3V3" H 4950 9200 50  0000 C CNN
 F 2 "" H 5100 9100 50  0001 C CNN
@@
 $EndComp
 $Comp
-L power:GND #PWR?
+L power:GND #PWR0133
 U 1 1 5F11C37C
 P 5100 8550
-F 0 "#PWR?" H 5100 8300 50  0001 C CNN
+F 0 "#PWR0133" H 5100 8300 50  0001 C CNN
 F 1 "GND" H 5105 8377 50  0000 C CNN
 F 2 "" H 5100 8550 50  0001 C CNN
@@
 $EndComp
 $Comp
-L power:GND #PWR?
+L power:GND #PWR0134
 U 1 1 5F11CA38
 P 5100 9400
-F 0 "#PWR?" H 5100 9150 50  0001 C CNN
+F 0 "#PWR0134" H 5100 9150 50  0001 C CNN
 F 1 "GND" H 5105 9227 50  0000 C CNN
 F 2 "" H 5100 9400 50  0001 C CNN
@@
 $EndComp
 $Comp
-L power:GND #PWR?
+L power:GND #PWR0135
 U 1 1 5F11CE3B
 P 5750 9400
-F 0 "#PWR?" H 5750 9150 50  0001 C CNN
+F 0 "#PWR0135" H 5750 9150 50  0001 C CNN
 F 1 "GND" H 5755 9227 50  0000 C CNN
 F 2 "" H 5750 9400 50  0001 C CNN
@@
 $EndComp
 $Comp
-L power:GND #PWR?
+L power:GND #PWR0136
 U 1 1 5F11D22D
 P 5750 8550
-F 0 "#PWR?" H 5750 8300 50  0001 C CNN
+F 0 "#PWR0136" H 5750 8300 50  0001 C CNN
 F 1 "GND" H 5755 8377 50  0000 C CNN
 F 2 "" H 5750 8550 50  0001 C CNN
@@
 	1950 8950 4750 8950
 $Comp
-L power:GND #PWR?
+L power:GND #PWR0137
 U 1 1 5F1575C1
 P 7150 8500
-F 0 "#PWR?" H 7150 8250 50  0001 C CNN
+F 0 "#PWR0137" H 7150 8250 50  0001 C CNN
 F 1 "GND" H 7155 8327 50  0000 C CNN
 F 2 "" H 7150 8500 50  0001 C CNN
@@
 $EndComp
 $Comp
-L power:GND #PWR?
+L power:GND #PWR0138
 U 1 1 5F157AC5
 P 7150 9150
-F 0 "#PWR?" H 7150 8900 50  0001 C CNN
+F 0 "#PWR0138" H 7150 8900 50  0001 C CNN
 F 1 "GND" H 7155 8977 50  0000 C CNN
 F 2 "" H 7150 9150 50  0001 C CNN
@@
 $EndComp
 $Comp
-L power:GND #PWR?
+L power:GND #PWR0139
 U 1 1 5F157F41
 P 7150 9800
-F 0 "#PWR?" H 7150 9550 50  0001 C CNN
+F 0 "#PWR0139" H 7150 9550 50  0001 C CNN
 F 1 "GND" H 7155 9627 50  0000 C CNN
 F 2 "" H 7150 9800 50  0001 C CNN
@@
 $EndComp
 $Comp
-L power:GND #PWR?
+L power:GND #PWR0140
 U 1 1 5F15987D
 P 6300 8400
-F 0 "#PWR?" H 6300 8150 50  0001 C CNN
+F 0 "#PWR0140" H 6300 8150 50  0001 C CNN
 F 1 "GND" H 6305 8227 50  0000 C CNN
 F 2 "" H 6300 8400 50  0001 C CNN
@@
 $EndComp
 $Comp
-L power:GND #PWR?
+L power:GND #PWR0141
 U 1 1 5F15A4DD
 P 6300 9050
-F 0 "#PWR?" H 6300 8800 50  0001 C CNN
+F 0 "#PWR0141" H 6300 8800 50  0001 C CNN
 F 1 "GND" H 6305 8877 50  0000 C CNN
 F 2 "" H 6300 9050 50  0001 C CNN
@@
 $EndComp
 $Comp
-L power:GND #PWR?
+L power:GND #PWR0142
 U 1 1 5F15A7F1
 P 6300 9700
-F 0 "#PWR?" H 6300 9450 50  0001 C CNN
+F 0 "#PWR0142" H 6300 9450 50  0001 C CNN
 F 1 "GND" H 6305 9527 50  0000 C CNN
 F 2 "" H 6300 9700 50  0001 C CNN
@@
 Text Label 5900 9250 0    49   ~ 0
 P4
+Text Label 14250 5300 2    49   ~ 0
+TFT_DC
+Text Label 14250 5200 2    49   ~ 0
+TFT_CS
+Text Label 14250 5500 2    49   ~ 0
+TFT_SCK
+Text Label 14250 5400 2    49   ~ 0
+TFT_MOSI
+Text Label 14250 7100 2    49   ~ 0
+GND
+Text Label 14250 4650 2    49   ~ 0
+GND
+$Comp
+L power:+5V #PWR0143
+U 1 1 5F2119BB
+P 13800 5600
+F 0 "#PWR0143" H 13800 5450 50  0001 C CNN
+F 1 "+5V" H 13815 5773 50  0000 C CNN
+F 2 "" H 13800 5600 50  0001 C CNN
+F 3 "" H 13800 5600 50  0001 C CNN
+	1    13800 5600
+	1    0    0    -1
+$EndComp
+Wire Wire Line
+	13800 5600 14250 5600
+Wire Wire Line
+	13300 5300 14250 5300
+Wire Wire Line
+	13300 5400 14250 5400
+Wire Wire Line
+	13300 5500 14250 5500
+Wire Wire Line
+	13300 5600 13800 5600
+Connection ~ 13800 5600
+Wire Wire Line
+	13300 5700 14250 5700
+Wire Wire Line
+	13300 5800 14250 5800
+Wire Wire Line
+	14250 5900 13300 5900
+Wire Wire Line
+	14250 6000 13300 6000
+Wire Wire Line
+	13300 4650 14250 4650
+Wire Wire Line
+	13300 2850 14250 2850
+Wire Wire Line
+	13300 2950 14250 2950
+Wire Wire Line
+	13300 3050 14250 3050
+Text Label 13300 4550 0    49   ~ 0
+MIDI_TX
+Text Label 13300 4450 0    49   ~ 0
+MIDI_RX
+Text Label 13300 2750 0    49   ~ 0
+ADC_BUSY
+Wire Wire Line
+	13300 4550 14250 4550
+Wire Wire Line
+	14250 4450 13300 4450
 $EndSCHEMATC

Commit message: wip
Parts:
- added FPC_SD1: 1734592-8, footprints:HFW8R-1STE1LF, symbol Connector_Generic:Conn_01x10
- added SDCARD1: YAMAICHI_SD_CARD, footprints:YAMAICHI_MICROSD_VERTICAL, symbol Connector_Generic:Conn_01x10
- D1: footprint (none) -> Diode_SMD:D_0805_2012Metric
- U2, U3: value ANALOG_DEVICES_AD5754BREZANALOG_DEVICES_AD5754BREZ_0_0 -> AD5754BREZ
- U6: value ANALOG_DEVICES_AD7606BSTZANALOG_DEVICES_AD7606BSTZ_0_0 -> AD7606BSTZ
Connections:
- net DAC_LDAC is gone; now on net GND: U2.10 (~LDAC~), U3.10 (~LDAC~)
- net +12V: now also JB1.19 (Pin_19), JB2.19 (Pin_19), JM1.19 (Pin_19), JM2.19 (Pin_19)
- net +5V: now also JB2.14 (Pin_14), JM2.14 (Pin_14); no longer JB2.16 (Pin_16), JM2.16 (Pin_16)
- net -12V: now also JB1.20 (Pin_20), JB2.20 (Pin_20), JM1.20 (Pin_20), JM2.20 (Pin_20)
- net ADC_BUSY: now also JB2.13 (Pin_13), JM2.13 (Pin_13); no longer JB1.20 (Pin_20), JM1.20 (Pin_20)
- net ADC_CONVST: now also JB2.10 (Pin_10), JM2.10 (Pin_10)
- net ADC_CS: now also JB2.12 (Pin_12), JM2.12 (Pin_12); no longer U4.12 (10_CS_MQSR)
- net ADC_MISO: now also JB1.15 (Pin_15), JM1.15 (Pin_15)
- net ADC_SCK: now also JB2.11 (Pin_11), JM2.11 (Pin_11)
- net DAC_SCK: now also JB1.16 (Pin_16), JM1.16 (Pin_16)
- net DAC_SDIN: now also JB1.17 (Pin_17), JM1.17 (Pin_17)
- net DAC_SYNC: now also JB2.5 (Pin_5), JM2.5 (Pin_5)
- net GND: now also FPC_SD1.10 (Pin_10), FPC_SD1.9 (Pin_9), SDCARD1.10 (Pin_10), SDCARD1.9 (Pin_9)
- net TFT_CS: now also JB2.18 (Pin_18), JM2.18 (Pin_18); no longer JB2.20 (Pin_20), JM2.20 (Pin_20)
- net TFT_DC: now also JB2.17 (Pin_17), JM2.17 (Pin_17); no longer JB2.19 (Pin_19), JM2.19 (Pin_19)
- net TFT_MOSI: now also JB2.16 (Pin_16), JM2.16 (Pin_16); no longer JB2.18 (Pin_18), JM2.18 (Pin_18)
- net TFT_SCK: now also JB2.15 (Pin_15), JM2.15 (Pin_15); no longer JB2.17 (Pin_17), JM2.17 (Pin_17)
- net at JM1.14 (Pin_14): now also JB1.14 (Pin_14)
- new net: FPC_SD1.1 (Pin_1), SDCARD1.8 (Pin_8)
- new net: FPC_SD1.2 (Pin_2), SDCARD1.7 (Pin_7)
- new net: FPC_SD1.3 (Pin_3), SDCARD1.6 (Pin_6)
- new net: FPC_SD1.4 (Pin_4), SDCARD1.5 (Pin_5)
- new net: FPC_SD1.5 (Pin_5), SDCARD1.4 (Pin_4)
- new net: FPC_SD1.6 (Pin_6), SDCARD1.3 (Pin_3)
- new net: FPC_SD1.7 (Pin_7), SDCARD1.2 (Pin_2)
- new net: FPC_SD1.8 (Pin_8), SDCARD1.1 (Pin_1)

Commit message: slowly
Parts:
- C1, C2, C3, C4: footprint Capacitor_SMD:C_0805_2012Metric -> Capacitor_THT:CP_Radial_D5.0mm_P2.50mm
Connections:
- net +3V3: now also JB1.18 (Pin_18), JB2.2 (Pin_2), JM1.18 (Pin_18), JM2.2 (Pin_2)
- net +5V: now also JB1.14 (Pin_14), JM1.14 (Pin_14)
- net ADC_BUSY: now also JB2.11 (Pin_11), JM2.11 (Pin_11); no longer JB2.13 (Pin_13), JM2.13 (Pin_13)
- net ADC_CONVST: now also JB2.8 (Pin_8), JM2.8 (Pin_8); no longer JB2.10 (Pin_10), JM2.10 (Pin_10)
- net ADC_CS: now also JB2.10 (Pin_10), JM2.10 (Pin_10); no longer JB2.12 (Pin_12), JM2.12 (Pin_12)
- net ADC_SCK: now also JB2.9 (Pin_9), JM2.9 (Pin_9); no longer JB2.11 (Pin_11), JM2.11 (Pin_11)
- net DAC_SDOUT: now also JB2.13 (Pin_13), JM2.13 (Pin_13)
- net DAC_SYNC: now also JB2.12 (Pin_12), JM2.12 (Pin_12); no longer JB2.5 (Pin_5), JM2.5 (Pin_5)
- net GND: now also JM2.1 (Pin_1)
- net at JM2.6 (Pin_6): now also JB2.6 (Pin_6)
- new net: JB2.5 (Pin_5), JM2.5 (Pin_5)
Other:
- moved on the sheet: JB2
Changed lines of the file:
@@
 Wire Wire Line
 	12000 1350 12000 1500
-Text Label 12000 1500 0    50   ~ 0
-SDA
 $Comp
 L power:GND #PWR019
@@
 F 0 "C3" H 2418 4146 50  0000 L CNN
 F 1 "4.7u" H 2418 4055 50  0000 L CNN
-F 2 "Capacitor_SMD:C_0805_2012Metric" H 2338 3950 50  0001 C CNN
+F 2 "Capacitor_THT:CP_Radial_D5.0mm_P2.50mm" H 2338 3950 50  0001 C CNN
 F 3 "~" H 2300 4100 50  0001 C CNN
 	1    2300 4100
@@
 F 0 "C2" H 2018 4146 50  0000 L CNN
 F 1 "4.7u" H 2018 4055 50  0000 L CNN
-F 2 "Capacitor_SMD:C_0805_2012Metric" H 1938 3950 50  0001 C CNN
+F 2 "Capacitor_THT:CP_Radial_D5.0mm_P2.50mm" H 1938 3950 50  0001 C CNN
 F 3 "~" H 1900 4100 50  0001 C CNN
 	1    1900 4100
@@
 F 0 "C1" H 1618 4146 50  0000 L CNN
 F 1 "4.7u" H 1618 4055 50  0000 L CNN
-F 2 "Capacitor_SMD:C_0805_2012Metric" H 1538 3950 50  0001 C CNN
+F 2 "Capacitor_THT:CP_Radial_D5.0mm_P2.50mm" H 1538 3950 50  0001 C CNN
 F 3 "~" H 1500 4100 50  0001 C CNN
 	1    1500 4100
@@
 F 0 "C4" H 2818 4146 50  0000 L CNN
 F 1 "4.7u" H 2818 4055 50  0000 L CNN
-F 2 "Capacitor_SMD:C_0805_2012Metric" H 2738 3950 50  0001 C CNN
+F 2 "Capacitor_THT:CP_Radial_D5.0mm_P2.50mm" H 2738 3950 50  0001 C CNN
 F 3 "~" H 2700 4100 50  0001 C CNN
 	1    2700 4100
@@
 L Connector_Generic:Conn_01x20 JB2
 U 1 1 5F122D19
-P 14450 6200
-F 0 "JB2" H 14368 4975 50  0000 C CNN
-F 1 "Conn_01x20" H 14368 5066 50  0000 C CNN
-F 2 "Connector_PinHeader_2.54mm:PinHeader_1x20_P2.54mm_Vertical" H 14450 6200 50  0001 C CNN
-F 3 "~" H 14450 6200 50  0001 C CNN
-	1    14450 6200
+P 14900 6200
+F 0 "JB2" H 14818 4975 50  0000 C CNN
+F 1 "Conn_01x20" H 14818 5066 50  0000 C CNN
+F 2 "Connector_PinHeader_2.54mm:PinHeader_1x20_P2.54mm_Vertical" H 14900 6200 50  0001 C CNN
+F 3 "~" H 14900 6200 50  0001 C CNN
+	1    14900 6200
 	1    0    0    1
 $EndComp
@@
 Text Label 5900 9250 0    49   ~ 0
 P4
-Text Label 14250 5500 2    49   ~ 0
+Text Label 13300 5500 0    49   ~ 0
 TFT_DC
-Text Label 14250 5400 2    49   ~ 0
+Text Label 13300 5400 0    49   ~ 0
 TFT_CS
-Text Label 14250 5700 2    49   ~ 0
+Text Label 13300 5700 0    49   ~ 0
 TFT_SCK
-Text Label 14250 5600 2    49   ~ 0
+Text Label 13300 5600 0    49   ~ 0
 TFT_MOSI
-Text Label 14250 7100 2    49   ~ 0
+Text Label 13300 7100 0    49   ~ 0
 GND
 Text Label 14250 4650 2    49   ~ 0
@@
 	13300 5300 13950 5300
 Wire Wire Line
-	13300 5400 14250 5400
+	13300 5400 14700 5400
 Wire Wire Line
-	13300 5500 14250 5500
+	13300 5500 14700 5500
 Wire Wire Line
-	13300 5700 14250 5700
+	13300 5700 14700 5700
 Wire Wire Line
 	13300 5800 13800 5800
 Wire Wire Line
-	14250 5900 13300 5900
+	14700 5900 13300 5900
 Wire Wire Line
-	14250 6000 13300 6000
+	14700 6000 13300 6000
 Wire Wire Line
 	13300 4650 14250 4650
@@
 	13300 2850 13950 2850
 Wire Wire Line
-	13300 2950 14250 2950
-Wire Wire Line
 	13300 3050 14250 3050
 Text Label 13300 4550 0    49   ~ 0
@@
 Text Label 13300 4450 0    49   ~ 0
 MIDI_RX
-Text Label 13300 5900 0    49   ~ 0
+Text Label 13300 6100 0    49   ~ 0
 ADC_BUSY
 Wire Wire Line
@@
 Wire Wire Line
 	15250 900  15300 900
-Text Label 13300 6200 0    49   ~ 0
+Text Label 13300 6400 0    49   ~ 0
 ADC_CONVST
-Text Label 13300 6100 0    49   ~ 0
+Text Label 13300 6300 0    49   ~ 0
 ADC_SCK
-Text Label 13300 6000 0    49   ~ 0
+Text Label 13300 6200 0    49   ~ 0
 ADC_CS
 Text Label 13300 3250 0    49   ~ 0
 ADC_MISO
 Wire Wire Line
-	13300 6100 14250 6100
+	13300 6100 14700 6100
 Text Label 13300 3050 0    49   ~ 0
 DAC_SDIN
@@
 DAC_SCK
 Wire Wire Line
-	13300 6200 14250 6200
+	13300 6200 14700 6200
 Connection ~ 13800 5800
 Wire Wire Line
-	13800 5800 14250 5800
+	13800 5800 14700 5800
 Wire Wire Line
-	13300 5600 14250 5600
+	13300 5600 14700 5600
 Wire Wire Line
 	13300 3150 14250 3150
@@
 	10200 13400 10200 13450
 Wire Wire Line
-	13300 3350 14250 3350
+	13300 3350 13800 3350
 Wire Wire Line
 	13300 3250 14250 3250
@@
 Connection ~ 13700 5200
 Wire Wire Line
-	13700 5200 14250 5200
+	13700 5200 14700 5200
 Wire Wire Line
 	13950 5150 13950 5300
 Connection ~ 13950 5300
 Wire Wire Line
-	13950 5300 14250 5300
-Text Label 13300 6700 0    49   ~ 0
+	13950 5300 14700 5300
+Text Label 13300 6000 0    49   ~ 0
 DAC_SYNC
 Wire Wire Line
-	13300 6700 14250 6700
+	13300 6700 14700 6700
+Text Label 13300 5900 0    49   ~ 0
+DAC_SDOUT
+Wire Wire Line
+	13300 6600 14700 6600
+Wire Wire Line
+	13300 6300 14700 6300
+Wire Wire Line
+	13300 6400 14700 6400
+Text Label 12000 1500 0    50   ~ 0
+SDA
+$Comp
+L power:+5V #PWR0154
+U 1 1 5F032E74
+P 13800 3350
+F 0 "#PWR0154" H 13800 3200 50  0001 C CNN
+F 1 "+5V" H 13815 3523 50  0000 C CNN
+F 2 "" H 13800 3350 50  0001 C CNN
+F 3 "" H 13800 3350 50  0001 C CNN
+	1    13800 3350
+	1    0    0    -1
+$EndComp
+Connection ~ 13800 3350
+Wire Wire Line
+	13800 3350 14250 3350
+$Comp
+L power:+3V3 #PWR?
+U 1 1 5F063899
+P 12900 7000
+F 0 "#PWR?" H 12900 6850 50  0001 C CNN
+F 1 "+3V3" H 12915 7173 50  0000 C CNN
+F 2 "" H 12900 7000 50  0001 C CNN
+F 3 "" H 12900 7000 50  0001 C CNN
+	1    12900 7000
+	1    0    0    -1
+$EndComp
+Text Label 14700 7100 2    49   ~ 0
+GND
+$Comp
+L power:+3V3 #PWR?
+U 1 1 5F068C2B
+P 15100 7000
+F 0 "#PWR?" H 15100 6850 50  0001 C CNN
+F 1 "+3V3" H 15115 7173 50  0000 C CNN
+F 2 "" H 15100 7000 50  0001 C CNN
+F 3 "" H 15100 7000 50  0001 C CNN
+	1    15100 7000
+	1    0    0    -1
+$EndComp
+Wire Wire Line
+	12900 7000 13300 7000
+Wire Wire Line
+	14700 7000 15100 7000
+$Comp
+L power:+3V3 #PWR?
+U 1 1 5F089478
+P 12950 2950
+F 0 "#PWR?" H 12950 2800 50  0001 C CNN
+F 1 "+3V3" H 12965 3123 50  0000 C CNN
+F 2 "" H 12950 2950 50  0001 C CNN
+F 3 "" H 12950 2950 50  0001 C CNN
+	1    12950 2950
+	1    0    0    -1
+$EndComp
+$Comp
+L power:+3V3 #PWR?
+U 1 1 5F089EA5
+P 14650 2950
+F 0 "#PWR?" H 14650 2800 50  0001 C CNN
+F 1 "+3V3" H 14665 3123 50  0000 C CNN
+F 2 "" H 14650 2950 50  0001 C CNN
+F 3 "" H 14650 2950 50  0001 C CNN
+	1    14650 2950
+	1    0    0    -1
+$EndComp
+Wire Wire Line
+	12950 2950 13300 2950
+Connection ~ 13300 2950
+Wire Wire Line
+	13300 2950 14250 2950
+Connection ~ 14250 2950
+Wire Wire Line
+	14250 2950 14650 2950
 $EndSCHEMATC
