File: hardware/boards/teensy-eurorack-breakout.sch (KiCad schematic (older format))
At the start: 75 parts, among them J1 Conn_01x08, SW1 Rotary_Encoder_Switch, SW2 Rotary_Encoder_Switch, SW3 Rotary_Encoder_Switch, U2 AD5754BREZ, U3 AD5754BREZ, U5 MCP1700-2502E, U6 AD7606BSTZ, U7 6N138

Commit message: schematic: change dac bypass caps to polar, correct polarity
Parts:
- C19, C21, C23, C25, C31, C32, C33, C34: symbol Device:C -> Device:CP
Connections:
- net -12V: now also C31.2, C32.2, C33.2, C34.2; no longer C31.1, C32.1, C33.1, C34.1
- net GND: now also C31.1, C32.1, C33.1, C34.1; no longer C31.2, C32.2, C33.2, C34.2
Changed lines of the file:
@@
 $EndComp
 $Comp
-L Device:C C33
+L Device:CP C33
 U 1 1 5F01A320
 P 6700 4650
-F 0 "C33" H 6815 4696 50  0000 L CNN
-F 1 "10u" H 6815 4605 50  0000 L CNN
+F 0 "C33" H 6450 4700 50  0000 L CNN
+F 1 "10u" H 6450 4600 50  0000 L CNN
 F 2 "Capacitors_THT:CP_Radial_D5.0mm_P2.00mm" H 6738 4500 50  0001 C CNN
 F 3 "~" H 6700 4650 50  0001 C CNN
 	1    6700 4650
-	1    0    0    -1
-$EndComp
-$Comp
-L Device:C C32
+	-1   0    0    1
+$EndComp
+$Comp
+L Device:CP C32
 U 1 1 5F0199E8
 P 6500 4650
-F 0 "C32" H 6250 4700 50  0000 L CNN
-F 1 "0.1u" H 6250 4600 50  0000 L CNN
+F 0 "C32" H 6600 4700 50  0000 L CNN
+F 1 "0.1u" H 6600 4600 50  0000 L CNN
 F 2 "Capacitors_THT:CP_Radial_D5.0mm_P2.00mm" H 6538 4500 50  0001 C CNN
 F 3 "~" H 6500 4650 50  0001 C CNN
 	1    6500 4650
-	1    0    0    -1
+	-1   0    0    1
 $EndComp
 $Comp
@@
 $EndComp
 $Comp
-L Device:C C23
+L Device:CP C23
 U 1 1 5F0093E0
 P 4400 4600
@@
 $EndComp
 $Comp
-L Device:C C19
+L Device:CP C19
 U 1 1 5F008568
 P 4200 4600
@@
 $EndComp
 $Comp
-L Device:C C34
+L Device:CP C34
 U 1 1 5EFF5A69
 P 6700 2100
-F 0 "C34" H 6815 2146 50  0000 L CNN
-F 1 "10u" H 6815 2055 50  0000 L CNN
+F 0 "C34" H 6450 2150 50  0000 L CNN
+F 1 "10u" H 6500 2000 50  0000 L CNN
 F 2 "Capacitors_THT:CP_Radial_D5.0mm_P2.00mm" H 6738 1950 50  0001 C CNN
 F 3 "~" H 6700 2100 50  0001 C CNN
 	1    6700 2100
-	1    0    0    -1
+	-1   0    0    1
 $EndComp
 $Comp
@@
 $EndComp
 $Comp
-L Device:C C21
+L Device:CP C21
 U 1 1 5EFF14C2
 P 4150 2100
@@
 $EndComp
 $Comp
-L Device:C C31
+L Device:CP C31
 U 1 1 5EFEC162
 P 6500 2100
-F 0 "C31" H 6250 2150 50  0000 L CNN
-F 1 "0.1u" H 6250 2050 50  0000 L CNN
+F 0 "C31" H 6600 2150 50  0000 L CNN
+F 1 "0.1u" H 6600 2050 50  0000 L CNN
 F 2 "Capacitors_THT:CP_Radial_D5.0mm_P2.00mm" H 6538 1950 50  0001 C CNN
 F 3 "~" H 6500 2100 50  0001 C CNN
 	1    6500 2100
-	1    0    0    -1
+	-1   0    0    1
 $EndComp
 $Comp
@@
 NoConn ~ 9850 750
 $Comp
-L Device:C C25
+L Device:CP C25
 U 1 1 5EFEB20A
 P 4350 2100

Commit message: schematic: adc to use same external voltage reference as dac
Connections:
- net +3V3: no longer R7.1
- net DAC_REF2V5: now also U6.42 (REFIN/REFOUT)
- net GND: now also R7.1
- no-connect marks 32 -> 31
Changed lines of the file:
@@
 	1    0    0    -1
 $EndComp
-NoConn ~ 3000 4050
 $Comp
 L Device:R R7
@@
 	1    3150 3850
 	0    1    1    0
-$EndComp
-$Comp
-L power:+3V3 #PWR0105
-U 1 1 5EEE48C9
-P 3300 3850
-F 0 "#PWR0105" H 3300 3700 50  0001 C CNN
-F 1 "+3V3" H 3315 4023 50  0000 C CNN
-F 2 "" H 3300 3850 50  0001 C CNN
-F 3 "" H 3300 3850 50  0001 C CNN
-	1    3300 3850
-	1    0    0    -1
 $EndComp
 Wire Wire Line
@@
 Wire Wire Line
 	3850 950  3850 3400
+Text Label 3000 4050 0    50   ~ 0
+DAC_REF2V5
+$Comp
+L power:GND #PWR?
+U 1 1 5FC61711
+P 3450 3850
+F 0 "#PWR?" H 3450 3600 50  0001 C CNN
+F 1 "GND" H 3455 3677 50  0001 C CNN
+F 2 "" H 3450 3850 50  0001 C CNN
+F 3 "" H 3450 3850 50  0001 C CNN
+	1    3450 3850
+	1    0    0    -1
+$EndComp
+Wire Wire Line
+	3300 3850 3450 3850
 $EndSCHEMATC
